File: dc_valve_control.sch (KiCad schematic (older format))
At the start: 33 parts

Commit message: tarpinis kommitas
Parts:
- removed J?: Valves LimitSW, symbol Connector_Generic:Conn_02x08_Counter_Clockwise
- added D13, D14, D16, D17: D, Diodes_SMD:D_MiniMELF, symbol ihouse-rescue:Device_D-ihouse-rescue
- added J13, J14, J15, J16: Conn_01x04, Connectors_Molex:Molex_KK-6410-04_04x2.54mm_Straight, symbol ihouse-rescue:Conn_01x04-ihouse-rescue
- added R43, R44, R45, R46, R47, R48, R50, R51, R52, R53, R54, R55, R56, R57: R, Resistors_SMD:R_0805, symbol ihouse-rescue:Device_R-ihouse-rescue
- C10, C11, C2, C3, C4, C5, C6, C7, C8, C9: renamed from C?; footprint (none) -> Capacitors_SMD:C_0805; symbol Device:C -> ihouse-rescue:Device_C-ihouse-rescue
- D15: renamed from D?; footprint (none) -> Diodes_SMD:D_MiniMELF; symbol Device:D -> ihouse-rescue:Device_D-ihouse-rescue
- D18, D19: renamed from D?; symbol Device:D -> ihouse-rescue:Device_D-ihouse-rescue
- J12: renamed from J?; footprint (none) -> Connectors_Molex:Molex_MiniFit-JR-5556-10A_2x05x4.20mm_Straight; symbol Connector_Generic:Conn_02x05_Counter_Clockwise -> ihouse-rescue:Connector_Generic_Conn_02x05_Counter_Clockwise-ihouse-rescue
- K10, K11, K14, K15: renamed from K?; value FINDER-40.51 -> FINDER-34.51; footprint Relay_THT:Relay_SPST_Schrack-RP-II-1-FormA_RM5mm -> Relays_THT:Relay_SPDT_SingleRow_Standing_FinderType34Point51; symbol Relay:FINDER-40.51 -> ihouse-rescue:Relay_FINDER-40.51-ihouse-rescue
- K12, K13, K16, K17: renamed from K?; footprint Relay_THT:Relay_DPDT_Schrack-RT2-FormC_RM5mm -> Relays_THT:Relay_DPDT_Schrack-RT2-FormC_RM5mm; symbol Relay:RT42xxxx -> ihouse-rescue:Relay_RT42xxxx-ihouse-rescue
- M1: renamed from M?; symbol Motor:Motor_DC -> ihouse-rescue:Motor_Motor_DC-ihouse-rescue
- R49: renamed from R?; footprint (none) -> Resistors_SMD:R_0805; symbol Device:R -> ihouse-rescue:Device_R-ihouse-rescue
- RN1, RN2, RN3, RN4: renamed from RN?; footprint (none) -> Resistors_SMD:R_Array_Convex_4x1206; symbol Device:R_Pack04 -> ihouse-rescue:Device_R_Pack04-ihouse-rescue
- SW1, SW2: renamed from SW?; symbol Switch:SW_Push_Open -> ihouse-rescue:Switch_SW_Push_Open-ihouse-rescue
- U15: renamed from U?; symbol dk_Interface-I-O-Expanders:MCP23017-E_SP -> ihouse-rescue:dk_Interface-I-O-Expanders_MCP23017-E_SP-ihouse-rescue
- U16: renamed from U?; footprint (none) -> Housings_SOIC:SOIC-18W_7.5x11.6mm_Pitch1.27mm; symbol Transistor_Array:ULN2803A -> ihouse-rescue:Transistor_Array_ULN2803A-ihouse-rescue
Connections:
- net labels added: V1TP, V1TST, V2TP, V2TST, V3TP, V3TST, V4TP, V4TST
- wire segments 283 -> 347
