File: power_outputs.sch (KiCad schematic (older format))
At the start: 23 parts, among them K1 FINDER-32.21-x300, K2 RT42xxxx, K3 FINDER-32.21-x300, K4 RT42xxxx, K5 G5Q-1A, K6 G5Q-1A, U3 MOC3060S, U4 LTV-817, U5 MOC3060S

Commit message: schemos paruosimas
Parts:
- removed D4: Z0103MN, Package_TO_SOT_SMD:SOT-223, symbol Triac_Thyristor:Z0103MN
- removed K2: RT42xxxx, Relay_THT:Relay_DPDT_Schrack-RT2-FormC_RM5mm, symbol Relay:RT42xxxx
- removed K5: G5Q-1A, Relay_THT:Relay_SPDT_Finder_34.51_Vertical, symbol Relay:G5Q-1A
- removed R16, R17, R18: R, Resistor_SMD:R_0805_2012Metric_Pad1.15x1.40mm_HandSolder, symbol Device:R
- removed U5: MOC3060S, disc:DIP-6_W9.53mm_SMD, symbol disc:MOC3060S
- added D? (x9): Z0103MN, Package_TO_SOT_SMD:SOT-223, symbol Triac_Thyristor:Z0103MN
- added K?: FINDER-40.51, Relay_THT:Relay_SPST_Schrack-RP-II-1-FormA_RM5mm, symbol Relay:FINDER-40.51
- added R? (x27): R, Resistor_SMD:R_0805_2012Metric_Pad1.15x1.40mm_HandSolder, symbol Device:R
- added U? (x9): MOC3060S, disc:DIP-6_W9.53mm_SMD, symbol disc:MOC3060S
- renumbered D3 to D?, D2 to D?, F1 to F?, K4 to K?, K1 to K?, K3 to K?, K6 to K?, R10 to R?, R11 to R?, R13 to R?, R14 to R?, R15 to R?, R9 to R?, R12 to R?, U3 to U?, U4 to U?
Connections:
- net labels added: INACL1, INACL2, INACN1, INACN2, OAC1, OAC2, OAC3, OAC4, OAC5, OAC6, OAC7, OAC8, OAC9, OUTAC1, OUTAC10, OUTAC10N, OUTAC2, OUTAC3, OUTAC4, OUTAC5, OUTAC6, OUTAC7, OUTAC8, OUTAC9
- net labels removed: EAKITCHN, EAWCN, EHALLLIGHT, EHALLLIGHT_N, ExtractAir_KITCH, ExtractAir_WC, ISOCKN, K2, LIGHTBASH1, LIGHTBASH2, LIGHTWC1, LIGHTWC2, OC2, WORKLIGHT, WORKLIGHT_N, iSocket
- wire segments 108 -> 209
Other:
- note removed: "Arkos rozete"
- note removed: "Koridoriaus\napsvietimas"
- note removed: "Virtuves darbo\nzonos apsvietimas"
- note removed: "Virtuves\nventiliatorius"
- note removed: "Vonios apsvietimas\n230VAC"
- note removed: "Vonios ir WC\nventiliatorius"
- note removed: "WC apsvietimas\n230VAC"

Commit message: tarpinis kommitas
Parts:
- removed D?: LL4148, Diode_SMD:D_MiniMELF, symbol Diode:LL4148
- removed D? (x7): Z0103MN, Package_TO_SOT_SMD:SOT-223, symbol Triac_Thyristor:Z0103MN
- removed F?: 3A, Fuse:Fuseholder_Cylinder-5x20mm_Schurter_0031_8201_Horizontal_Open, symbol Device:Fuse
- removed K?: RT42xxxx, Relay_THT:Relay_DPDT_Schrack-RT2-FormC_RM5mm, symbol Relay:RT42xxxx
- removed K?: FINDER-32.21-x300, Relay_THT:Relay_SPST_Schrack-RT1-FormA_RM5mm, symbol Relay:FINDER-32.21-x300
- removed K?: G5Q-1A, Relay_THT:Relay_SPDT_Finder_34.51_Vertical, symbol Relay:G5Q-1A
- removed K?: FINDER-40.51, Relay_THT:Relay_SPST_Schrack-RP-II-1-FormA_RM5mm, symbol Relay:FINDER-40.51
- removed R? (x15): R, Resistor_SMD:R_0805_2012Metric_Pad1.15x1.40mm_HandSolder, symbol Device:R
- removed R? (x3): 33k, Resistor_SMD:R_1206_3216Metric_Pad1.42x1.75mm_HandSolder, symbol Device:R
- removed U? (x5): MOC3060S, disc:DIP-6_W9.53mm_SMD, symbol disc:MOC3060S
- removed U?: LTV-817, Package_DIP:DIP-4_W7.62mm, symbol Isolator:LTV-817
- added D10, D11, D12, D2, D5, D7, D8: Z0103MN, Package_TO_SOT_SMD:SOT-223, symbol Triac_Thyristor:Z0103MN
- added D3: LL4148, Diode_SMD:D_MiniMELF, symbol Diode:LL4148
- added F1: 3A, Fuse:Fuseholder_Cylinder-5x20mm_Schurter_0031_8201_Horizontal_Open, symbol Device:Fuse
- added J?: EXT1, symbol Connector:Screw_Terminal_01x03
- added J?: EXT2, symbol Connector:Screw_Terminal_01x03
- added J?: EXT3, symbol Connector:Screw_Terminal_01x03
- added J?: EXT4, symbol Connector:Screw_Terminal_01x03
- added K1: FINDER-32.21-x300, Relay_THT:Relay_SPST_Schrack-RT1-FormA_RM5mm, symbol Relay:FINDER-32.21-x300
- added K2, K? (x4): FINDER-40.51, Relay_THT:Relay_SPST_Schrack-RP-II-1-FormA_RM5mm, symbol Relay:FINDER-40.51
- added K4: RT42xxxx, Relay_THT:Relay_DPDT_Schrack-RT2-FormC_RM5mm, symbol Relay:RT42xxxx
- added K5: G5Q-1A, Relay_THT:Relay_SPDT_Finder_34.51_Vertical, symbol Relay:G5Q-1A
- added R11, R15, R18, R19, R20, R21, R22, R25, R27, R28, R31, R32, R37, R38, R39: R, Resistor_SMD:R_0805_2012Metric_Pad1.15x1.40mm_HandSolder, symbol Device:R
- added R12, R13, R17: 33k, Resistor_SMD:R_1206_3216Metric_Pad1.42x1.75mm_HandSolder, symbol Device:R
- added U10, U12, U4, U7, U9: MOC3060S, disc:DIP-6_W9.53mm_SMD, symbol disc:MOC3060S
- added U5: LTV-817, Package_DIP:DIP-4_W7.62mm, symbol Isolator:LTV-817
- added U?: ULN2803A, symbol Transistor_Array:ULN2803A
- gave numbers to parts that had none: 25
Connections:
- net labels added: EXT1, EXT1_11, EXT1_12, EXT1_14, EXT2, EXT2_11, EXT2_12, EXT2_14, EXT3, EXT3_11, EXT3_12, EXT3_14, EXT4, EXT4_11, EXT4_12, EXT4_14
- wire segments 209 -> 269

Commit message: tarpinis kommitas
Parts:
- D10, D11, D12, D4, D5, D6, D7, D8, D9: symbol Triac_Thyristor:Z0103MN -> ihouse-rescue:Triac_Thyristor_Z0103MN-ihouse-rescue
- D2: renamed from D3; symbol Diode:LL4148 -> ihouse-rescue:Diode_LL4148-ihouse-rescue
- D3: renamed from D2; symbol Triac_Thyristor:Z0103MN -> ihouse-rescue:Triac_Thyristor_Z0103MN-ihouse-rescue
- F1: symbol Device:Fuse -> ihouse-rescue:Device_Fuse-ihouse-rescue
- J10, J11, J8, J9: renamed from J?; symbol Connector:Screw_Terminal_01x03 -> ihouse-rescue:Connector_Screw_Terminal_01x03-ihouse-rescue
- K1: renamed from K2; symbol Relay:FINDER-40.51 -> ihouse-rescue:Relay_FINDER-40.51-ihouse-rescue
- K2: renamed from K4; symbol Relay:RT42xxxx -> ihouse-rescue:Relay_RT42xxxx-ihouse-rescue
- K3, K4, K5, K6: renamed from K?; symbol Relay:FINDER-40.51 -> ihouse-rescue:Relay_FINDER-40.51-ihouse-rescue
- K7: renamed from K1; symbol Relay:FINDER-32.21-x300 -> ihouse-rescue:Relay_FINDER-32.21-x300-ihouse-rescue
- K8: renamed from K3; symbol Relay:FINDER-32.21-x300 -> ihouse-rescue:Relay_FINDER-32.21-x300-ihouse-rescue
- K9: renamed from K5; symbol Relay:G5Q-1A -> ihouse-rescue:Relay_G5Q-1A-ihouse-rescue
- R10: renamed from R12; symbol Device:R -> ihouse-rescue:Device_R-ihouse-rescue
- R11: renamed from R16; symbol Device:R -> ihouse-rescue:Device_R-ihouse-rescue
- R12: renamed from R13; symbol Device:R -> ihouse-rescue:Device_R-ihouse-rescue
- R13: renamed from R17; symbol Device:R -> ihouse-rescue:Device_R-ihouse-rescue
- R14: renamed from R10; symbol Device:R -> ihouse-rescue:Device_R-ihouse-rescue
- R15: renamed from R11; symbol Device:R -> ihouse-rescue:Device_R-ihouse-rescue
- R16: renamed from R14; symbol Device:R -> ihouse-rescue:Device_R-ihouse-rescue
- R17: renamed from R19; symbol Device:R -> ihouse-rescue:Device_R-ihouse-rescue
- R18: renamed from R22; symbol Device:R -> ihouse-rescue:Device_R-ihouse-rescue
- R19: renamed from R25; symbol Device:R -> ihouse-rescue:Device_R-ihouse-rescue
- R20: renamed from R28; symbol Device:R -> ihouse-rescue:Device_R-ihouse-rescue
- R21: renamed from R31; symbol Device:R -> ihouse-rescue:Device_R-ihouse-rescue
- R22: renamed from R34; symbol Device:R -> ihouse-rescue:Device_R-ihouse-rescue
- R23: renamed from R37; symbol Device:R -> ihouse-rescue:Device_R-ihouse-rescue
- R24: renamed from R40; symbol Device:R -> ihouse-rescue:Device_R-ihouse-rescue
- R25: renamed from R15; symbol Device:R -> ihouse-rescue:Device_R-ihouse-rescue
- R26: renamed from R18; symbol Device:R -> ihouse-rescue:Device_R-ihouse-rescue
- R27: renamed from R20; symbol Device:R -> ihouse-rescue:Device_R-ihouse-rescue
- R28: renamed from R21; symbol Device:R -> ihouse-rescue:Device_R-ihouse-rescue
- R29: renamed from R23; symbol Device:R -> ihouse-rescue:Device_R-ihouse-rescue
- R30: renamed from R24; symbol Device:R -> ihouse-rescue:Device_R-ihouse-rescue
- R31: renamed from R26; symbol Device:R -> ihouse-rescue:Device_R-ihouse-rescue
- R32: renamed from R27; symbol Device:R -> ihouse-rescue:Device_R-ihouse-rescue
- R33: renamed from R29; symbol Device:R -> ihouse-rescue:Device_R-ihouse-rescue
- R34: renamed from R30; symbol Device:R -> ihouse-rescue:Device_R-ihouse-rescue
- R35: renamed from R32; symbol Device:R -> ihouse-rescue:Device_R-ihouse-rescue
- R36: renamed from R33; symbol Device:R -> ihouse-rescue:Device_R-ihouse-rescue
- R37: renamed from R35; symbol Device:R -> ihouse-rescue:Device_R-ihouse-rescue
- R38: renamed from R36; symbol Device:R -> ihouse-rescue:Device_R-ihouse-rescue
- R39: renamed from R38; symbol Device:R -> ihouse-rescue:Device_R-ihouse-rescue
- R40: renamed from R39; symbol Device:R -> ihouse-rescue:Device_R-ihouse-rescue
- R41, R42, R9: symbol Device:R -> ihouse-rescue:Device_R-ihouse-rescue
- U10: renamed from U9; symbol disc:MOC3060S -> ihouse-rescue:disc_MOC3060S-ihouse-rescue
- U11: renamed from U10; symbol disc:MOC3060S -> ihouse-rescue:disc_MOC3060S-ihouse-rescue
- U12: renamed from U11; symbol disc:MOC3060S -> ihouse-rescue:disc_MOC3060S-ihouse-rescue
- U13: renamed from U12; symbol disc:MOC3060S -> ihouse-rescue:disc_MOC3060S-ihouse-rescue
- U14: renamed from U13; symbol disc:MOC3060S -> ihouse-rescue:disc_MOC3060S-ihouse-rescue
- U3: renamed from U?; symbol Transistor_Array:ULN2803A -> ihouse-rescue:Transistor_Array_ULN2803A-ihouse-rescue
- U4: renamed from U5; symbol Isolator:LTV-817 -> ihouse-rescue:Isolator_LTV-817-ihouse-rescue
- U5: renamed from U3; symbol disc:MOC3060S -> ihouse-rescue:disc_MOC3060S-ihouse-rescue
- U6: renamed from U4; symbol disc:MOC3060S -> ihouse-rescue:disc_MOC3060S-ihouse-rescue
- U7: renamed from U6; symbol disc:MOC3060S -> ihouse-rescue:disc_MOC3060S-ihouse-rescue
- U8: renamed from U7; symbol disc:MOC3060S -> ihouse-rescue:disc_MOC3060S-ihouse-rescue
- U9: renamed from U8; symbol disc:MOC3060S -> ihouse-rescue:disc_MOC3060S-ihouse-rescue
