File: ihouse.sch (KiCad schematic (older format))
At the start: 0 parts

Commit message: tarpinis komitas
Parts:
- added J1, J2, J3, J4: Conn_01x01, mech:Faston_6.3x0.8x14, symbol Connector_Generic:Conn_01x01
- added J5: Conn_01x16, Connectors_Phoenix:PhoenixContact_MSTBA-G_16x5.00mm_Angled, symbol Connector_Generic:Conn_01x16
- added J6, J7: Conn_01x02, Connectors_Phoenix:PhoenixContact_MSTBA-G_02x5.00mm_Angled, symbol Connector_Generic:Conn_01x02
- added J?: Conn_01x03, Connectors_Phoenix:PhoenixContact_MSTBA-G_03x5.00mm_Angled, symbol Connector_Generic:Conn_01x03
Connections:
- net labels added: 230VAC_L, 230VAC_N, AIREXT_L, AIREXT_N, BASHCAB_L, BASHCAB_N, EHALLIT_L, EHALLIT_N, EXTKITCH_L, EXTKITCH_N, EXTWC_L, EXTWC_N, ISOCK_L, ISOCK_N, PE, WRKLIT_L, WRKLIT_N
- net labels removed: EAWCN, ExtractAir_WC, ISOCKN, iSocket
- wire segments 0 -> 57
Other:
- note added: "Duso kabina"
- note added: "Garu surinkejas"

Commit message: schemos paruosimas
Parts:
- removed J5: Conn_01x16, Connectors_Phoenix:PhoenixContact_MSTBA-G_16x5.00mm_Angled, symbol Connector_Generic:Conn_01x16
- removed J6, J7: Conn_01x02, Connectors_Phoenix:PhoenixContact_MSTBA-G_02x5.00mm_Angled, symbol Connector_Generic:Conn_01x02
- added J?: AC OUTS, Connector_Molex:Molex_Mini-Fit_Jr_5566-24A_2x12_P4.20mm_Vertical, symbol Connector_Generic:Conn_02x12_Counter_Clockwise
- added J?: AC INPUTS, Connector_Molex:Molex_Mini-Fit_Jr_5566-04A_2x02_P4.20mm_Vertical, symbol Connector_Generic:Conn_02x02_Counter_Clockwise
- renumbered J1 to J?, J2 to J?, J3 to J?, J4 to J?
Connections:
- net labels added: ACN, INACL1, INACL2, INACN1, INACN2, OUTAC1, OUTAC10, OUTAC10N, OUTAC11, OUTAC11N, OUTAC12, OUTAC12N, OUTAC2, OUTAC3, OUTAC4, OUTAC5, OUTAC6, OUTAC7, OUTAC8, OUTAC9
- net labels removed: AIREXT_L, AIREXT_N, BASHCAB_L, BASHCAB_N, EHALLIT_L, EHALLIT_N, EXTKITCH_L, EXTKITCH_N, EXTWC_L, EXTWC_N, ISOCK_L, ISOCK_N, WRKLIT_L, WRKLIT_N
- wire segments 57 -> 64
Other:
- note added: "INACL1 -> WC apsvietimas L\nINACN1 -> WC apsvietimas N\nINACL2 -> vonios apsvietimas L\nINACN2 -> vonios apsvietimas N"
- note added: "OUTAC1 -> lempa 1\nOUTAC2 -> lempa 2\nOUTAC3 -> lempa 3\nOUTAC4 -> lempa 4\nOUTAC5 -> lempa 5\nOUTAC6 -> koridoriaus apsvietimas\nOUTAC7 -> \nOUTAC8 -> \nOUTAC9 -> ventiliatorius WC\nOUTAC10 -> protinga rozete\nOUTAC11 -> garu surinktuvas\nOUTAC12 -> duso kabina"
- note removed: "Duso kabina"
- note removed: "Garu surinkejas"

Commit message: tarpinis kommitas
Parts:
- gave numbers to parts that had none: 7
Changed lines of the file:
@@
 $Descr A4 11693 8268
 encoding utf-8
-Sheet 1 3
+Sheet 1 4
 Title ""
 Date ""
@@
 $EndDescr
 $Sheet
-S 2100 1350 1950 4700
+S 2000 5200 1750 1550
 U 5BC6397F
 F0 "Controller" 50
@@
 PE
 $Comp
-L Connector_Generic:Conn_01x01 J?
+L Connector_Generic:Conn_01x01 J1
 U 1 1 5BC9AA2A
 P 10550 1600
-F 0 "J?" H 10630 1596 50  0000 L CNN
+F 0 "J1" H 10630 1596 50  0000 L CNN
 F 1 "Conn_01x01" H 10630 1551 50  0001 L CNN
 F 2 "mech:Faston_6.3x0.8x14" H 10550 1600 50  0001 C CNN
@@
 $EndComp
 $Comp
-L Connector_Generic:Conn_01x01 J?
+L Connector_Generic:Conn_01x01 J2
 U 1 1 5BC9AB40
 P 10550 1750
-F 0 "J?" H 10630 1746 50  0000 L CNN
+F 0 "J2" H 10630 1746 50  0000 L CNN
 F 1 "Conn_01x01" H 10630 1701 50  0001 L CNN
 F 2 "mech:Faston_6.3x0.8x14" H 10550 1750 50  0001 C CNN
@@
 $EndComp
 $Comp
-L Connector_Generic:Conn_01x01 J?
+L Connector_Generic:Conn_01x01 J3
 U 1 1 5BC9AB58
 P 10550 1900
-F 0 "J?" H 10630 1896 50  0000 L CNN
+F 0 "J3" H 10630 1896 50  0000 L CNN
 F 1 "Conn_01x01" H 10630 1851 50  0001 L CNN
 F 2 "mech:Faston_6.3x0.8x14" H 10550 1900 50  0001 C CNN
@@
 $EndComp
 $Comp
-L Connector_Generic:Conn_01x01 J?
+L Connector_Generic:Conn_01x01 J4
 U 1 1 5BC9AB72
 P 10550 2050
-F 0 "J?" H 10630 2046 50  0000 L CNN
+F 0 "J4" H 10630 2046 50  0000 L CNN
 F 1 "Conn_01x01" H 10630 2001 50  0001 L CNN
 F 2 "mech:Faston_6.3x0.8x14" H 10550 2050 50  0001 C CNN
@@
 	6400 4050 6700 4050
 $Comp
-L Connector_Generic:Conn_01x03 J?
+L Connector_Generic:Conn_01x03 J5
 U 1 1 5BC74B70
 P 10550 2550
-F 0 "J?" H 10630 2546 50  0000 L CNN
+F 0 "J5" H 10630 2546 50  0000 L CNN
 F 1 "Conn_01x03" H 10630 2501 50  0001 L CNN
 F 2 "Connectors_Phoenix:PhoenixContact_MSTBA-G_03x5.00mm_Angled" H 10550 2550 50  0001 C CNN
@@
 P 6050 5850
 AR Path="/5BC77CC5/5C039156" Ref="J?"  Part="1"
-AR Path="/5C039156" Ref="J?"  Part="1"
-F 0 "J?" H 6100 6450 50  0000 C CNN
+AR Path="/5C039156" Ref="J7"  Part="1"
+F 0 "J7" H 6100 6450 50  0000 C CNN
 F 1 "AC OUTS" H 6100 5150 50  0000 C CNN
 F 2 "Connector_Molex:Molex_Mini-Fit_Jr_5566-24A_2x12_P4.20mm_Vertical" H 6050 5850 50  0001 C CNN
@@
 P 7800 5350
 AR Path="/5BC77CC5/5C03917E" Ref="J?"  Part="1"
-AR Path="/5C03917E" Ref="J?"  Part="1"
-F 0 "J?" H 7850 5450 50  0000 C CNN
+AR Path="/5C03917E" Ref="J6"  Part="1"
+F 0 "J6" H 7850 5450 50  0000 C CNN
 F 1 "AC INPUTS" H 7850 5150 50  0000 C CNN
 F 2 "Connector_Molex:Molex_Mini-Fit_Jr_5566-04A_2x02_P4.20mm_Vertical" H 7800 5350 50  0001 C CNN
@@
 F36 "OAC9" I R 7900 2950 50
 $EndSheet
+$Sheet
+S 2000 1200 1750 1250
+U 5E405C96
+F0 "DC sklendziu valdymas" 50
+F1 "dc_valve_control.sch" 50
+$EndSheet
 $EndSCHEMATC

Commit message: tarpinis kommitas
Parts:
- J1: renamed from J7; symbol Connector_Generic:Conn_02x12_Counter_Clockwise -> ihouse-rescue:Connector_Generic_Conn_02x12_Counter_Clockwise-ihouse-rescue
- J2: renamed from J6; symbol Connector_Generic:Conn_02x02_Counter_Clockwise -> ihouse-rescue:Connector_Generic_Conn_02x02_Counter_Clockwise-ihouse-rescue
- J3: renamed from J1; symbol Connector_Generic:Conn_01x01 -> ihouse-rescue:Connector_Generic_Conn_01x01-ihouse-rescue
- J4: renamed from J2; symbol Connector_Generic:Conn_01x01 -> ihouse-rescue:Connector_Generic_Conn_01x01-ihouse-rescue
- J5: renamed from J3; symbol Connector_Generic:Conn_01x01 -> ihouse-rescue:Connector_Generic_Conn_01x01-ihouse-rescue
- J6: renamed from J4; symbol Connector_Generic:Conn_01x01 -> ihouse-rescue:Connector_Generic_Conn_01x01-ihouse-rescue
- J7: renamed from J5; symbol Connector_Generic:Conn_01x03 -> ihouse-rescue:Connector_Generic_Conn_01x03-ihouse-rescue
Changed lines of the file:
@@
 $EndSheet
 Wire Wire Line
-	6700 2150 6500 2150
-Wire Wire Line
-	6700 2250 6600 2250
+	6000 2150 6500 2150
+Wire Wire Line
+	6000 2250 6600 2250
 Text Label 6000 2150 0    50   ~ 0
 230VAC_L
@@
 Connection ~ 6500 2150
 Wire Wire Line
-	6500 2150 6000 2150
-Wire Wire Line
-	6600 2250 6600 1600
+	6600 1350 6600 1600
 Wire Wire Line
 	6600 1350 7300 1350
 Connection ~ 6600 2250
 Wire Wire Line
-	6600 2250 6000 2250
-Wire Wire Line
 	6500 1500 7300 1500
 Connection ~ 6500 1500
 Wire Wire Line
-	6500 1500 6500 1250
+	6500 1250 6500 1500
 Text Label 7300 1250 2    50   ~ 0
 OUTAC11
@@
 PE
 $Comp
-L Connector_Generic:Conn_01x01 J1
+L ihouse-rescue:Connector_Generic_Conn_01x01-ihouse-rescue J3
 U 1 1 5BC9AA2A
 P 10550 1600
-F 0 "J1" H 10630 1596 50  0000 L CNN
+F 0 "J3" H 10630 1596 50  0000 L CNN
 F 1 "Conn_01x01" H 10630 1551 50  0001 L CNN
 F 2 "mech:Faston_6.3x0.8x14" H 10550 1600 50  0001 C CNN
@@
 $EndComp
 $Comp
-L Connector_Generic:Conn_01x01 J2
+L ihouse-rescue:Connector_Generic_Conn_01x01-ihouse-rescue J4
 U 1 1 5BC9AB40
 P 10550 1750
-F 0 "J2" H 10630 1746 50  0000 L CNN
+F 0 "J4" H 10630 1746 50  0000 L CNN
 F 1 "Conn_01x01" H 10630 1701 50  0001 L CNN
 F 2 "mech:Faston_6.3x0.8x14" H 10550 1750 50  0001 C CNN
@@
 $EndComp
 $Comp
-L Connector_Generic:Conn_01x01 J3
+L ihouse-rescue:Connector_Generic_Conn_01x01-ihouse-rescue J5
 U 1 1 5BC9AB58
 P 10550 1900
-F 0 "J3" H 10630 1896 50  0000 L CNN
+F 0 "J5" H 10630 1896 50  0000 L CNN
 F 1 "Conn_01x01" H 10630 1851 50  0001 L CNN
 F 2 "mech:Faston_6.3x0.8x14" H 10550 1900 50  0001 C CNN
@@
 $EndComp
 $Comp
-L Connector_Generic:Conn_01x01 J4
+L ihouse-rescue:Connector_Generic_Conn_01x01-ihouse-rescue J6
 U 1 1 5BC9AB72
 P 10550 2050
-F 0 "J4" H 10630 2046 50  0000 L CNN
+F 0 "J6" H 10630 2046 50  0000 L CNN
 F 1 "Conn_01x01" H 10630 2001 50  0001 L CNN
 F 2 "mech:Faston_6.3x0.8x14" H 10550 2050 50  0001 C CNN
@@
 	10250 1600 10250 1750
 Wire Wire Line
-	10250 2050 10350 2050
-Wire Wire Line
-	10350 1900 10250 1900
+	9850 2050 10250 2050
+Wire Wire Line
+	10250 1900 10350 1900
 Connection ~ 10250 1900
 Wire Wire Line
-	10250 1900 10250 2050
-Wire Wire Line
-	10350 1750 10250 1750
+	10250 1750 10350 1750
 Connection ~ 10250 1750
-Wire Wire Line
-	10250 1750 10250 1900
-Wire Wire Line
-	10250 2050 9850 2050
 Connection ~ 10250 2050
 Text Label 9850 2050 0    50   ~ 0
@@
 	6400 4050 6700 4050
 $Comp
-L Connector_Generic:Conn_01x03 J5
+L ihouse-rescue:Connector_Generic_Conn_01x03-ihouse-rescue J7
 U 1 1 5BC74B70
 P 10550 2550
-F 0 "J5" H 10630 2546 50  0000 L CNN
+F 0 "J7" H 10630 2546 50  0000 L CNN
 F 1 "Conn_01x03" H 10630 2501 50  0001 L CNN
 F 2 "Connectors_Phoenix:PhoenixContact_MSTBA-G_03x5.00mm_Angled" H 10550 2550 50  0001 C CNN
@@
 OUTAC7
 $Comp
-L Connector_Generic:Conn_02x12_Counter_Clockwise J?
+L ihouse-rescue:Connector_Generic_Conn_02x12_Counter_Clockwise-ihouse-rescue J1
 U 1 1 5C039156
 P 6050 5850
-AR Path="/5BC77CC5/5C039156" Ref="J?"  Part="1"
-AR Path="/5C039156" Ref="J7"  Part="1"
-F 0 "J7" H 6100 6450 50  0000 C CNN
+F 0 "J1" H 6100 6450 50  0000 C CNN
 F 1 "AC OUTS" H 6100 5150 50  0000 C CNN
 F 2 "Connector_Molex:Molex_Mini-Fit_Jr_5566-24A_2x12_P4.20mm_Vertical" H 6050 5850 50  0001 C CNN
@@
 	6450 5750 6350 5750
 Wire Wire Line
-	6350 5650 6450 5650
+	6450 5650 6350 5650
 Connection ~ 6450 5650
 Wire Wire Line
-	6450 5650 6450 5750
-Wire Wire Line
-	6350 5550 6450 5550
+	6450 5550 6350 5550
 Connection ~ 6450 5550
 Wire Wire Line
-	6450 5550 6450 5650
-Wire Wire Line
-	6350 5450 6450 5450
+	6450 5450 6350 5450
 Connection ~ 6450 5450
-Wire Wire Line
-	6450 5450 6450 5550
-Wire Wire Line
-	6450 5350 6800 5350
 Connection ~ 6450 5350
 Wire Wire Line
@@
 	5850 5950 5450 5950
 Wire Wire Line
-	6350 5950 6450 5950
-Wire Wire Line
-	6450 5950 6450 5850
+	6450 5950 6350 5950
 Connection ~ 6450 5750
 Wire Wire Line
@@
 Connection ~ 6450 5850
 Wire Wire Line
-	6450 5850 6450 5750
-Wire Wire Line
 	7600 5350 7300 5350
 Wire Wire Line
@@
 	8100 5450 8400 5450
 $Comp
-L Connector_Generic:Conn_02x02_Counter_Clockwise J?
+L ihouse-rescue:Connector_Generic_Conn_02x02_Counter_Clockwise-ihouse-rescue J2
 U 1 1 5C03917E
 P 7800 5350
-AR Path="/5BC77CC5/5C03917E" Ref="J?"  Part="1"
-AR Path="/5C03917E" Ref="J6"  Part="1"
-F 0 "J6" H 7850 5450 50  0000 C CNN
+F 0 "J2" H 7850 5450 50  0000 C CNN
 F 1 "AC INPUTS" H 7850 5150 50  0000 C CNN
 F 2 "Connector_Molex:Molex_Mini-Fit_Jr_5566-04A_2x02_P4.20mm_Vertical" H 7800 5350 50  0001 C CNN
@@
 INACN2
 Wire Wire Line
-	6350 6050 6450 6050
-Wire Wire Line
-	6450 6050 6450 5950
+	6450 6050 6350 6050
 Connection ~ 6450 5950
 Wire Wire Line
@@
 OUTAC9
 Wire Wire Line
-	6350 6150 6450 6150
+	6450 6150 6350 6150
 Wire Wire Line
 	5850 6350 5450 6350
@@
 Text Label 6800 6250 2    50   ~ 0
 OUTAC10N
-Wire Wire Line
-	6450 6150 6450 6050
 Connection ~ 6450 6050
 Text Notes 7300 6000 0    50   ~ 0
@@
 INACN2
 Wire Wire Line
-	6500 1500 6500 2150
-Wire Wire Line
-	7300 1600 6600 1600
+	6600 1600 7300 1600
 Connection ~ 6600 1600
-Wire Wire Line
-	6600 1600 6600 1350
 $Sheet
 S 6700 2050 1200 2400
@@
 F1 "dc_valve_control.sch" 50
 $EndSheet
+Wire Wire Line
+	6500 2150 6700 2150
+Wire Wire Line
+	6600 2250 6700 2250
+Wire Wire Line
+	6500 1500 6500 2150
+Wire Wire Line
+	10250 1900 10250 2050
+Wire Wire Line
+	10250 1750 10250 1900
+Wire Wire Line
+	10250 2050 10350 2050
+Wire Wire Line
+	6450 5650 6450 5750
+Wire Wire Line
+	6450 5550 6450 5650
+Wire Wire Line
+	6450 5450 6450 5550
+Wire Wire Line
+	6450 5350 6800 5350
+Wire Wire Line
+	6450 5750 6450 5850
+Wire Wire Line
+	6450 5850 6450 5950
+Wire Wire Line
+	6450 5950 6450 6050
+Wire Wire Line
+	6450 6050 6450 6150
+Wire Wire Line
+	6600 1600 6600 2250
 $EndSCHEMATC

Commit message: tarpinis kommitas
Changed lines of the file:
@@
 $Descr A4 11693 8268
 encoding utf-8
-Sheet 1 4
+Sheet 1 5
 Title ""
 Date ""
@@
 Wire Wire Line
 	6600 1600 6600 2250
+$Sheet
+S 2000 2800 1750 1300
+U 5C3058F0
+F0 "DC sklendziu valdymas L293" 50
+F1 "dc_valve_control_L293.sch" 50
+$EndSheet
 $EndSCHEMATC

Commit message: tarpinis kommitas
Parts:
- added C?: 100uFx16V, Capacitors_SMD:CP_Elec_6.3x5.7, symbol ihouse-rescue:capacitors_CP_100uFx16V-ihouse-rescue
- added D? (x2): LL4148, Diode_SMD:D_MiniMELF, symbol ihouse-rescue:Diode_LL4148-ihouse-rescue
- added D? (x10): Z0103MN, Package_TO_SOT_SMD:SOT-223, symbol ihouse-rescue:Triac_Thyristor_Z0103MN-ihouse-rescue
- added F?: 3A, Fuse:Fuseholder_Cylinder-5x20mm_Schurter_0031_8201_Horizontal_Open, symbol ihouse-rescue:Device_Fuse-ihouse-rescue
- added J?: EXT2, symbol ihouse-rescue:Connector_Screw_Terminal_01x03-ihouse-rescue
- added J?: EXT3, symbol ihouse-rescue:Connector_Screw_Terminal_01x03-ihouse-rescue
- added J?: EXT4, symbol ihouse-rescue:Connector_Screw_Terminal_01x03-ihouse-rescue
- added J?: EXT1, symbol ihouse-rescue:Connector_Screw_Terminal_01x03-ihouse-rescue
- added K1: FINDER-34.51, symbol ihouse-rescue:Relay_FINDER-40.51-ihouse-rescue
- added K2: RT42xxxx, Relay_THT:Relay_DPDT_Schrack-RT2-FormC_RM5mm, symbol ihouse-rescue:Relay_RT42xxxx-ihouse-rescue
- added K3, K4, K5, K6: FINDER-34.51, Relays_THT:Relay_SPDT_SingleRow_Standing_FinderType34Point51, symbol ihouse-rescue:Relay_FINDER-40.51-ihouse-rescue
- added K? (x2): FINDER-32.21-x300, Relay_THT:Relay_SPST_Schrack-RT1-FormA_RM5mm, symbol ihouse-rescue:Relay_FINDER-32.21-x300-ihouse-rescue
- added K?: G5Q-1A, Relay_THT:Relay_SPDT_Finder_34.51_Vertical, symbol ihouse-rescue:Relay_G5Q-1A-ihouse-rescue
- added M?: unicon_v1, unicon:unicon_v1, symbol unicon:unicon_v1
- added R? (x21): R, Resistor_SMD:R_0805_2012Metric_Pad1.15x1.40mm_HandSolder, symbol ihouse-rescue:Device_R-ihouse-rescue
- added R?: 1k, Resistor_SMD:R_0805_2012Metric_Pad1.15x1.40mm_HandSolder, symbol ihouse-rescue:Device_R-ihouse-rescue
- added R?: 120, Resistor_SMD:R_0805_2012Metric_Pad1.15x1.40mm_HandSolder, symbol ihouse-rescue:Device_R-ihouse-rescue
- added R? (x2): Rx, Resistor_SMD:R_0805_2012Metric_Pad1.15x1.40mm_HandSolder, symbol ihouse-rescue:Device_R-ihouse-rescue
- added R? (x8): 33k, Resistor_SMD:R_1206_3216Metric_Pad1.42x1.75mm_HandSolder, symbol ihouse-rescue:Device_R-ihouse-rescue
- added T?: Transformer_TEZ_22x24_6V, Transformer_THT:Transformer_Breve_TEZ-22x24, symbol ihouse-rescue:disc_Transformer_TEZ_22x24_6V-ihouse-rescue
- added TH?: 230V/150mA, symbol ihouse-rescue:Device_Thermistor_PTC-ihouse-rescue
- added U? (x10): MOC3060S, disc:DIP-6_W9.53mm_SMD, symbol ihouse-rescue:disc_MOC3060S-ihouse-rescue
- added U? (x2): LTV-817, Package_DIP:DIP-4_W7.62mm, symbol ihouse-rescue:Isolator_LTV-817-ihouse-rescue
- added U?: ULN2803A, symbol ihouse-rescue:Transistor_Array_ULN2803A-ihouse-rescue
- renumbered J7 to J?, J3 to J?, J4 to J?, J5 to J?, J6 to J?, J1 to J?, J2 to J?
Connections:
- net 230VAC_L: no longer J?.11 (Pin_11), J?.12 (Pin_12)
- net 230VAC_N: no longer J?.13 (Pin_13), J?.14 (Pin_14)
- net ACN: now also K1.11
- net INACL1: now also K?.A1
- net INACL2: now also K?.A1
- net INACN1: now also K?.A2
- net INACN2: now also K?.A2
- net OUTAC1: now also D?.1 (A1), R?.2, U?.4
- net OUTAC10: now also K2.21
- net OUTAC10N: now also K2.11
- net OUTAC2: now also D?.1 (A1), R?.2, U?.4
- net OUTAC3: now also D?.1 (A1), R?.2, U?.4
- net OUTAC4: now also D?.1 (A1), R?.2, U?.4
- net OUTAC5: now also D?.1 (A1), R?.2, U?.4
- net OUTAC6: now also D?.1 (A1), K?.2, R?.2, U?.4
- net OUTAC7: now also D?.1 (A1), R?.2, U?.4
- net OUTAC8: now also D?.1 (A1), R?.2, U?.4
- net OUTAC9: now also D?.1 (A1), D?.1 (A1), K?.11, K?.14, R?.1, R?.2, R?.2, U?.4, U?.4
- new net: R?.1, U?.1
- new net: R?.2, U?.6 (x10)
- new net: D?.1 (K), R?.2, U?.1 (x2)
- new net: D?.2 (A), R?.2, U?.2 (x2)
- new net: R?.1, T?.6 (SB)
- new net: C?.1, R?.1, R?.2, R?.2, T?.7 (SA)
- new net: R?.1, T?.1 (AA), TH?.2
- new net: D?.3 (G), R?.1 (x10)
- new net: R?.1, R?.2 (x4)
- new net 12VDC: K1.A1, K2.A1, K3.A1, K4.A1, K5.A1, K6.A1, K?.5, M?.1 (12VDC), R?.2, U?.10 (COM)
- new net 230L: F?.2, K2.24, TH?.1
- new net 230N: K1.14, K2.14, R?.1, T?.4 (AB)
- new net 5VDC: M?.2 (5VDC)
- new net ACL: D?.2 (A2), D?.2 (A2), D?.2 (A2), D?.2 (A2), D?.2 (A2), D?.2 (A2), D?.2 (A2), D?.2 (A2), D?.2 (A2), D?.2 (A2), D?.4 (A4), D?.4 (A4), D?.4 (A4), D?.4 (A4), D?.4 (A4), D?.4 (A4), D?.4 (A4), D?.4 (A4), D?.4 (A4), D?.4 (A4), F?.1, K?.11, K?.14, K?.3, R?.1, R?.1, R?.1, R?.1, R?.1, R?.1, R?.1, R?.1, R?.1, R?.1, R?.1
- new net AIN: R?.1, R?.2
- new net COM: C?.2, M?.28 (COM), M?.4 (COM), M?.5 (COM), M?.6 (COM), R?.2, U?.3, U?.3, U?.9 (GND)
- new net EXT0: U?.1 (I1)
- new net EXT1: U?.3 (I3)
- new net EXT1_11: J?.2 (Pin_2), K3.11
- new net EXT1_12: J?.3 (Pin_3), K3.12
- new net EXT1_14: J?.1 (Pin_1), K3.14
- new net EXT2: U?.4 (I4)
- new net EXT2_11: J?.2 (Pin_2), K5.11
- new net EXT2_12: J?.3 (Pin_3), K5.12
- new net EXT2_14: J?.1 (Pin_1), K5.14
- new net EXT3: U?.5 (I5)
- new net EXT3_11: J?.2 (Pin_2), K4.11
- new net EXT3_12: J?.3 (Pin_3), K4.12
- new net EXT3_14: J?.1 (Pin_1), K4.14
- new net EXT4: U?.6 (I6)
- new net EXT4_11: J?.2 (Pin_2), K6.11
- new net EXT4_12: J?.3 (Pin_3), K6.12
- new net EXT4_14: J?.1 (Pin_1), K6.14
- new net K1: K1.A2, U?.18 (O1)
- new net K2: K2.A2, U?.17 (O2)
- new net K3: K3.A2, K?.1, U?.16 (O3)
- new net K4: K4.A2, U?.15 (O4)
- new net K5: K5.A2, U?.14 (O5)
- new net K6: K6.A2, U?.13 (O6)
- new net LIGHTON: U?.4
- new net LPULSE: U?.4
- new net MCP23017 extended port/EO0: U?.2
- new net MCP23017 extended port/EO1: U?.2
- new net MCP23017 extended port/EO2: U?.2
- new net MCP23017 extended port/EO3: U?.2
- new net MCP23017 extended port/EO4: U?.2
- new net MCP23017 extended port/EO5: U?.2
- new net MCP23017 extended port/EO6: U?.2
- new net MCP23017 extended port/EO7: U?.2
- new net MCP23017 extended port/EO8: U?.2
- new net MCP23017 extended port/EO9: U?.2 (I2)
- new net MCP23017 extended port/OC5V: U?.1, U?.1, U?.1, U?.1, U?.1, U?.1, U?.1, U?.1, U?.1
- new net OC1: U?.2
- new net OUTAC11: J?.11 (Pin_11)
- new net OUTAC11N: J?.14 (Pin_14)
- new net OUTAC12: J?.12 (Pin_12)
- new net OUTAC12N: J?.13 (Pin_13)
- new net VREF: R?.1
Other:
- moved on the sheet: J?

Commit message: sukurtas embitz proektas
Parts:
- M?: symbol unicon:unicon_v1 -> ihouse-rescue:unicon_v1-unicon
Connections:
- net AIN is gone; now on net VLINE: R?.1, R?.2
- net VREF is gone; now on net 3VDC: R?.1
- net LPULSE: now also M?.35 (PF6)
- net SCL: now also M?.10 (PB6)
- net SDA: now also M?.11 (PB7)
- net BUZZ: now reaches M?.13 (PB9)
- net VLINE: now reaches M?.19 (PA0)
- net 3VDC: now reaches M?.3 (3VDC)
- net UART_DE: now reaches M?.38 (PA12)
- net UART_TX: now reaches M?.39 (PA9)
- net UART_RX: now reaches M?.40 (PA10)
Changed lines of the file:
@@
 	1750 9800 1450 9800
 Text Label 1450 9400 0    50   ~ 0
-AIN
+VLINE
 Text Label 1450 9800 0    50   ~ 0
-VREF
+3VDC
 $Comp
 L ihouse-rescue:capacitors_CP_100uFx16V-ihouse-rescue C?
@@
 COM
 $Comp
-L unicon:unicon_v1 M?
+L ihouse-rescue:unicon_v1-unicon M?
 U 1 1 5C94CB7C
 P 3200 3250
@@
 $EndComp
 Wire Wire Line
-	2250 2200 1950 2200
-Text Label 1950 2200 0    50   ~ 0
+	2250 2200 1900 2200
+Text Label 1900 2200 0    50   ~ 0
 5VDC
 Wire Wire Line
-	2250 2100 1950 2100
-Text Label 1950 2100 0    50   ~ 0
+	2250 2100 1900 2100
+Text Label 1900 2100 0    50   ~ 0
 12VDC
 Wire Wire Line
@@
 	2150 2500 2150 2600
 Wire Wire Line
-	2150 2600 1950 2600
+	2150 2600 1900 2600
 Connection ~ 2150 2600
-Text Label 1950 2600 0    50   ~ 0
+Text Label 1900 2600 0    50   ~ 0
 COM
 Wire Wire Line
@@
 Text Label 9100 3700 0    50   ~ 0
 EXT0
+Wire Wire Line
+	2250 2900 1900 2900
+Wire Wire Line
+	2250 3000 1900 3000
+Text Label 1900 3000 0    50   ~ 0
+SDA
+Text Label 1900 2900 0    50   ~ 0
+SCL
+Wire Wire Line
+	4150 3800 4500 3800
+Wire Wire Line
+	4150 3900 4500 3900
+Text Label 4500 3800 2    50   ~ 0
+UART_TX
+Text Label 4500 3900 2    50   ~ 0
+UART_RX
+Wire Wire Line
+	4150 3700 4500 3700
+Text Label 4500 3700 2    50   ~ 0
+UART_DE
+Wire Wire Line
+	2250 3200 1900 3200
+Text Label 1900 3200 0    50   ~ 0
+BUZZ
+Wire Wire Line
+	4150 3400 4500 3400
+Text Label 4500 3400 2    50   ~ 0
+LPULSE
+Wire Wire Line
+	2250 3800 1900 3800
+Text Label 1900 3800 0    50   ~ 0
+VLINE
+Wire Wire Line
+	1900 2300 2250 2300
+Text Label 1900 2300 0    50   ~ 0
+3VDC
 $EndSCHEMATC
