File: ihouse.sch (KiCad schematic (older format))
At the start: 83 parts, among them K1 FINDER-34.51, K2 RT42xxxx, K3 FINDER-34.51, K4 FINDER-34.51, K5 FINDER-34.51, K6 FINDER-34.51

Commit message: tarpinis kommitas
Connections:
- net BUZZ: now also M?.17 (PA6); no longer M?.13 (PB9)
- net OPTIC: now reaches M?.15 (PA4)
- net PWM2: now reaches M?.41 (PB15)
- net PWM1: now reaches M?.44 (PB14)
Changed lines of the file:
@@
 Text Label 4500 3700 2    50   ~ 0
 UART_DE
-Wire Wire Line
-	2250 3200 1900 3200
-Text Label 1900 3200 0    50   ~ 0
+Text Label 1900 3600 0    50   ~ 0
 BUZZ
 Wire Wire Line
@@
 Text Label 1900 2300 0    50   ~ 0
 3VDC
+Text Label 1900 3400 0    50   ~ 0
+OPTIC
+Wire Wire Line
+	2250 3400 1900 3400
+Wire Wire Line
+	2250 3600 1900 3600
+Wire Wire Line
+	4150 4300 4500 4300
+Wire Wire Line
+	4150 4000 4500 4000
+Text Label 4500 4300 2    50   ~ 0
+PWM1
+Text Label 4500 4000 2    50   ~ 0
+PWM2
 $EndSCHEMATC

Commit message: tarpinis kommitas
Connections:
- net UART2_DE: now reaches M?.20 (PA1)
- net UART2_TX: now reaches M?.21 (PA2)
- net UART2_RX: now reaches M?.22 (PA3)
Changed lines of the file:
@@
 Text Label 4500 4000 2    50   ~ 0
 PWM2
+Wire Wire Line
+	2250 4000 1900 4000
+Text Label 1900 4000 0    50   ~ 0
+UART2_TX
+Wire Wire Line
+	2250 4100 1900 4100
+Text Label 1900 4100 0    50   ~ 0
+UART2_RX
+Wire Wire Line
+	2250 3900 1900 3900
+Text Label 1900 3900 0    50   ~ 0
+UART2_DE
 $EndSCHEMATC
