File: Kicad/ihouse.kicad_pcb (KiCad board)
At the start: 2 copper layers, 30 x 31 mm, 61 parts, among them J10 Conn_01x01, J11 Conn_01x01, J12 Conn_01x03, J13 Valves, J14 Conn_01x01, J15 Conn_01x08, J16 Conn_01x01, J17 Conn_01x01, J18 Conn_01x01, J8 Conn_01x01, J9 Conn_01x01, K3 FINDER-34.51, K4 FINDER-34.51, K5 FINDER-34.51, K6 FINDER-34.51, U1 MOC3060S, U10 MOC3060S, U11 MOC3060S, U12 MOC3060S, U17 St232C, U18 ST232C, U3 MOC3060S, U4 MOC3060S, U5 MOC3060S, U7 MOC3060S, U8 MOC3060S, U9 MOC3060S

Commit message: tarpinis kommitas
Parts:
- added C13: 0.1, Capacitors_SMD:C_0805_HandSoldering, F.Cu at (105.3, 96.0)
- added J1: UART2, Connectors:RJ45_8, F.Cu at (100.0, 61.0)
- added J19: EV1527, Pin_Headers:Pin_Header_Straight_1x07_Pitch2.54mm, F.Cu at (100.9, 0.10)
- added J20: Valves, Connectors_Molex:Molex_MiniFit-JR-5556-10A_2x05x4.20mm_Straight, F.Cu at (55.5, -18.4)
- added J3: AC OUTS, Connectors_Molex:Molex_MiniFit-JR-5556-24A_2x12x4.20mm_Straight, F.Cu at (225.9, 88.2)
- added K1: FINDER-34.51, Relays_THT:Relay_DPST_Schrack-RT2-FormA_RM5mm, F.Cu at (183.3, 61.3)
- added K2: RT42xxxx, Relays_THT:Relay_DPDT_Finder_40.52, F.Cu at (183.3, 74.6)
- added R49: 2k, Resistors_SMD:R_0805_HandSoldering, F.Cu at (108.3, 53.2)
- added U14: MCP23017, digikey-footprints:SOIC-28_W7.5mm, F.Cu at (102.2, 88.6)
- added U19: MCP23017, digikey-footprints:SOIC-28_W7.5mm, F.Cu at (121.9, 88.6)
- C2, C3: footprint Capacitors_SMD:C_0805 -> Capacitors_SMD:C_0805_HandSoldering
- D13: value D -> BAS32
- J13: value Valves -> UART1; footprint Connectors_Molex:Molex_MiniFit-JR-5556-10A_2x05x4.20mm_Straight -> Pin_Headers:Pin_Header_Straight_1x05_Pitch2.54mm
- R34: value R -> 15k; footprint Resistors_SMD:R_0805 -> Resistors_SMD:R_0805_HandSoldering
- R35, R36, R37: value R -> 1k; footprint Resistors_SMD:R_0805 -> Resistors_SMD:R_0805_HandSoldering
- TH2: value 500mA -> 1210L005WR
- moved C3 164.0 mm to (134.6, 85.2)
- moved R34 161.5 mm to (134.6, 90.0), turned to 180 degrees
- moved C2 159.6 mm to (125.0, 96.0)
- moved R36 158.7 mm to (134.6, 93.8)
- moved R37 156.8 mm to (134.6, 82.9), turned to 180 degrees
- moved R35 155.1 mm to (134.6, 91.9)
- moved D13 146.7 mm to (134.7, 87.7), turned to 180 degrees
- moved K5 118.7 mm to (188.2, 53.8), turned to 180 degrees
- moved K3 115.3 mm to (188.2, 38.2), turned to 180 degrees
- moved K4 113.7 mm to (188.2, 43.4), turned to 180 degrees
- moved K6 112.2 mm to (188.2, 48.6), turned to 180 degrees
- moved J13 96.4 mm to (110.6, 3.70)
- moved C6 88.6 mm to (107.1, 61.4), turned to 180 degrees
- moved C11 87.8 mm to (107.1, 63.9)
- moved TH2 82.2 mm to (109.3, 69.9), turned to 180 degrees
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Connections:
- D18 pad 1: (no net) -> /RS232 interfeisas/RSCNTRL
- D18 pad 2: (no net) -> Net-(D18-Pad2)
- J13 pad 4: (no net) -> /COM
- J13 pad 5: (no net) -> /5VDC
- R35 pad 1: (no net) -> /SCL
- R36 pad 1: (no net) -> /SDA
- R37 pad 1: /MCP23017 extended port/EO0 -> /5VDC
- R37 pad 2: /MCP23017 extended port/EO0 -> Net-(R37-Pad2)
- TH2 pad 2: (no net) -> /RS232 interfeisas/RS5VDC
- U10 pad 1: /5VDC -> Net-(U10-Pad1)
- U10 pad 2: /MCP23017 extended port/EO6 -> (no net)
- U10 pad 4: (no net) -> /OUTAC7
- U11 pad 1: /5VDC -> Net-(U10-Pad1)
- U11 pad 2: /MCP23017 extended port/EO7 -> (no net)
- U11 pad 4: (no net) -> /OUTAC8
- U12 pad 1: /5VDC -> Net-(U10-Pad1)
- U12 pad 2: /MCP23017 extended port/EO8 -> (no net)
- U18 pad 7: (no net) -> /RS232 interfeisas/RSTX
- U18 pad 8: (no net) -> /RS232 interfeisas/RSRX
- U3 pad 1: /5VDC -> Net-(U10-Pad1)
- U3 pad 2: /MCP23017 extended port/EO0 -> (no net)
- U3 pad 4: (no net) -> /OUTAC1
- U4 pad 1: /5VDC -> Net-(U10-Pad1)
- U4 pad 2: /MCP23017 extended port/EO1 -> (no net)
- U4 pad 4: (no net) -> /OUTAC2
- U5 pad 1: /5VDC -> Net-(U10-Pad1)
- U5 pad 2: /MCP23017 extended port/EO2 -> (no net)
- U5 pad 4: (no net) -> /OUTAC3
- U7 pad 1: /5VDC -> Net-(U10-Pad1)
- U7 pad 2: /MCP23017 extended port/EO3 -> (no net)
- U7 pad 4: (no net) -> /OUTAC4
- U8 pad 1: /5VDC -> Net-(U10-Pad1)
- U8 pad 2: /MCP23017 extended port/EO4 -> (no net)
- U8 pad 4: (no net) -> /OUTAC5
- U9 pad 1: /5VDC -> Net-(U10-Pad1)
- U9 pad 2: /MCP23017 extended port/EO5 -> (no net)
- U9 pad 4: (no net) -> /OUTAC6
Other:
- board size 30 x 31 mm -> 188 x 80 mm

Commit message: schemos paruosimas
Parts:
- removed J10: Conn_01x01, mech:Faston_6.3x0.8x14
- removed R45, R46: R, Resistors_SMD:R_0805
- added C14: CP, Capacitor_SMD:CP_Elec_10x7.9, F.Cu at (-77.3, 72.8)
- added C15: CP, Capacitor_SMD:CP_Elec_10x7.9, F.Cu at (-77.3, 91.8)
- added D1: LL4148, Diode_SMD:D_MiniMELF, F.Cu at (67.0, 98.2)
- added D10: Z0103MN, Package_TO_SOT_SMD:SOT-223, F.Cu at (338.0, 78.0)
- added D11: Z0103MN, Package_TO_SOT_SMD:SOT-223, F.Cu at (338.0, 158.0)
- added D12: LL4148, Diode_SMD:D_MiniMELF, F.Cu at (67.0, 91.2)
- added D19: LL4004, Diode_SMD:D_MELF, F.Cu at (-75.3, 100.8)
- added D2: LL4148, Diode_SMD:D_MiniMELF, F.Cu at (67.0, 104.8)
- added D20: LL4004, Diode_SMD:D_MELF, F.Cu at (-75.3, 63.8)
- added D3: Z0103MN, Package_TO_SOT_SMD:SOT-223, F.Cu at (338.0, 148.0)
- added D4: Z0103MN, Package_TO_SOT_SMD:SOT-223, F.Cu at (338.0, 138.0)
- added D5: Z0103MN, Package_TO_SOT_SMD:SOT-223, F.Cu at (338.0, 128.0)
- added D6: Z0103MN, Package_TO_SOT_SMD:SOT-223, F.Cu at (338.0, 118.0)
- added D7: Z0103MN, Package_TO_SOT_SMD:SOT-223, F.Cu at (338.0, 108.0)
- added D8: Z0103MN, Package_TO_SOT_SMD:SOT-223, F.Cu at (338.0, 98.0)
- added D9: Z0103MN, Package_TO_SOT_SMD:SOT-223, F.Cu at (338.0, 88.0)
- added F1: 0.5A, Fuse:Fuseholder_Cylinder-5x20mm_Schurter_0031_8201_Horizontal_Open, F.Cu at (67.0, 36.0)
- added J2: AC Inputs, Connector_Molex:Molex_Mini-Fit_Jr_5566-04A_2x02_P4.20mm_Vertical, F.Cu at (40.0, 103.0)
- added J21: Valve2, Connectors_Molex:Molex_KK-6410-02_02x2.54mm_Straight, F.Cu at (205.8, 36.8)
- added J22: Valve3, Connectors_Molex:Molex_KK-6410-02_02x2.54mm_Straight, F.Cu at (174.1, 32.9)
- added J23: Valve4, Connectors_Molex:Molex_KK-6410-02_02x2.54mm_Straight, F.Cu at (174.1, 39.3)
- added J4: EXT1, Connectors_Terminal_Blocks:TerminalBlock_bornier-3_P5.08mm, F.Cu at (245.1, 105.6)
- added J5: EXT2, Connectors_Terminal_Blocks:TerminalBlock_bornier-3_P5.08mm, F.Cu at (197.1, 105.6)
- added J6: EXT3, Connectors_Terminal_Blocks:TerminalBlock_bornier-3_P5.08mm, F.Cu at (229.1, 105.6)
- added J7: EXT4, Connectors_Terminal_Blocks:TerminalBlock_bornier-3_P5.08mm, F.Cu at (213.1, 105.6)
- added M1: unicon_v1, unicon:unicon_v1, F.Cu at (176.2, 78.8)
- added R1: 33k, Resistor_SMD:R_1206_3216Metric_Pad1.42x1.75mm_HandSolder, F.Cu at (63.0, 96.5)
- added R10: R, Resistor_SMD:R_0805_2012Metric_Pad1.15x1.40mm_HandSolder, F.Cu at (332.0, 135.0)
- added R11: R, Resistor_SMD:R_0805_2012Metric_Pad1.15x1.40mm_HandSolder, F.Cu at (343.0, 140.0)
- added R12: R, Resistor_SMD:R_0805_2012Metric_Pad1.15x1.40mm_HandSolder, F.Cu at (332.0, 125.0)
- added R13: R, Resistor_SMD:R_0805_2012Metric_Pad1.15x1.40mm_HandSolder, F.Cu at (343.0, 130.0)
- added R14: R, Resistor_SMD:R_0805_2012Metric_Pad1.15x1.40mm_HandSolder, F.Cu at (332.0, 115.0)
- added R15: R, Resistor_SMD:R_0805_2012Metric_Pad1.15x1.40mm_HandSolder, F.Cu at (343.0, 120.0)
- added R16: R, Resistor_SMD:R_0805_2012Metric_Pad1.15x1.40mm_HandSolder, F.Cu at (332.0, 105.0)
- added R17: R, Resistor_SMD:R_0805_2012Metric_Pad1.15x1.40mm_HandSolder, F.Cu at (343.0, 110.0)
- added R18: R, Resistor_SMD:R_0805_2012Metric_Pad1.15x1.40mm_HandSolder, F.Cu at (332.0, 95.0)
- added R19: R, Resistor_SMD:R_0805_2012Metric_Pad1.15x1.40mm_HandSolder, F.Cu at (343.0, 100.0)
- added R2: 33k, Resistor_SMD:R_1206_3216Metric_Pad1.42x1.75mm_HandSolder, F.Cu at (63.0, 100.0)
- added R20: R, Resistor_SMD:R_0805_2012Metric_Pad1.15x1.40mm_HandSolder, F.Cu at (332.0, 84.0)
- added R21: R, Resistor_SMD:R_0805_2012Metric_Pad1.15x1.40mm_HandSolder, F.Cu at (343.0, 90.0)
- added R22: R, Resistor_SMD:R_0805_2012Metric_Pad1.15x1.40mm_HandSolder, F.Cu at (332.0, 75.0)
- added R23: R, Resistor_SMD:R_0805_2012Metric_Pad1.15x1.40mm_HandSolder, F.Cu at (343.0, 80.0)
- added R24: R, Resistor_SMD:R_0805_2012Metric_Pad1.15x1.40mm_HandSolder, F.Cu at (332.0, 155.0)
- added R25: R, Resistor_SMD:R_0805_2012Metric_Pad1.15x1.40mm_HandSolder, F.Cu at (343.0, 160.0)
- added R26: 33k, Resistor_SMD:R_1206_3216Metric_Pad1.42x1.75mm_HandSolder, F.Cu at (63.0, 89.5)
- added R27: 33k, Resistor_SMD:R_1206_3216Metric_Pad1.42x1.75mm_HandSolder, F.Cu at (58.0, 89.5)
- added R28: 33k, Resistor_SMD:R_1206_3216Metric_Pad1.42x1.75mm_HandSolder, F.Cu at (63.0, 93.0)
- added R29: 33k, Resistor_SMD:R_1206_3216Metric_Pad1.42x1.75mm_HandSolder, F.Cu at (58.0, 93.0)
- added R3: 33k, Resistor_SMD:R_1206_3216Metric_Pad1.42x1.75mm_HandSolder, F.Cu at (63.0, 103.0)
- added R30: 1k, Resistor_SMD:R_0805_2012Metric_Pad1.15x1.40mm_HandSolder, F.Cu at (58.0, 84.0)
- added R31: 120, Resistor_SMD:R_0805_2012Metric_Pad1.15x1.40mm_HandSolder, F.Cu at (60.0, 81.0)
- added R32: Rx, Resistor_SMD:R_0805_2012Metric_Pad1.15x1.40mm_HandSolder, F.Cu at (62.0, 84.0)
- added R33: Rx, Resistor_SMD:R_0805_2012Metric_Pad1.15x1.40mm_HandSolder, F.Cu at (64.0, 81.0)
- added R4: 33k, Resistor_SMD:R_1206_3216Metric_Pad1.42x1.75mm_HandSolder, F.Cu at (63.0, 106.5)
- added R5: 33k, Resistor_SMD:R_1206_3216Metric_Pad1.42x1.75mm_HandSolder, F.Cu at (58.0, 96.5)
- added R50: 1k, Resistor_SMD:R_0805_2012Metric_Pad1.15x1.40mm_HandSolder, F.Cu at (147.0, 27.0)
- added R52: 1k, Resistor_SMD:R_0805_2012Metric_Pad1.15x1.40mm_HandSolder, F.Cu at (166.0, 38.0)
- added R54: 1k, Resistor_SMD:R_0805_2012Metric_Pad1.15x1.40mm_HandSolder, F.Cu at (166.0, 40.0)
- added R6: 33k, Resistor_SMD:R_1206_3216Metric_Pad1.42x1.75mm_HandSolder, F.Cu at (58.0, 100.0)
- added R7: 33k, Resistor_SMD:R_1206_3216Metric_Pad1.42x1.75mm_HandSolder, F.Cu at (58.0, 103.0)
- added R8: R, Resistor_SMD:R_0805_2012Metric_Pad1.15x1.40mm_HandSolder, F.Cu at (332.0, 145.0)
- added R9: R, Resistor_SMD:R_0805_2012Metric_Pad1.15x1.40mm_HandSolder, F.Cu at (343.0, 150.0)
- added REF**: MountingHole_3.2mm_M3, MountingHole:MountingHole_3.2mm_M3, F.Cu at (33.0, 106.0)
- added REF**: MountingHole_3.2mm_M3, MountingHole:MountingHole_3.2mm_M3, F.Cu at (83.0, 106.0)
- added REF**: MountingHole_3.2mm_M3, MountingHole:MountingHole_3.2mm_M3, F.Cu at (83.0, 26.0)
- added REF**: MountingHole_3.2mm_M3, MountingHole:MountingHole_3.2mm_M3, F.Cu at (33.0, 26.0)
- added TH3: 1.5A/30V, Resistor_SMD:R_1210_3225Metric, F.Cu at (-78.3, 82.2)
- added TH4: 0.5A/230V, Varistor:RV_Disc_D7mm_W3.4mm_P5mm, F.Cu at (35.0, 90.0)
- added TR1: TSZZ20-006M_1, Transformer_THT:Transformer_Breve_TEZ-47x57_1, F.Cu at (-92.0, 66.0)
- added TR2: Transformer_TEZ_22x24_6V, Transformers_THT:Transformer_Breve_TEZ-22x24, F.Cu at (35.0, 67.0)
- added U13: LTV-817, Package_DIP:DIP-4_W7.62mm, F.Cu at (70.0, 90.0)
- added U15: L293D, Housings_DIP:DIP-16_W7.62mm_LongPads, F.Cu at (191.7, 27.3)
- added U16: L293D, Housings_DIP:DIP-16_W7.62mm_LongPads, F.Cu at (180.4, 27.3)
- added U2: LTV-817, Package_DIP:DIP-4_W7.62mm, F.Cu at (70.0, 103.5)
- J11: value Conn_01x01 -> To AC/DC; footprint mech:Faston_6.3x0.8x14 -> Connector_Phoenix_MSTB:PhoenixContact_MSTBVA_2,5_2-G_1x02_P5.00mm_Vertical
- J12: footprint Connectors_Phoenix:PhoenixContact_MSTBA-G_03x5.00mm_Angled -> Connector_Phoenix_MSTB:PhoenixContact_MSTBVA_2,5_3-G_1x03_P5.00mm_Vertical
- J20: value Valves -> Valve1; footprint Connectors_Molex:Molex_MiniFit-JR-5556-10A_2x05x4.20mm_Straight -> Connectors_Molex:Molex_KK-6410-02_02x2.54mm_Straight
- K1: footprint Relays_THT:Relay_DPST_Schrack-RT2-FormA_RM5mm -> Relay_THT:Relay_SPDT_Finder_34.51_Vertical
- K3, K4, K5, K6: footprint Relays_THT:Relay_SPDT_SingleRow_Standing_FinderType34Point51 -> Relay_THT:Relay_SPDT_Finder_34.51_Vertical
- R38, R39, R40, R41, R42, R43, R44: value R -> 33k; footprint Resistors_SMD:R_0805 -> Resistor_SMD:R_1206_3216Metric_Pad1.42x1.75mm_HandSolder
- U1: value MOC3060S -> LTV-817; footprint disc:DIP-6_W9.53mm_SMD -> Package_DIP:DIP-4_W7.62mm
- moved U12 289.2 mm to (323.0, 158.0)
- moved U3 250.7 mm to (323.0, 148.0)
- moved U4 249.4 mm to (323.0, 138.0)
- moved U5 245.2 mm to (323.0, 128.0)
- moved U10 242.6 mm to (323.0, 88.0)
- moved U7 239.1 mm to (323.0, 118.0)
- moved U8 238.0 mm to (323.0, 108.0)
- moved U9 237.3 mm to (323.0, 98.0)
- moved U11 231.1 mm to (323.0, 78.0)
- moved R40 219.3 mm to (53.0, 100.0)
- moved R38 207.5 mm to (58.0, 106.5)
- moved R42 206.6 mm to (53.0, 106.5)
- moved R41 206.1 mm to (53.0, 103.0)
- moved R39 205.1 mm to (53.0, 96.5)
- moved R43 197.9 mm to (53.0, 89.5)
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Connections:
- C1 pad 1: (no net) -> Net-(C1-Pad1)
- C10 pad 2: /COM -> /RS232 interfeisas/NEX_COM
- C12 pad 1: /COM -> /RS232 interfeisas/NEX_COM
- C12 pad 2: /5VDC -> /RS232 interfeisas/NEX_5VDC
- C8 pad 2: /5VDC -> /RS232 interfeisas/NEX_5VDC
- J11 pad 1: /PE -> Net-(F1-Pad2)
- J12 pad 1: (no net) -> /ACN
- J12 pad 2: (no net) -> Net-(F1-Pad2)
- J13 pad 1: (no net) -> /UART_DE
- J13 pad 2: (no net) -> /UART_RX
- J13 pad 3: (no net) -> /UART_TX
- J14 pad 1: /5VDC -> /RS232 interfeisas/NEX_5VDC
- J15 pad 1: /5VDC -> /RS232 interfeisas/NEX_5VDC
- J15 pad 2: /COM -> /RS232 interfeisas/NEX_COM
- J15 pad 3: /COM -> /RS232 interfeisas/NEX_COM
- J15 pad 5: /COM -> /RS232 interfeisas/NEX_COM
- J15 pad 7: /COM -> /RS232 interfeisas/NEX_COM
- J15 pad 8: /5VDC -> /RS232 interfeisas/NEX_5VDC
- J18 pad 1: /COM -> /RS232 interfeisas/NEX_COM
- J19 pad 3: (no net) -> /EV1
- J19 pad 4: (no net) -> /EV2
- J19 pad 5: (no net) -> /EV3
- J19 pad 6: (no net) -> /EV4
- J19 pad 7: (no net) -> Net-(J19-Pad7)
- J20 pad 1: (no net) -> Net-(J20-Pad1)
- J20 pad 2: (no net) -> Net-(J20-Pad2)
- J3 pad 10: /OUTAC10 -> Net-(J3-Pad10)
- J3 pad 11: (no net) -> /OUTAC11
- J3 pad 12: (no net) -> /OUTAC12
- J3 pad 13: (no net) -> /OUTAC12N
- J3 pad 14: (no net) -> /OUTAC11N
- J3 pad 15: /OUTAC10N -> Net-(J3-Pad15)
- K1 pad 11: /ACN -> /ACL
- K1 pad 14: /230N -> Net-(F1-Pad1)
- K1 pad A2: (no net) -> /K1
- K2 pad 11: /OUTAC10N -> Net-(J10-Pad2)
- K2 pad 12: (no net) -> Net-(K2-Pad12)
- K2 pad 14: /230N -> Net-(F1-Pad2)
- K2 pad 21: /OUTAC10 -> Net-(J10-Pad1)
- K2 pad 22: (no net) -> Net-(K2-Pad22)
- K2 pad 24: (no net) -> /ACN
- K2 pad A2: (no net) -> /K2
- K3 pad 11: (no net) -> /EXT1_11
- K3 pad 12: (no net) -> /EXT1_12
- K3 pad 14: (no net) -> /EXT1_14
- K3 pad A2: (no net) -> /K3
- K4 pad 11: (no net) -> /EXT3_11
- K4 pad 12: (no net) -> /EXT3_12
- K4 pad 14: (no net) -> /EXT3_14
- K4 pad A2: (no net) -> /K4
- K5 pad 11: (no net) -> /EXT2_11
- K5 pad 12: (no net) -> /EXT2_12
- K5 pad 14: (no net) -> /EXT2_14
- K5 pad A2: (no net) -> /K5
- K6 pad 11: (no net) -> /EXT4_11
- K6 pad 12: (no net) -> /EXT4_12
- K6 pad 14: (no net) -> /EXT4_14
- K6 pad A2: (no net) -> /K6
- R38 pad 1: /MCP23017 extended port/EO1 -> Net-(R38-Pad1)
- R38 pad 2: /MCP23017 extended port/EO1 -> Net-(R38-Pad2)
- R39 pad 1: /MCP23017 extended port/EO2 -> Net-(J2-Pad2)
- R39 pad 2: /MCP23017 extended port/EO2 -> Net-(R39-Pad2)
- R40 pad 1: /MCP23017 extended port/EO3 -> Net-(J2-Pad3)
- R40 pad 2: /MCP23017 extended port/EO3 -> Net-(R40-Pad2)
- R41 pad 1: /MCP23017 extended port/EO4 -> Net-(J2-Pad3)
- R41 pad 2: /MCP23017 extended port/EO4 -> Net-(R41-Pad2)
- R42 pad 1: /MCP23017 extended port/EO5 -> Net-(J2-Pad1)
- R42 pad 2: /MCP23017 extended port/EO5 -> Net-(R38-Pad1)
- R43 pad 1: /MCP23017 extended port/EO6 -> /ACN
- R43 pad 2: /MCP23017 extended port/EO6 -> Net-(R27-Pad1)
- R44 pad 1: /MCP23017 extended port/EO7 -> Net-(R44-Pad1)
- R44 pad 2: /MCP23017 extended port/EO7 -> Net-(R29-Pad1)
- R47 pad 1: /5VDC -> /RS232 interfeisas/NEX_5VDC
- R48 pad 1: /5VDC -> /RS232 interfeisas/NEX_5VDC
- U1 pad 1: (no net) -> Net-(D1-Pad1)
- U1 pad 2: (no net) -> Net-(D1-Pad2)
- U1 pad 3: (no net) -> /COM
- U1 pad 4: /OUTAC9 -> /LIGHTWC
- U10 pad 2: (no net) -> Net-(U10-Pad2)
- U10 pad 3: (no net) -> Net-(U10-Pad3)
- U10 pad 5: (no net) -> Net-(U10-Pad5)
- U10 pad 6: (no net) -> Net-(R20-Pad2)
- U11 pad 2: (no net) -> Net-(U11-Pad2)
- U11 pad 3: (no net) -> Net-(U11-Pad3)
- U11 pad 5: (no net) -> Net-(U11-Pad5)
- U11 pad 6: (no net) -> Net-(R22-Pad2)
- U12 pad 2: (no net) -> Net-(U12-Pad2)
- U12 pad 3: (no net) -> Net-(U12-Pad3)
- U12 pad 5: (no net) -> Net-(U12-Pad5)
- U12 pad 6: (no net) -> Net-(R24-Pad2)
- U14 pad 1: (no net) -> /MCP23017 extended port/EA0
- U14 pad 11: (no net) -> Net-(U14-Pad11)
- U14 pad 14: (no net) -> Net-(U14-Pad14)
- U14 pad 19: (no net) -> /MCP23017 extended port/INTB1
- U14 pad 2: (no net) -> /MCP23017 extended port/EA1
- U14 pad 20: (no net) -> /MCP23017 extended port/INTA1
- U14 pad 21: (no net) -> /MCP23017 extended port/EA8
- U14 pad 22: (no net) -> /MCP23017 extended port/EA9
- U14 pad 23: (no net) -> /MCP23017 extended port/EA10
- U14 pad 24: (no net) -> /MCP23017 extended port/EA11
- U14 pad 25: (no net) -> /MCP23017 extended port/EA12
- U14 pad 26: (no net) -> /MCP23017 extended port/EA13
- U14 pad 27: (no net) -> /MCP23017 extended port/EA14
- U14 pad 28: (no net) -> /MCP23017 extended port/EA15
- U14 pad 3: (no net) -> /MCP23017 extended port/EA2
- U14 pad 4: (no net) -> /MCP23017 extended port/EA3
- U14 pad 5: (no net) -> /MCP23017 extended port/EA4
- U14 pad 6: (no net) -> /MCP23017 extended port/EA5
- U14 pad 7: (no net) -> /MCP23017 extended port/EA6
- U14 pad 8: (no net) -> /MCP23017 extended port/EA7
- U17 pad 11: (no net) -> Net-(U17-Pad11)
- U17 pad 12: (no net) -> Net-(U17-Pad12)
- U17 pad 13: (no net) -> Net-(U17-Pad13)
- U17 pad 14: (no net) -> Net-(U17-Pad14)
- U17 pad 15: /COM -> /RS232 interfeisas/NEX_COM
- U17 pad 16: /5VDC -> /RS232 interfeisas/NEX_5VDC
- U18 pad 10: (no net) -> Net-(R52-Pad2)
- U18 pad 11: (no net) -> Net-(U18-Pad11)
- U18 pad 12: (no net) -> Net-(U18-Pad12)
- U18 pad 13: (no net) -> Net-(U18-Pad13)
- U18 pad 14: (no net) -> Net-(U18-Pad14)
- U18 pad 9: (no net) -> Net-(R54-Pad2)
- U19 pad 1: (no net) -> /MCP23017 extended port/EB0
- U19 pad 11: (no net) -> Net-(U19-Pad11)
- U19 pad 14: (no net) -> Net-(U19-Pad14)
- U19 pad 19: (no net) -> /MCP23017 extended port/INTB2
- U19 pad 2: (no net) -> /MCP23017 extended port/EB1
- U19 pad 20: (no net) -> /MCP23017 extended port/INTA2
- U19 pad 21: (no net) -> /MCP23017 extended port/EB8
- U19 pad 22: (no net) -> /MCP23017 extended port/EB9
- U19 pad 23: (no net) -> /MCP23017 extended port/EB10
- U19 pad 24: (no net) -> /MCP23017 extended port/EB11
- U19 pad 25: (no net) -> /MCP23017 extended port/EB12
- U19 pad 26: (no net) -> /MCP23017 extended port/EB13
- U19 pad 27: (no net) -> /MCP23017 extended port/EB14
- U19 pad 28: (no net) -> /MCP23017 extended port/EB15
- U19 pad 3: (no net) -> /MCP23017 extended port/EB2
- U19 pad 4: (no net) -> /MCP23017 extended port/EB3
- U19 pad 5: (no net) -> /MCP23017 extended port/EB4
- U19 pad 6: (no net) -> /MCP23017 extended port/EB5
- U19 pad 7: (no net) -> /MCP23017 extended port/EB6
- U19 pad 8: (no net) -> /MCP23017 extended port/EB7
- U3 pad 2: (no net) -> Net-(U3-Pad2)
- U3 pad 3: (no net) -> Net-(U3-Pad3)
- U3 pad 5: (no net) -> Net-(U3-Pad5)
- U3 pad 6: (no net) -> Net-(R8-Pad2)
- U4 pad 2: (no net) -> Net-(U4-Pad2)
- U4 pad 3: (no net) -> Net-(U4-Pad3)
- U4 pad 5: (no net) -> Net-(U4-Pad5)
- U4 pad 6: (no net) -> Net-(R10-Pad2)
- U5 pad 2: (no net) -> Net-(U5-Pad2)
- U5 pad 3: (no net) -> Net-(U5-Pad3)
- U5 pad 5: (no net) -> Net-(U5-Pad5)
- U5 pad 6: (no net) -> Net-(R12-Pad2)
- U7 pad 2: (no net) -> Net-(U7-Pad2)
- U7 pad 3: (no net) -> Net-(U7-Pad3)
- U7 pad 5: (no net) -> Net-(U7-Pad5)
- U7 pad 6: (no net) -> Net-(R14-Pad2)
- U8 pad 2: (no net) -> Net-(U8-Pad2)
- U8 pad 3: (no net) -> Net-(U8-Pad3)
- U8 pad 5: (no net) -> Net-(U8-Pad5)
- U8 pad 6: (no net) -> Net-(R16-Pad2)
- U9 pad 2: (no net) -> Net-(U9-Pad2)
- U9 pad 3: (no net) -> Net-(U9-Pad3)
- U9 pad 5: (no net) -> Net-(U9-Pad5)
- U9 pad 6: (no net) -> Net-(R18-Pad2)
Routing:
- net /5VDC: track 87.1 -> 0.00 mm
- net /RS232 interfeisas/NEX_5VDC: track 0.00 -> 87.1 mm
- net Net-(F1-Pad2): track 0.00 -> 70.9 mm
- net /ACN: track 0.00 -> 61.6 mm, vias 0 -> 2
- net Net-(F1-Pad1): track 0.00 -> 28.5 mm
- net Net-(R44-Pad1): track 0.00 -> 27.4 mm
- net Net-(C1-Pad1): track 0.00 -> 23.4 mm, vias 0 -> 1
- net /12VDC: track 0.00 -> 16.8 mm
- net Net-(J2-Pad1): track 0.00 -> 14.1 mm, vias 0 -> 1
- net Net-(J2-Pad2): track 0.00 -> 14.1 mm, vias 0 -> 1
- net Net-(R30-Pad1): track 0.00 -> 13.4 mm, vias 0 -> 1
- net Net-(J2-Pad3): track 0.00 -> 13.2 mm, vias 0 -> 1
- net /COM: track 0.00 -> 6.13 mm
- net Net-(D2-Pad2): track 0.00 -> 5.72 mm
- net Net-(D12-Pad1): track 0.00 -> 5.72 mm
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- added copper zone on B.Cu, net /ACN
- added copper zone on F.Cu, net /RS232 interfeisas/NEX_COM
- added copper zone on B.Cu, net Net-(F1-Pad2)
Other:
- board size 188 x 80 mm -> 254 x 149 mm
