File: Kicad/mcp_port.sch (KiCad schematic (older format))
At the start: 41 parts

Commit message: schemos paruosimas
Parts:
- removed D? (x16): 10MQ100, Diodes_SMD:D_SMA, symbol Device:D
- U? (x2): value L293 -> L293D

Commit message: schemos, pcb paruosimas
Parts:
- removed C?: 0.1, Capacitors_SMD:C_0805, symbol ihouse-rescue:Device_C-ihouse-rescue
- removed D? (x2): D, symbol ihouse-rescue:Device_D-ihouse-rescue
- removed M?: Motor_DC, symbol ihouse-rescue:Motor_Motor_DC-ihouse-rescue
- removed R? (x7): R, Resistors_SMD:R_0805, symbol ihouse-rescue:Device_R-ihouse-rescue
- removed SW?: RHome, symbol ihouse-rescue:Switch_SW_Push_Open-ihouse-rescue
- removed U?: MCP23017, digikey-footprints:DIP-28_W7.62mm, symbol ihouse-rescue:dk_Interface-I-O-Expanders_MCP23017-E_SP-ihouse-rescue
- removed U?: L293D, Package_DIP:DIP-16_W7.62mm, symbol ihouse-rescue:L293-Driver_Motor
- added C3: 0.1, Capacitors_SMD:C_0805, symbol ihouse-rescue:Device_C-ihouse-rescue
- added D14, D15: D, symbol ihouse-rescue:Device_D-ihouse-rescue
- added M2: Motor_DC, symbol ihouse-rescue:Motor_Motor_DC-ihouse-rescue
- added R34, R40, R41, R43, R44, R45, R46: R, Resistors_SMD:R_0805, symbol ihouse-rescue:Device_R-ihouse-rescue
- added SW1: RHome, symbol ihouse-rescue:Switch_SW_Push_Open-ihouse-rescue
- added U14: MCP23017, digikey-footprints:DIP-28_W7.62mm, symbol ihouse-rescue:dk_Interface-I-O-Expanders_MCP23017-E_SP-ihouse-rescue
- added U16: L293D, Package_DIP:DIP-16_W7.62mm, symbol ihouse-rescue:L293-Driver_Motor
- gave numbers to parts that had none: 11
Connections:
- net 12VDC: now also U16.8 (VCC2)
- net 5VDC: now also R34.1, U14.9 (VDD), U16.16 (VCC1)
- net COM: now also C3.2, U14.10 (VSS), U14.15 (A0), U14.16 (A1), U14.17 (A2), U16.12 (GND), U16.13 (GND), U16.4 (GND), U16.5 (GND)
- net DIRA: now also U14.5 (GPB4), U16.10 (3A), U16.2 (1A)
- net DIRB: now also U14.6 (GPB5), U16.15 (4A), U16.7 (2A)
- net EO0: now also U14.7 (GPB6)
- net EO1: now also U14.8 (GPB7)
- net EO2: now also U14.21 (GPA0)
- net EO3: now also R40.1, R40.2, U14.22 (GPA1)
- net EO4: now also R41.1, R41.2, U14.23 (GPA2)
- net EO5: now also U14.24 (GPA3)
- net EO6: now also R43.1, R43.2, U14.25 (GPA4)
- net EO7: now also R44.1, R44.2, U14.26 (GPA5)
- net EO8: now also R45.1, R45.2, U14.27 (GPA6)
- net EO9: now also R46.1, R46.2, U14.28 (GPA7)
- net SCL: now also U14.12 (SCK)
- net SDA: now also U14.13 (SDA)
- net V3A1: now also U16.3 (1Y)
- net V3A2: now also U16.6 (2Y)
- net V4A1: now also U16.11 (3Y)
- net V4A2: now also U16.14 (4Y)
- net VL1: now also U14.1 (GPB0)
- net VL2: now also U14.2 (GPB1)
- net VL3: now also U14.3 (GPB2), U16.1 (EN1,2)
- net VL4: now also U14.4 (GPB3), U16.9 (EN3,4)
- net ~MCPRST: now also C3.1, R34.2, U14.18 (~RESET)
- net at SW2.2 (B): now also D15.1 (K), M2.2 (-)
- net at SW2.1 (A): now also D15.2 (A)
- new net: D14.1 (K), M2.1 (+), SW1.2 (B)
- new net: D14.2 (A), SW1.1 (A)
Other:
- moved on the sheet: C2, D13, J13, R35, R36, R37, R38, R39, R42, U15

Commit message: tarpinis kommitas
Parts:
- removed J13: Valves, Connectors_Molex:Molex_MiniFit-JR-5556-10A_2x05x4.20mm_Straight, symbol ihouse-rescue:Connector_Generic_Conn_02x05_Counter_Clockwise-ihouse-rescue
- removed R38, R39, R40, R41, R42, R43, R44, R45, R46: R, Resistors_SMD:R_0805, symbol ihouse-rescue:Device_R-ihouse-rescue
- removed U15, U16: L293D, Package_DIP:DIP-16_W7.62mm, symbol ihouse-rescue:L293-Driver_Motor
- added C13: 0.1, Capacitors_SMD:C_0805_HandSoldering, symbol ihouse-rescue:Device_C-ihouse-rescue
- added U19: MCP23017, digikey-footprints:SOIC-28_W7.5mm, symbol ihouse-rescue:dk_Interface-I-O-Expanders_MCP23017-E_SP-ihouse-rescue
- C2, C3: footprint Capacitors_SMD:C_0805 -> Capacitors_SMD:C_0805_HandSoldering
- D13: value D -> BAS32
- R34: value R -> 15k; footprint Resistors_SMD:R_0805 -> Resistors_SMD:R_0805_HandSoldering
- R35, R36, R37: value R -> 1k; footprint Resistors_SMD:R_0805 -> Resistors_SMD:R_0805_HandSoldering
- U14: footprint digikey-footprints:DIP-28_W7.62mm -> digikey-footprints:SOIC-28_W7.5mm
Connections:
- net 5VDC: now also R37.1, C13.1, U19.9 (VDD)
- net COM: now also C13.2, U19.10 (VSS), U19.16 (A1), U19.17 (A2)
- net SCL: now also U19.12 (SCK)
- net SDA: now also U19.13 (SDA)
- net ~MCPRST: now also U19.18 (~RESET)
- net INTB1: now reaches U14.19 (INTB)
- net INTA1: now reaches U14.20 (INTA)
- net DIRA renamed EA4
- net DIRB renamed EA5
- removed net EO0: R37.1, R37.2, U14.7 (GPB6)
- net EO1 renamed EA7
- net EO2 renamed EA8
- net EO3 renamed EA9
- net EO4 renamed EA10
- net EO5 renamed EA11
- net EO6 renamed EA12
- net EO7 renamed EA13
- net EO8 renamed EA14
- net EO9 renamed EA15
- net VL1 renamed EA0
- net VL2 renamed EA1
- net VL3 renamed EA2
- net VL4 renamed EA3
- new net: R37.2, U19.15 (A0)
- new net EA6: U14.7 (GPB6)
- new net EB0: U19.1 (GPB0)
- new net EB1: U19.2 (GPB1)
- new net EB10: U19.23 (GPA2)
- new net EB11: U19.24 (GPA3)
- new net EB12: U19.25 (GPA4)
- new net EB13: U19.26 (GPA5)
- new net EB14: U19.27 (GPA6)
- new net EB15: U19.28 (GPA7)
- new net EB2: U19.3 (GPB2)
- new net EB3: U19.4 (GPB3)
- new net EB4: U19.5 (GPB4)
- new net EB5: U19.6 (GPB5)
- new net EB6: U19.7 (GPB6)
- new net EB7: U19.8 (GPB7)
- new net EB8: U19.21 (GPA0)
- new net EB9: U19.22 (GPA1)
- new net INTA2: U19.20 (INTA)
- new net INTB2: U19.19 (INTB)
Other:
- moved on the sheet: R35, R36
