File: Kicad/ihouse.sch (KiCad schematic (older format))
At the start: 83 parts, among them K1 FINDER-34.51, K2 RT42xxxx, K3 FINDER-34.51, K4 FINDER-34.51, K5 FINDER-34.51, K6 FINDER-34.51

Commit message: pataisyta schema, sukonfiguruotas uartas per dma
Parts:
- added C?: 0.1, Capacitors_SMD:C_0805_HandSoldering, symbol Device:C
- added C? (x2): 1n, Capacitors_SMD:C_0805_HandSoldering, symbol Device:C
- added D?: TX, LEDs:LED_0805_HandSoldering, symbol Device:LED
- added D?: RX, LEDs:LED_0805_HandSoldering, symbol Device:LED
- added D?: RC, LEDs:LED_0805_HandSoldering, symbol Device:LED
- added J?: 8P8C, symbol Connector:8P8C
- added J?: Conn_01x08, symbol Connector_Generic:Conn_01x08
- added Q? (x2): BC817, Package_TO_SOT_SMD:SOT-23, symbol Transistor_BJT:BC817
- added R? (x4): 47R, Resistor_SMD:R_0805_2012Metric_Pad1.15x1.40mm_HandSolder, symbol ihouse-rescue:Device_R-ihouse-rescue
- added R? (x5): 1k, Resistor_SMD:R_0805_2012Metric_Pad1.15x1.40mm_HandSolder, symbol ihouse-rescue:Device_R-ihouse-rescue
- added R? (x3): 10k, Resistor_SMD:R_0805_2012Metric_Pad1.15x1.40mm_HandSolder, symbol ihouse-rescue:Device_R-ihouse-rescue
Connections:
- net labels added: NEXTION_RX, NEXTION_TX, RC_CONTROL
- wire segments 391 -> 469
Other:
- note added: "NEXTION"
- moved on the sheet: M?

Commit message: tarpinis kommitas
Parts:
- removed R? (x2): 47R, Resistor_SMD:R_0805_2012Metric_Pad1.15x1.40mm_HandSolder, symbol ihouse-rescue:Device_R-ihouse-rescue
- added Q?: BC807, Package_TO_SOT_SMD:SOT-23, symbol Transistor_BJT:BC807
- added R?: 100k, Resistor_SMD:R_0805_2012Metric_Pad1.15x1.40mm_HandSolder, symbol ihouse-rescue:Device_R-ihouse-rescue
- added TH?: 500mA, Resistors_SMD:R_1206_HandSoldering, symbol Device:Thermistor_NTC
Connections:
- wire segments 469 -> 473
Other:
- moved on the sheet: C?, D?, R?

Commit message: schemos paruosimas
Parts:
- removed C?: 0.1, Capacitors_SMD:C_0805_HandSoldering, symbol Device:C
- removed C? (x2): 1n, Capacitors_SMD:C_0805_HandSoldering, symbol Device:C
- removed D?: TX, LEDs:LED_0805_HandSoldering, symbol Device:LED
- removed D?: RX, LEDs:LED_0805_HandSoldering, symbol Device:LED
- removed D?: RC, LEDs:LED_0805_HandSoldering, symbol Device:LED
- removed J?: 8P8C, symbol Connector:8P8C
- removed J?: Conn_01x08, symbol Connector_Generic:Conn_01x08
- removed Q? (x2): BC817, Package_TO_SOT_SMD:SOT-23, symbol Transistor_BJT:BC817
- removed Q?: BC807, Package_TO_SOT_SMD:SOT-23, symbol Transistor_BJT:BC807
- removed R? (x2): 47R, Resistor_SMD:R_0805_2012Metric_Pad1.15x1.40mm_HandSolder, symbol ihouse-rescue:Device_R-ihouse-rescue
- removed R? (x5): 1k, Resistor_SMD:R_0805_2012Metric_Pad1.15x1.40mm_HandSolder, symbol ihouse-rescue:Device_R-ihouse-rescue
- removed R?: 100k, Resistor_SMD:R_0805_2012Metric_Pad1.15x1.40mm_HandSolder, symbol ihouse-rescue:Device_R-ihouse-rescue
- removed R? (x3): 10k, Resistor_SMD:R_0805_2012Metric_Pad1.15x1.40mm_HandSolder, symbol ihouse-rescue:Device_R-ihouse-rescue
- removed TH?: 500mA, Resistors_SMD:R_1206_HandSoldering, symbol Device:Thermistor_NTC
- added C? (x8): 1u, Capacitors_SMD:C_0805_HandSoldering, symbol Device:C
- added D?: RX, LEDs:LED_0805_HandSoldering, symbol Device:LED
- added D?: TX, LEDs:LED_0805_HandSoldering, symbol Device:LED
- added D?: RC, LEDs:LED_0805_HandSoldering, symbol Device:LED
- added J?: 8P8C, symbol ihouse-rescue:8P8C-Connector
- added J?: Conn_01x08, symbol ihouse-rescue:Conn_01x08-Connector_Generic
- added R? (x5): 1k, Resistor_SMD:R_0805_2012Metric_Pad1.15x1.40mm_HandSolder, symbol ihouse-rescue:Device_R-ihouse-rescue
- added R?: 2k, Resistor_SMD:R_0805_2012Metric_Pad1.15x1.40mm_HandSolder, symbol ihouse-rescue:Device_R-ihouse-rescue
- added TH?: 500mA, Resistors_SMD:R_1206_HandSoldering, symbol Device:Thermistor_NTC
- added U? (x2): MAX232, symbol Interface:MAX232
Connections:
- net labels added: GND, NEX_RX, NEX_TX, RXC, RXN, TXC, TXN
- net labels removed: NEXTION_RX, NEXTION_TX
- wire segments 473 -> 482
Other:
- note removed: "NEXTION"

Commit message: schemos, pcb paruosimas
Parts:
- removed C?: 100uFx16V, Capacitors_SMD:CP_Elec_6.3x5.7, symbol ihouse-rescue:capacitors_CP_100uFx16V-ihouse-rescue
- removed C? (x8): 1u, Capacitors_SMD:C_0805_HandSoldering, symbol Device:C
- removed D? (x3): Z0103MN, Package_TO_SOT_SMD:SOT-223, symbol ihouse-rescue:Triac_Thyristor_Z0103MN-ihouse-rescue
- removed D?: RX, LEDs:LED_0805_HandSoldering, symbol Device:LED
- removed D?: TX, LEDs:LED_0805_HandSoldering, symbol Device:LED
- removed D?: RC, LEDs:LED_0805_HandSoldering, symbol Device:LED
- removed F?: 3A, Fuse:Fuseholder_Cylinder-5x20mm_Schurter_0031_8201_Horizontal_Open, symbol ihouse-rescue:Device_Fuse-ihouse-rescue
- removed J? (x3): Conn_01x01, mech:Faston_6.3x0.8x14, symbol ihouse-rescue:Connector_Generic_Conn_01x01-ihouse-rescue
- removed J?: AC OUTS, Connector_Molex:Molex_Mini-Fit_Jr_5566-24A_2x12_P4.20mm_Vertical, symbol ihouse-rescue:Connector_Generic_Conn_02x12_Counter_Clockwise-ihouse-rescue
- removed J?: AC INPUTS, Connector_Molex:Molex_Mini-Fit_Jr_5566-04A_2x02_P4.20mm_Vertical, symbol ihouse-rescue:Connector_Generic_Conn_02x02_Counter_Clockwise-ihouse-rescue
- removed J?: 8P8C, symbol ihouse-rescue:8P8C-Connector
- removed J?: Conn_01x08, symbol ihouse-rescue:Conn_01x08-Connector_Generic
- removed J?: EXT2, symbol ihouse-rescue:Connector_Screw_Terminal_01x03-ihouse-rescue
- removed J?: EXT3, symbol ihouse-rescue:Connector_Screw_Terminal_01x03-ihouse-rescue
- removed J?: EXT4, symbol ihouse-rescue:Connector_Screw_Terminal_01x03-ihouse-rescue
- removed K? (x2): FINDER-32.21-x300, Relay_THT:Relay_SPST_Schrack-RT1-FormA_RM5mm, symbol ihouse-rescue:Relay_FINDER-32.21-x300-ihouse-rescue
- removed K?: G5Q-1A, Relay_THT:Relay_SPDT_Finder_34.51_Vertical, symbol ihouse-rescue:Relay_G5Q-1A-ihouse-rescue
- removed R? (x12): R, Resistor_SMD:R_0805_2012Metric_Pad1.15x1.40mm_HandSolder, symbol ihouse-rescue:Device_R-ihouse-rescue
- removed R? (x4): 33k, Resistor_SMD:R_1206_3216Metric_Pad1.42x1.75mm_HandSolder, symbol ihouse-rescue:Device_R-ihouse-rescue
- removed R?: Rx, Resistor_SMD:R_0805_2012Metric_Pad1.15x1.40mm_HandSolder, symbol ihouse-rescue:Device_R-ihouse-rescue
- removed R? (x5): 1k, Resistor_SMD:R_0805_2012Metric_Pad1.15x1.40mm_HandSolder, symbol ihouse-rescue:Device_R-ihouse-rescue
- removed R?: 2k, Resistor_SMD:R_0805_2012Metric_Pad1.15x1.40mm_HandSolder, symbol ihouse-rescue:Device_R-ihouse-rescue
- removed T?: Transformer_TEZ_22x24_6V, Transformer_THT:Transformer_Breve_TEZ-22x24, symbol ihouse-rescue:disc_Transformer_TEZ_22x24_6V-ihouse-rescue
- removed TH?: 500mA, Resistors_SMD:R_1206_HandSoldering, symbol Device:Thermistor_NTC
- removed U? (x6): MOC3060S, disc:DIP-6_W9.53mm_SMD, symbol ihouse-rescue:disc_MOC3060S-ihouse-rescue
- removed U? (x2): MAX232, symbol Interface:MAX232
- removed U?: ULN2803A, symbol ihouse-rescue:Transistor_Array_ULN2803A-ihouse-rescue
- removed U?: LTV-817, Package_DIP:DIP-4_W7.62mm, symbol ihouse-rescue:Isolator_LTV-817-ihouse-rescue
- added C1: 100uFx16V, Capacitors_SMD:CP_Elec_6.3x5.7, symbol ihouse-rescue:capacitors_CP_100uFx16V-ihouse-rescue
- added D1, D5, D9: Z0103MN, Package_TO_SOT_SMD:SOT-223, symbol ihouse-rescue:Triac_Thyristor_Z0103MN-ihouse-rescue
- added F1: 3A, Fuse:Fuseholder_Cylinder-5x20mm_Schurter_0031_8201_Horizontal_Open, symbol ihouse-rescue:Device_Fuse-ihouse-rescue
- added J1: 8P8C, symbol ihouse-rescue:8P8C-Connector
- added J10, J8, J9: Conn_01x01, mech:Faston_6.3x0.8x14, symbol ihouse-rescue:Connector_Generic_Conn_01x01-ihouse-rescue
- added J2: AC INPUTS, Connector_Molex:Molex_Mini-Fit_Jr_5566-04A_2x02_P4.20mm_Vertical, symbol ihouse-rescue:Connector_Generic_Conn_02x02_Counter_Clockwise-ihouse-rescue
- added J3: AC OUTS, Connector_Molex:Molex_Mini-Fit_Jr_5566-24A_2x12_P4.20mm_Vertical, symbol ihouse-rescue:Connector_Generic_Conn_02x12_Counter_Clockwise-ihouse-rescue
- added J5: EXT2, symbol ihouse-rescue:Connector_Screw_Terminal_01x03-ihouse-rescue
- added J6: EXT3, symbol ihouse-rescue:Connector_Screw_Terminal_01x03-ihouse-rescue
- added J7: EXT4, symbol ihouse-rescue:Connector_Screw_Terminal_01x03-ihouse-rescue
- added K7, K8: FINDER-32.21-x300, Relay_THT:Relay_SPST_Schrack-RT1-FormA_RM5mm, symbol ihouse-rescue:Relay_FINDER-32.21-x300-ihouse-rescue
- added K9: G5Q-1A, Relay_THT:Relay_SPDT_Finder_34.51_Vertical, symbol ihouse-rescue:Relay_G5Q-1A-ihouse-rescue
- added R1, R11, R12, R13, R15, R16, R17, R18, R2, R20, R21, R8: R, Resistor_SMD:R_0805_2012Metric_Pad1.15x1.40mm_HandSolder, symbol ihouse-rescue:Device_R-ihouse-rescue
- added R27, R28, R29, R6: 33k, Resistor_SMD:R_1206_3216Metric_Pad1.42x1.75mm_HandSolder, symbol ihouse-rescue:Device_R-ihouse-rescue
- added R32: Rx, Resistor_SMD:R_0805_2012Metric_Pad1.15x1.40mm_HandSolder, symbol ihouse-rescue:Device_R-ihouse-rescue
- added T1: Transformer_TEZ_22x24_6V, Transformer_THT:Transformer_Breve_TEZ-22x24, symbol ihouse-rescue:disc_Transformer_TEZ_22x24_6V-ihouse-rescue
- added U1, U10, U11, U12, U3, U8: MOC3060S, disc:DIP-6_W9.53mm_SMD, symbol ihouse-rescue:disc_MOC3060S-ihouse-rescue
- added U2: LTV-817, Package_DIP:DIP-4_W7.62mm, symbol ihouse-rescue:Isolator_LTV-817-ihouse-rescue
- added U6: ULN2803A, symbol ihouse-rescue:Transistor_Array_ULN2803A-ihouse-rescue
- gave numbers to parts that had none: 35
Connections:
- net labels removed: GND, NEX_RX, NEX_TX, RC_CONTROL, RXC, RXN, TXC, TXN
- wire segments 482 -> 410
Other:
- moved on the sheet: D10, D11, D12, D3, D4, D6, D7, D8, J4, K1, K2, K4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

Commit message: tarpinis kommitas
Parts:
- added J13: UART1, Pin_Headers:Pin_Header_Straight_1x05_Pitch2.54mm, symbol Connector_Generic:Conn_01x05
- added J19: EV1527, Pin_Headers:Pin_Header_Straight_1x07_Pitch2.54mm, symbol Connector_Generic:Conn_01x07
- added J20: Valves, Connectors_Molex:Molex_MiniFit-JR-5556-10A_2x05x4.20mm_Straight, symbol ihouse-rescue:Connector_Generic_Conn_02x05_Counter_Clockwise-ihouse-rescue
- added U15, U16: L293D, Package_DIP:DIP-16_W7.62mm, symbol ihouse-rescue:L293-Driver_Motor
- J1: value 8P8C -> UART2; footprint (none) -> Connectors:RJ45_8
- J3: footprint Connector_Molex:Molex_Mini-Fit_Jr_5566-24A_2x12_P4.20mm_Vertical -> Connectors_Molex:Molex_MiniFit-JR-5556-24A_2x12x4.20mm_Straight
- K1: footprint (none) -> Relays_THT:Relay_DPST_Schrack-RT2-FormA_RM5mm
- K2: footprint Relay_THT:Relay_DPDT_Schrack-RT2-FormC_RM5mm -> Relays_THT:Relay_DPDT_Finder_40.52
Connections:
- net labels added: DIRA, DIRB, EV1, EV2, EV3, EV4, RCCTRL, V1A1, V1A2, V2A1, V2A2, V3A1, V3A2, V4A1, V4A2, VL1, VL2, VL3, VL4
- wire segments 410 -> 478
- no-connect marks 0 -> 2
Other:
- note added: "TB387\nRS485"
- moved on the sheet: J1, M1

Commit message: schemos paruosimas
Parts:
- removed D1: Z0103MN, Package_TO_SOT_SMD:SOT-223, symbol ihouse-rescue:Triac_Thyristor_Z0103MN-ihouse-rescue
- removed J10, J11: Conn_01x01, mech:Faston_6.3x0.8x14, symbol ihouse-rescue:Connector_Generic_Conn_01x01-ihouse-rescue
- removed J2: AC INPUTS, Connector_Molex:Molex_Mini-Fit_Jr_5566-04A_2x02_P4.20mm_Vertical, symbol ihouse-rescue:Connector_Generic_Conn_02x02_Counter_Clockwise-ihouse-rescue
- removed J20: Valves, Connectors_Molex:Molex_MiniFit-JR-5556-10A_2x05x4.20mm_Straight, symbol ihouse-rescue:Connector_Generic_Conn_02x05_Counter_Clockwise-ihouse-rescue
- removed K7, K8: FINDER-32.21-x300, Relay_THT:Relay_SPST_Schrack-RT1-FormA_RM5mm, symbol ihouse-rescue:Relay_FINDER-32.21-x300-ihouse-rescue
- removed K9: G5Q-1A, Relay_THT:Relay_SPDT_Finder_34.51_Vertical, symbol ihouse-rescue:Relay_G5Q-1A-ihouse-rescue
- removed TH1: 230V/150mA, symbol ihouse-rescue:Device_Thermistor_PTC-ihouse-rescue
- removed U1: MOC3060S, disc:DIP-6_W9.53mm_SMD, symbol ihouse-rescue:disc_MOC3060S-ihouse-rescue
- added C14, C15: CP, Capacitor_SMD:CP_Elec_10x7.9, symbol Device:CP
- added D1: LL4148, Diode_SMD:D_MiniMELF, symbol ihouse-rescue:Diode_LL4148-ihouse-rescue
- added D19, D20: LL4004, Diode_SMD:D_MELF, symbol Device:D
- added J10: iSOCKET, symbol Connector_Generic:Conn_01x02
- added J11: To AC/DC, Connector_Phoenix_MSTB:PhoenixContact_MSTBVA_2,5_2-G_1x02_P5.00mm_Vertical, symbol Connector_Generic:Conn_01x02
- added J2: AC Inputs, Connector_Molex:Molex_Mini-Fit_Jr_5566-04A_2x02_P4.20mm_Vertical, symbol Connector_Generic:Conn_02x02_Top_Bottom
- added J20: Valve1, Connectors_Molex:Molex_KK-6410-02_02x2.54mm_Straight, symbol Connector_Generic:Conn_01x02
- added J21: Valve2, Connectors_Molex:Molex_KK-6410-02_02x2.54mm_Straight, symbol Connector_Generic:Conn_01x02
- added J22: Valve3, Connectors_Molex:Molex_KK-6410-02_02x2.54mm_Straight, symbol Connector_Generic:Conn_01x02
- added J23: Valve4, Connectors_Molex:Molex_KK-6410-02_02x2.54mm_Straight, symbol Connector_Generic:Conn_01x02
- added R38, R39, R40, R41, R42, R43, R44: 33k, Resistor_SMD:R_1206_3216Metric_Pad1.42x1.75mm_HandSolder, symbol ihouse-rescue:Device_R-ihouse-rescue
- added TH3: 1.5A/30V, Resistor_SMD:R_1210_3225Metric, symbol Device:Thermistor_PTC
- added TH4: 0.5A/230V, Varistor:RV_Disc_D7mm_W3.4mm_P5mm, symbol Device:Thermistor_PTC
- added TR1: TSZZ20-006M_1, Transformer_THT:Transformer_Breve_TEZ-47x57_1, symbol Transformer:TSZZ20-006M_1
- added U1: LTV-817, Package_DIP:DIP-4_W7.62mm, symbol ihouse-rescue:Isolator_LTV-817-ihouse-rescue
- F1: value 3A -> 5A
- J12: footprint Connectors_Phoenix:PhoenixContact_MSTBA-G_03x5.00mm_Angled -> Connector_Phoenix_MSTB:PhoenixContact_MSTBVA_2,5_3-G_1x03_P5.00mm_Vertical
- J13: symbol Connector_Generic:Conn_01x05 -> ihouse-rescue:Conn_01x05-Connector_Generic
- J19: symbol Connector_Generic:Conn_01x07 -> ihouse-rescue:Conn_01x07-Connector_Generic
- J4, J5, J6, J7: footprint (none) -> Connectors_Terminal_Blocks:TerminalBlock_bornier-3_P5.08mm
- K1: footprint Relays_THT:Relay_DPST_Schrack-RT2-FormA_RM5mm -> Relay_THT:Relay_SPDT_Finder_34.51_Vertical
- K3, K4, K5, K6: footprint Relays_THT:Relay_SPDT_SingleRow_Standing_FinderType34Point51 -> Relay_THT:Relay_SPDT_Finder_34.51_Vertical
- R1, R2, R3: value R -> 33k; footprint Resistor_SMD:R_0805_2012Metric_Pad1.15x1.40mm_HandSolder -> Resistor_SMD:R_1206_3216Metric_Pad1.42x1.75mm_HandSolder
- TR2: renamed from T1; footprint Transformer_THT:Transformer_Breve_TEZ-22x24 -> Transformers_THT:Transformer_Breve_TEZ-22x24
- U15, U16: footprint Package_DIP:DIP-16_W7.62mm -> Housings_DIP:DIP-16_W7.62mm_LongPads
Connections:
- net labels added: LIGHTBASH, LIGHTWC
- net labels removed: 230L, 230N, 230VAC_L, 230VAC_N, INACL1, INACL2, INACN1, INACN2, LIGHTON, OC1, OUTAC10, OUTAC10N, OUTAC11, OUTAC11N, OUTAC12, OUTAC12N, V1A1, V1A2, V2A1, V2A2, V3A1, V3A2, V4A1, V4A2
- wire segments 478 -> 495
Other:
- moved on the sheet: C1, D12, F1, J12, J4, J5, J6, J7, J8, J9, K1, K2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

Commit message: tarpinis kommitas
Parts:
- added BT?: Battery_Cell, symbol device:Battery_Cell
- added C? (x2): C, Capacitors_SMD:C_0805_HandSoldering, symbol device:C
- added U?: DS1307+, Housings_SOIC:SOIC-8_3.9x4.9mm_Pitch1.27mm, symbol maxim:DS1307+
- added Y?: Crystal, symbol device:Crystal
- C14, C15: symbol Device:CP -> ihouse-rescue:CP-Device
- D19, D20: symbol Device:D -> ihouse-rescue:D-Device
- J10, J11, J20, J21, J22, J23: symbol Connector_Generic:Conn_01x02 -> ihouse-rescue:Conn_01x02-Connector_Generic
- J2: symbol Connector_Generic:Conn_02x02_Top_Bottom -> ihouse-rescue:Conn_02x02_Top_Bottom-Connector_Generic
- TH3, TH4: symbol Device:Thermistor_PTC -> ihouse-rescue:Thermistor_PTC-Device
- TR1: symbol Transformer:TSZZ20-006M_1 -> ihouse-rescue:TSZZ20-006M_1-Transformer
Connections:
- wire segments 495 -> 515
Other:
- moved on the sheet: J20, J21, J22, J23, U15, U16
