File: Kicad/rs232.sch (KiCad schematic (older format))
At the start: 28 parts, among them J14 Conn_01x01, J15 Conn_01x08, J16 Conn_01x01, J17 Conn_01x01, J18 Conn_01x01, U17 St232C, U18 ST232C

Commit message: tarpinis kommitas
Parts:
- R49: footprint Resistor_SMD:R_0805_2012Metric_Pad1.15x1.40mm_HandSolder -> Resistors_SMD:R_0805_HandSoldering
- TH2: value 500mA -> 1210L005WR
Other:
- note added: "150mA MAX"
Changed lines of the file:
@@
 P 6550 1900
 F 0 "TH2" H 6250 1950 50  0000 L CNN
-F 1 "500mA" H 6150 1850 50  0000 L CNN
+F 1 "1210L005WR" H 5950 1850 50  0000 L CNN
 F 2 "Resistors_SMD:R_1206_HandSoldering" H 6550 1950 50  0001 C CNN
 F 3 "~" H 6550 1950 50  0001 C CNN
@@
 F 0 "R49" V 6750 2250 50  0000 C CNN
 F 1 "2k" V 6850 2250 50  0000 C CNN
-F 2 "Resistor_SMD:R_0805_2012Metric_Pad1.15x1.40mm_HandSolder" V 6680 2250 50  0001 C CNN
+F 2 "Resistors_SMD:R_0805_HandSoldering" V 6680 2250 50  0001 C CNN
 F 3 "~" H 6750 2250 50  0001 C CNN
 	1    6750 2250
@@
 	5200 1600 5200 1900
 Connection ~ 4950 1600
+Text Notes 5950 2800 0    50   ~ 0
+150mA MAX
 $EndSCHEMATC

Commit message: schemos paruosimas
Parts:
- J14, J16, J17, J18: symbol conn:Conn_01x01 -> ihouse-rescue:Conn_01x01-conn
Connections:
- net labels added: NEX_5VDC, NEX_COM
Other:
- moved on the sheet: C10, C11, C12, C4, C5, C6, C7, C8, C9, D16, D17, D18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

Commit message: tarpinis kommitas
Parts:
- C10, C11, C12, C4, C5, C6, C7, C8, C9: symbol Device:C -> ihouse-rescue:C-Device
- D16, D17, D18: symbol Device:LED -> ihouse-rescue:LED-Device
- TH2: symbol Device:Thermistor_NTC -> ihouse-rescue:Thermistor_NTC-Device
Changed lines of the file:
@@
 Connection ~ 5600 6000
 $Comp
-L Device:C C5
+L ihouse-rescue:C-Device C5
 U 1 1 5C5DAC7B
 P 4500 5050
@@
 	4400 5200 4500 5200
 $Comp
-L Device:C C4
+L ihouse-rescue:C-Device C4
 U 1 1 5C5DAC7C
 P 2700 5050
@@
 	2700 5200 2800 5200
 $Comp
-L Device:C C8
+L ihouse-rescue:C-Device C8
 U 1 1 5C5DAC7D
 P 4650 5400
@@
 	4500 5400 4400 5400
 $Comp
-L Device:C C10
+L ihouse-rescue:C-Device C10
 U 1 1 5C5DAC7F
 P 4650 5700
@@
 	5450 2950 5350 2950
 $Comp
-L Device:C C6
+L ihouse-rescue:C-Device C6
 U 1 1 5DF2F8F2
 P 5350 1500
@@
 $EndComp
 $Comp
-L Device:C C7
+L ihouse-rescue:C-Device C7
 U 1 1 5C5DAC99
 P 7150 1500
@@
 $EndComp
 $Comp
-L Device:C C9
+L ihouse-rescue:C-Device C9
 U 1 1 5DF2FB58
 P 5200 1850
@@
 $EndComp
 $Comp
-L Device:C C11
+L ihouse-rescue:C-Device C11
 U 1 1 5C5DAC9B
 P 5200 2150
@@
 	7050 2950 7250 2950
 $Comp
-L Device:Thermistor_NTC TH2
+L ihouse-rescue:Thermistor_NTC-Device TH2
 U 1 1 5C5DACB1
 P 3600 1250
@@
 $EndComp
 $Comp
-L Device:LED D16
+L ihouse-rescue:LED-Device D16
 U 1 1 5C5DACB5
 P 2150 5550
@@
 $EndComp
 $Comp
-L Device:LED D17
+L ihouse-rescue:LED-Device D17
 U 1 1 5C5DACB6
 P 2400 5550
@@
 	2400 5400 2400 4900
 $Comp
-L Device:LED D18
+L ihouse-rescue:LED-Device D18
 U 1 1 5F57F66C
 P 3800 2100
@@
 $EndComp
 $Comp
-L Device:C C12
+L ihouse-rescue:C-Device C12
 U 1 1 5CC72503
 P 5600 4950
