File: Kicad/ihouse_new/ihouse_new.kicad_pcb (KiCad board)
At the start: 2 copper layers, 51 parts, among them U1 PCF8583T, U10 MOC3063M, U11 MOC3063M, U12 MOC3063M, U2 MCP23017-E_SO, U3 L293D, U4 L293D, U5 MOC3063M, U6 MOC3063M, U7 MOC3063M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

Commit message: schemos paruosimas
Parts:
- removed R10, R15, R16, R17, R18, R7, R8, R9: 300, Resistor_SMD:R_0805_2012Metric_Pad1.15x1.40mm_HandSolder
- removed RN2, RN4: R_Pack04, Resistor_SMD:R_Array_Convex_4x1206
- added D11: BAS32, Diode_SMD:D_MiniMELF, F.Cu at (216.2, 95.5)
- added D12: Z0103MN, Package_TO_SOT_SMD:SOT-223, F.Cu at (145.2, 121.3)
- added J1: Valve 1, Connector_Molex:Molex_KK-254_AE-6410-02A_1x02_P2.54mm_Vertical, F.Cu at (133.5, 85.0)
- added J2: Valve 1, Connector_Molex:Molex_KK-254_AE-6410-02A_1x02_P2.54mm_Vertical, F.Cu at (141.5, 85.0)
- added J3: Valve 1, Connector_Molex:Molex_KK-254_AE-6410-02A_1x02_P2.54mm_Vertical, F.Cu at (156.0, 85.0)
- added J4: Valve 1, Connector_Molex:Molex_KK-254_AE-6410-02A_1x02_P2.54mm_Vertical, F.Cu at (164.5, 85.0)
- added K1: FINDER-32.21-x000, Relay_THT:Relay_SPDT_Finder_34.51_Vertical, F.Cu at (222.0, 103.8)
- added Q1: BC817, Package_TO_SOT_SMD:SOT-23, F.Cu at (222.0, 95.2)
- added R23: 10k, Resistor_SMD:R_0805_2012Metric_Pad1.15x1.40mm_HandSolder, F.Cu at (221.0, 91.2)
- added R24: 1k, Resistor_SMD:R_0805_2012Metric_Pad1.15x1.40mm_HandSolder, F.Cu at (223.0, 91.2)
- added R27: 470, Resistor_SMD:R_0805_2012Metric_Pad1.15x1.40mm_HandSolder, F.Cu at (147.7, 114.6)
- added R29: 470, Resistor_SMD:R_0805_2012Metric_Pad1.15x1.40mm_HandSolder, F.Cu at (177.5, 96.2)
- added U13: MOC3063M, Package_DIP:DIP-6_W7.62mm_SMDSocket_SmallPads, F.Cu at (145.2, 107.6)
- D1: value BAS32 -> BAS85
- moved U4 55.0 mm to (154.0, 97.9), turned to 90 degrees
- moved U3 54.8 mm to (131.0, 98.0), turned to 90 degrees
- moved D10 51.5 mm to (153.5, 121.3)
- moved D3 51.5 mm to (212.9, 121.3)
- moved D4 51.5 mm to (204.8, 121.3)
- moved D5 51.5 mm to (196.2, 121.3)
- moved D6 51.5 mm to (187.8, 121.2)
- moved D7 51.5 mm to (179.0, 121.3)
- moved D8 51.5 mm to (170.5, 121.3)
- moved D9 51.5 mm to (162.0, 121.3)
- moved R11 51.5 mm to (215.7, 114.5)
- moved R12 51.5 mm to (207.2, 114.5)
- moved R13 51.5 mm to (198.8, 114.5)
- moved R14 51.5 mm to (190.2, 114.5)
- moved R19 51.5 mm to (181.5, 114.5)
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Connections:
- D10 pad 2: Net-(D10-Pad2) -> /ACL
- D10 pad 4: Net-(D10-Pad2) -> /ACL
- D3 pad 2: Net-(D3-Pad2) -> /ACL
- D3 pad 4: Net-(D3-Pad2) -> /ACL
- D4 pad 2: Net-(D4-Pad2) -> /ACL
- D4 pad 4: Net-(D4-Pad2) -> /ACL
- D5 pad 2: Net-(D5-Pad2) -> /ACL
- D5 pad 4: Net-(D5-Pad2) -> /ACL
- D6 pad 2: Net-(D6-Pad2) -> /ACL
- D6 pad 4: Net-(D6-Pad2) -> /ACL
- D7 pad 2: Net-(D7-Pad2) -> /ACL
- D7 pad 4: Net-(D7-Pad2) -> /ACL
- D8 pad 2: Net-(D8-Pad2) -> /ACL
- D8 pad 4: Net-(D8-Pad2) -> /ACL
- D9 pad 2: Net-(D9-Pad2) -> /ACL
- D9 pad 4: Net-(D9-Pad2) -> /ACL
- R11 pad 1: Net-(D3-Pad2) -> /ACL
- R12 pad 1: Net-(D4-Pad2) -> /ACL
- R13 pad 1: Net-(D5-Pad2) -> /ACL
- R14 pad 1: Net-(D6-Pad2) -> /ACL
- R19 pad 1: Net-(D7-Pad2) -> /ACL
- R20 pad 1: Net-(D8-Pad2) -> /ACL
- R21 pad 1: Net-(D9-Pad2) -> /ACL
- R22 pad 1: Net-(D10-Pad2) -> /ACL
- U10 pad 4: Net-(D8-Pad1) -> Net-(D8-Pad3)
- U11 pad 4: Net-(D9-Pad1) -> Net-(D9-Pad3)
- U12 pad 4: Net-(D10-Pad1) -> Net-(D10-Pad3)
- U2 pad 21: Net-(RN2-Pad4) -> /ACON
- U2 pad 23: Net-(RN2-Pad2) -> /MA
- U2 pad 24: Net-(RN2-Pad1) -> /MB
- U2 pad 25: Net-(RN4-Pad4) -> /M1ENA
- U2 pad 26: Net-(RN4-Pad3) -> /M2ENA
- U2 pad 27: Net-(RN4-Pad2) -> /M3ENA
- U2 pad 28: Net-(RN4-Pad1) -> /M4ENA
- U3 pad 10: /MA -> /MB
- U3 pad 15: /MB -> /MA
- U4 pad 10: /MA -> /MB
- U4 pad 15: /MB -> /MA
- U5 pad 4: Net-(D3-Pad1) -> Net-(D3-Pad3)
- U6 pad 4: Net-(D4-Pad1) -> Net-(D4-Pad3)
- U7 pad 4: Net-(D5-Pad1) -> Net-(D5-Pad3)
- U8 pad 4: Net-(D6-Pad1) -> Net-(D6-Pad3)
- U9 pad 4: Net-(D7-Pad1) -> Net-(D7-Pad3)
Routing:
- net /ACL: track 0.00 -> 193.1 mm, vias 0 -> 9
- net /MA: track 0.00 -> 58.9 mm, vias 0 -> 2
- net /MB: track 0.00 -> 57.5 mm, vias 0 -> 2
- net /OC9: track 0.00 -> 33.4 mm
- net /ACON: track 0.00 -> 29.1 mm
- net Net-(RN2-Pad4): track 26.5 -> 0.00 mm
- net +5V: track 35.0 -> 61.3 mm, vias 0 -> 2
- net Net-(RN2-Pad2): track 20.2 -> 0.00 mm
- net /M1ENA: track 0.00 -> 18.0 mm
- net Net-(RN2-Pad1): track 17.1 -> 0.00 mm
- net /M2ENA: track 0.00 -> 16.6 mm
- net /M3ENA: track 0.00 -> 15.1 mm
- net Net-(D11-Pad2): track 0.00 -> 13.8 mm, vias 0 -> 1
- net Net-(RN4-Pad4): track 12.7 -> 0.00 mm
- net /M4ENA: track 0.00 -> 12.5 mm
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Other:
- board outline added: 170 x 100 mm

Commit message: pcb plokstes projektavimas
Parts:
- BT1: moved to F.Cu
- moved J1 95.6 mm to (229.0, 87.0), turned to 270 degrees
- moved J2 88.0 mm to (229.0, 94.0), turned to 270 degrees
- moved J3 74.7 mm to (229.0, 101.0), turned to 270 degrees
- moved J4 68.5 mm to (229.0, 108.0), turned to 270 degrees
- moved C1 30.2 mm to (116.0, 92.0)
- moved D1 30.2 mm to (113.0, 87.0)
- moved D2 30.2 mm to (119.0, 87.0)
- moved R1 30.2 mm to (124.0, 92.0)
- moved R2 30.2 mm to (122.0, 92.0)
- moved R3 30.2 mm to (119.0, 92.0)
- moved U1 30.2 mm to (119.0, 98.0)
- moved Y1 30.2 mm to (112.0, 94.0)
- moved BT1 27.9 mm to (120.0, 113.1), turned to 0 degrees
- moved R29 1.48 mm to (176.8, 97.5)
Connections:
- net Net-(D10-Pad1) renamed /OC8O
- net Net-(D12-Pad1) renamed /OC9O
- net Net-(D3-Pad1) renamed /OC1O
- net Net-(D4-Pad1) renamed /UC2O
- net Net-(D5-Pad1) renamed /OC3O
- net Net-(D6-Pad1) renamed /OC4O
- net Net-(D7-Pad1) renamed /OC5O
- net Net-(D8-Pad1) renamed /OC6O
- net Net-(D9-Pad1) renamed /OC7O
Routing:
- net Net-(J1-Pad1): track 0.00 -> 110.5 mm
- net Net-(J1-Pad2): track 0.00 -> 109.2 mm
- net Net-(J2-Pad2): track 0.00 -> 102.9 mm, vias 0 -> 2
- net Net-(J4-Pad2): track 0.00 -> 96.3 mm
- net Net-(J2-Pad1): track 0.00 -> 95.3 mm
- net /SDA: track 8.98 -> 95.9 mm, vias 0 -> 2
- net Net-(J3-Pad1): track 0.00 -> 85.4 mm
- net /SCL: track 8.44 -> 93.1 mm, vias 0 -> 2
- net Net-(J4-Pad1): track 0.00 -> 83.9 mm
- net +15V: track 10.9 -> 84.7 mm, vias 1 -> 3
- net Net-(J3-Pad2): track 0.00 -> 69.6 mm
- net +5V: track 61.3 -> 127.7 mm, vias 2 -> 3
- net /M1ENA: track 18.0 -> 70.7 mm, vias 0 -> 1
- net /M3ENA: track 15.1 -> 49.9 mm, vias 0 -> 1
- net /M2ENA: track 16.6 -> 48.7 mm, vias 0 -> 1
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
Commit message: tarpinis kommitas
Parts:
- added B1: Conn_01x01, disc:Sold_Pad, B.Cu at (92.5, 47.0)
- added B1: Conn_01x01, disc:Sold_Pad, B.Cu at (200.0, 47.0)
- added B10: Conn_01x01, disc:Sold_Pad, B.Cu at (102.0, 47.0)
- added B11: Conn_01x01, disc:Sold_Pad, B.Cu at (99.0, 47.0)
- added B12: Conn_01x01, disc:Sold_Pad, B.Cu at (96.0, 47.0)
- added B14: Conn_01x01, disc:Sold_Pad, B.Cu at (105.0, 47.0)
- added B15: Conn_01x01, disc:Sold_Pad, B.Cu at (207.0, 47.0)
- added B2: Conn_01x01, disc:Sold_Pad, B.Cu at (192.0, 47.0)
- added B3: Conn_01x01, disc:Sold_Pad, B.Cu at (183.5, 47.0)
- added B4: Conn_01x01, disc:Sold_Pad, B.Cu at (175.0, 47.0)
- added B5: Conn_01x01, disc:Sold_Pad, B.Cu at (166.5, 47.0)
- added B6: Conn_01x01, disc:Sold_Pad, B.Cu at (158.0, 47.0)
- added B7: Conn_01x01, disc:Sold_Pad, B.Cu at (149.5, 47.0)
- added B8: Conn_01x01, disc:Sold_Pad, B.Cu at (141.0, 47.0)
- added B9: Conn_01x01, disc:Sold_Pad, B.Cu at (132.5, 47.0)
- added BG2: Conn_01x01, disc:Sold_Pad, B.Cu at (116.0, 47.0)
- added BP1: Conn_01x01, disc:Sold_Pad, B.Cu at (109.0, 47.0)
- added BP2: Conn_01x01, disc:Sold_Pad, B.Cu at (112.0, 47.0)
- added T1: Conn_01x01, disc:Sold_Pad, F.Cu at (200.0, -14.0)
- added T10: Conn_01x01, disc:Sold_Pad, F.Cu at (102.0, -14.0)
- added T11: Conn_01x01, disc:Sold_Pad, F.Cu at (99.0, -14.0)
- added T12: Conn_01x01, disc:Sold_Pad, F.Cu at (96.0, -14.0)
- added T14: Conn_01x01, disc:Sold_Pad, F.Cu at (105.0, -14.0)
- added T15: Conn_01x01, disc:Sold_Pad, F.Cu at (207.0, -14.0)
- added T2: Conn_01x01, disc:Sold_Pad, F.Cu at (192.0, -14.0)
- added T3: Conn_01x01, disc:Sold_Pad, F.Cu at (183.5, -14.0)
- added T4: Conn_01x01, disc:Sold_Pad, F.Cu at (175.0, -14.0)
- added T5: Conn_01x01, disc:Sold_Pad, F.Cu at (166.5, -14.0)
- added T6: Conn_01x01, disc:Sold_Pad, F.Cu at (158.0, -14.0)
- added T7: Conn_01x01, disc:Sold_Pad, F.Cu at (149.5, -14.0)
- added T8: Conn_01x01, disc:Sold_Pad, F.Cu at (141.0, -14.0)
- added T9: Conn_01x01, disc:Sold_Pad, F.Cu at (132.5, -14.0)
- added TG1: Conn_01x01, disc:Sold_Pad, F.Cu at (92.5, -14.0)
- added TG2: Conn_01x01, disc:Sold_Pad, F.Cu at (116.0, -14.0)
- added TH1: Thermistor_PTC, Varistor:RV_Disc_D7mm_W3.5mm_P5mm, F.Cu at (213.0, -24.0)
- added TP1: Conn_01x01, disc:Sold_Pad, F.Cu at (109.0, -14.0)
- added TP2: Conn_01x01, disc:Sold_Pad, F.Cu at (112.0, -14.0)
- moved K1 144.0 mm to (205.0, -39.2)
- moved BT1 143.0 mm to (103.0, -28.9)
- moved C1 143.0 mm to (99.0, -50.0)
- moved D1 143.0 mm to (96.0, -55.0)
- moved D10 143.0 mm to (136.5, -20.7)
- moved D11 143.0 mm to (199.2, -46.5)
- moved D12 143.0 mm to (128.2, -20.7)
- moved D2 143.0 mm to (102.0, -55.0)
- moved D3 143.0 mm to (195.9, -20.7)
- moved D4 143.0 mm to (187.8, -20.7)
- moved D5 143.0 mm to (179.2, -20.7)
- moved D6 143.0 mm to (170.8, -20.8)
- moved D7 143.0 mm to (162.0, -20.7)
- moved D8 143.0 mm to (153.5, -20.7)
- moved D9 143.0 mm to (145.0, -20.7)
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Connections:
- D10 pad 1: /OC8O -> Net-(D10-Pad1)
- D12 pad 1: /OC9O -> Net-(D12-Pad1)
- D3 pad 1: /OC1O -> Net-(D3-Pad1)
- D4 pad 1: /UC2O -> Net-(D4-Pad1)
- D5 pad 1: /OC3O -> Net-(D5-Pad1)
- D6 pad 1: /OC4O -> Net-(D6-Pad1)
- D7 pad 1: /OC5O -> Net-(D7-Pad1)
- D8 pad 1: /OC6O -> Net-(D8-Pad1)
- D9 pad 1: /OC7O -> Net-(D9-Pad1)
- K1 pad 11: /ACL -> Net-(K1-Pad11)
- K1 pad 12: Net-(K1-Pad12) -> /ACL
- K1 pad 14: Net-(K1-Pad14) -> Net-(K1-Pad11)
Routing:
- net /~RST: track 18.1 -> 138.9 mm, vias 0 -> 2
- net +15V: track 84.7 -> 132.8 mm
- net +5V: track 127.7 -> 164.6 mm
- net /~INT: track 6.77 -> 41.2 mm
- net /SCL: track 93.1 -> 126.1 mm
- net /SDA: track 95.9 -> 126.4 mm
- net GND: track 25.5 -> 0.00 mm, vias 2 -> 3
- net Net-(K1-Pad11): track 0.00 -> 13.4 mm
- net Net-(D9-Pad1): track 0.00 -> 11.6 mm
- net Net-(D8-Pad1): track 0.00 -> 11.6 mm
- net Net-(D7-Pad1): track 0.00 -> 11.6 mm
- net Net-(D10-Pad1): track 0.00 -> 11.6 mm
- net Net-(D12-Pad1): track 0.00 -> 11.4 mm
- net Net-(D6-Pad1): track 0.00 -> 11.3 mm
- net Net-(D5-Pad1): track 0.00 -> 11.3 mm
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- added copper zone on B.Cu, net GND
Other:
- board size 170 x 100 mm -> 170 x 186 mm
