File: Kicad/ihouse_new/ihouse_new.sch (KiCad schematic (older format))
At the start: 51 parts, among them U1 PCF8583T, U10 MOC3063M, U11 MOC3063M, U12 MOC3063M, U2 MCP23017-E_SO, U3 L293D, U4 L293D, U5 MOC3063M, U6 MOC3063M, U7 MOC3063M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

Commit message: schemos paruosimas
Parts:
- removed RN2, RN4: R_Pack04, Resistor_SMD:R_Array_Convex_4x1206, symbol Device:R_Pack04
- added D11: BAS32, Diode_SMD:D_MiniMELF, symbol Device:D
- added D12: Z0103MN, Package_TO_SOT_SMD:SOT-223, symbol Triac_Thyristor:Z0103MN
- added J1, J2, J3, J4: Valve 1, Connector_Molex:Molex_KK-254_AE-6410-02A_1x02_P2.54mm_Vertical, symbol Connector_Generic:Conn_01x02
- added K1: FINDER-32.21-x000, Relay_THT:Relay_SPDT_Finder_34.51_Vertical, symbol Relay:FINDER-32.21-x000
- added Q1: BC817, Package_TO_SOT_SMD:SOT-23, symbol Transistor_BJT:BC817
- added R23: 10k, Resistor_SMD:R_0805_2012Metric_Pad1.15x1.40mm_HandSolder, symbol Device:R
- added R24: 1k, Resistor_SMD:R_0805_2012Metric_Pad1.15x1.40mm_HandSolder, symbol Device:R
- added R25: 300, symbol Device:R
- added R27, R29: 470, Resistor_SMD:R_0805_2012Metric_Pad1.15x1.40mm_HandSolder, symbol Device:R
- added U13: MOC3063M, Package_DIP:DIP-6_W7.62mm_SMDSocket_SmallPads, symbol Relay_SolidState:MOC3063M
- D1: value BAS32 -> BAS85
- R10, R15, R16, R17, R18, R7, R8, R9: footprint Resistor_SMD:R_0805_2012Metric_Pad1.15x1.40mm_HandSolder -> (none)
- U1: symbol mylibrary:PCF8583T -> ihouse_new-rescue:PCF8583T-mylibrary
- U2: symbol dk_Interface-I-O-Expanders:MCP23017-E_SO -> ihouse_new-rescue:MCP23017-E_SO-dk_Interface-I-O-Expanders
Connections:
- net labels added: ACL, ACON, OC9
- wire segments 239 -> 296
Other:
- moved on the sheet: D10, D3, D4, D5, D6, D7, D8, D9, R10, R11, R12, R13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

Commit message: pcb plokstes projektavimas
Parts:
- U1: symbol ihouse_new-rescue:PCF8583T-mylibrary -> ihouse_new-rescue:PCF8583T-mylibrary-ihouse_new-rescue
- U2: symbol ihouse_new-rescue:MCP23017-E_SO-dk_Interface-I-O-Expanders -> ihouse_new-rescue:MCP23017-E_SO-dk_Interface-I-O-Expanders-ihouse_new-rescue
Connections:
- net labels added: OC1O, OC3O, OC4O, OC5O, OC6O, OC7O, OC8O, OC9O, UC2O
Changed lines of the file:
@@
 $EndDescr
 $Comp
-L ihouse_new-rescue:PCF8583T-mylibrary U1
+L ihouse_new-rescue:PCF8583T-mylibrary-ihouse_new-rescue U1
 U 1 1 5C779654
 P 2350 2150
@@
 ~INT
 $Comp
-L ihouse_new-rescue:MCP23017-E_SO-dk_Interface-I-O-Expanders U2
+L ihouse_new-rescue:MCP23017-E_SO-dk_Interface-I-O-Expanders-ihouse_new-rescue U2
 U 1 1 5C78068D
 P 2450 4350
@@
 Wire Wire Line
 	14450 4600 14550 4600
+Text Label 8600 6350 2    50   ~ 0
+OC1O
+Text Label 8600 7150 2    50   ~ 0
+UC2O
+Text Label 8600 7950 2    50   ~ 0
+OC3O
+Text Label 8600 8750 2    50   ~ 0
+OC4O
+Text Label 8600 9550 2    50   ~ 0
+OC5O
+Text Label 11200 6350 2    50   ~ 0
+OC6O
+Text Label 11200 7150 2    50   ~ 0
+OC7O
+Text Label 11200 7950 2    50   ~ 0
+OC8O
+Text Label 11200 8750 2    50   ~ 0
+OC9O
 $EndSCHEMATC

Commit message: tarpinis kommitas
Parts:
- added T1, T10, T11, T12, T14, T15, T2, T3, T4, T5, T6, T7, T8, T9, TG1, TG2, TP1, TP2: Conn_01x01, disc:Sold_Pad, symbol Connector_Generic:Conn_01x01
- added TH1: Thermistor_PTC, Varistor:RV_Disc_D7mm_W3.5mm_P5mm, symbol Device:Thermistor_PTC
- U1: symbol ihouse_new-rescue:PCF8583T-mylibrary-ihouse_new-rescue -> ihouse_new-rescue:PCF8583T-mylibrary-ihouse_new-rescue-ihouse_new-rescue
- U2: symbol ihouse_new-rescue:MCP23017-E_SO-dk_Interface-I-O-Expanders-ihouse_new-rescue -> ihouse_new-rescue:MCP23017-E_SO-dk_Interface-I-O-Expanders-ihouse_new-rescue-ihouse_new-rescue
Connections:
- net labels removed: OC1O, OC3O, OC4O, OC5O, OC6O, OC7O, OC8O, OC9O, UC2O
- wire segments 296 -> 315
