File: Kicad/ihouse_power/ihouse_power/ihouse_power.kicad_pcb (KiCad board)
At the start: 2 copper layers, 175 x 135 mm, 125 parts, among them J1 Conn_02x12_Top_Bottom, J10 Conn_02x05_Odd_Even, J11 Conn_01x06, J14 Optic, J15 Hum1, J16 Hum2, J17 Hum3, J18 Temp, J2 Conn_02x05_Top_Bottom, J3 230L, J4 230N, J5 Conn_01x16, J6 Conn_01x06, J7 Conn_02x05_Odd_Even, J8 Conn_01x16, J9 Conn_01x06, K1 FINDER-34.51, K10 FINDER-34.51, K11 FINDER-41.52, K12 FINDER-34.51, K13 FINDER-34.51, K14 FINDER-34.51, K2 FINDER-34.51, K3 FINDER-34.51, K4 FINDER-34.51, K5 FINDER-34.51, K6 FINDER-34.51, K7 FINDER-34.51, K8 FINDER-34.51, K9 FINDER-34.51, M1 stm32f1_module, M2 TB387, U1 ULN2004, U10 MAX232, U2 ULN2004, U3 L293D, U4 MCP23017_SO, U5 L7805, U6 EL814, U7 EL814, U8 EL814, U9 24LC32

Commit message: principines schemos, pcb ruosimas
Parts:
- added C22: C, Capacitor_SMD:C_0805_2012Metric_Pad1.15x1.40mm_HandSolder, B.Cu at (220.0, 149.8)
- added R34: R, Resistor_SMD:R_1206_3216Metric_Pad1.42x1.75mm_HandSolder, B.Cu at (195.0, 144.5)
- C2: footprint Capacitor_THT:CP_Radial_D4.0mm_P2.00mm -> Capacitor_SMD:CP_Elec_4x5.8; moved to B.Cu
- moved M2 128.9 mm to (201.4, 142.4), turned to 0 degrees
- moved J7 26.8 mm to (165.4, 77.0)
- moved D2 3.55 mm to (233.8, 151.0)
- moved >NAME 2.90 mm to (242.0, 30.4)
- moved C2 1.64 mm to (224.5, 148.4)
- moved >NAME 0.78 mm to (242.0, 34.1)
Connections:
- net Net-(J7-Pad6) renamed /MCU plokste/M1EN
- net Net-(J7-Pad8) renamed /MCU plokste/M2EN
- >NAME pad 1: (no net) -> /230L
- >NAME pad 1: (no net) -> /230N
- U4 pad 18: /MCP23017 modulis/~RST -> Net-(R34-Pad1)
Routing:
- net /MCP23017 modulis/~RST: track 75.6 -> 63.6 mm
- net Net-(R34-Pad1): track 0.00 -> 8.34 mm
- net GND: track 20.6 -> 14.4 mm, vias 6 -> 4
- net /MCP23017 modulis/GPB6: track 26.6 -> 23.0 mm
- net /MCP23017 modulis/GPB5: track 26.8 -> 23.4 mm
- net /MCP23017 modulis/GPB7: track 25.4 -> 22.5 mm
- net /MCP23017 modulis/GPB4: track 26.6 -> 23.8 mm
- net Net-(D2-Pad2): track 5.84 -> 3.22 mm
- net /MCP23017 modulis/GPB3: track 26.6 -> 24.2 mm
- net /MCP23017 modulis/5VDC1: track 62.4 -> 60.4 mm
- net /MCP23017 modulis/GPB2: track 26.6 -> 25.3 mm
- net /Reliu modulis/12VDC: track 21.6 -> 22.7 mm
- net /Reliu modulis/5VDC: track 33.5 -> 34.5 mm
- net /Reliu modulis/MA: track 70.2 -> 69.6 mm

Commit message: schemos ir pcb paruosimas
Parts:
- removed >NAME: 6, SparkFun_Connectors:1X01
- removed >NAME: 5, SparkFun_Connectors:1X01
- removed >NAME: 4, SparkFun_Connectors:1X01
- removed >NAME: 2, SparkFun_Connectors:1X01
- removed >NAME: 3, SparkFun_Connectors:1X01
- removed >NAME: 1, SparkFun_Connectors:1X01
- removed REF** (x8): MountingHole_3.2mm_M3, MountingHole:MountingHole_3.2mm_M3
- added J19: Conn_01x20, Connector_PinHeader_2.54mm:PinHeader_1x20_P2.54mm_Vertical, F.Cu at (107.8, 90.0)
- added J20: Conn_01x20, Connector_PinHeader_2.54mm:PinHeader_1x20_P2.54mm_Vertical, F.Cu at (107.8, 113.0)
- C2: footprint Capacitor_SMD:CP_Elec_4x5.8 -> Capacitor_SMD:CP_Elec_4x5.3
- J10, J7: value Conn_02x05_Odd_Even -> Conn_02x07_Odd_Even; footprint Connector_IDC:IDC-Header_2x05_P2.54mm_Vertical -> Connector_Multicomp:Multicomp_MC9A12-1434_2x07_P2.54mm_Vertical
- J11: footprint Connector_Molex:Molex_KK-254_AE-6410-06A_1x06_P2.54mm_Vertical -> Connector_PinHeader_2.54mm:PinHeader_1x06_P2.54mm_Vertical
- J3: value 230L -> Conn_01x20; footprint mech:Faston_6.3x0.8x14 -> Connector_PinHeader_2.54mm:PinHeader_1x20_P2.54mm_Vertical
- J4: value 230N -> Conn_01x20; footprint mech:Faston_6.3x0.8x14 -> Connector_PinHeader_2.54mm:PinHeader_1x20_P2.54mm_Vertical
- M2: value TB387 -> tb387_uart_expander
- moved J3 141.7 mm to (107.8, 86.0)
- moved J4 130.5 mm to (107.8, 117.0)
- moved J2 6.80 mm to (220.8, 121.0)
- moved BT1 6.33 mm to (94.8, 101.0)
- moved M1 5.36 mm to (107.8, 109.0)
- moved J10 3.03 mm to (235.7, 147.0), turned to 0 degrees
- moved C2 3.00 mm to (221.5, 148.4)
- moved C22 3.00 mm to (217.0, 149.8)
- moved D2 3.00 mm to (230.8, 151.0)
- moved D3 3.00 mm to (238.3, 140.2)
- moved J8 3.00 mm to (193.8, 135.0)
- moved J9 3.00 mm to (236.9, 135.0)
- moved M2 3.00 mm to (198.4, 142.4)
- moved R34 3.00 mm to (192.0, 144.5)
- moved U4 3.00 mm to (202.8, 145.0)
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Connections:
- BT1 pad 1: Net-(BT1-Pad1) -> /MCU plokste/VBAT
- BT1 pad 2: GND -> /MCU plokste/COM
- C10 pad 2: GND -> /MCU plokste/COM
- C11 pad 1: /MCU plokste/VB -> /MCU plokste/12VDC
- C11 pad 2: GND -> /MCU plokste/COM1
- C12 pad 2: GND -> /MCU plokste/COM
- C13 pad 2: GND -> /MCU plokste/COM
- C14 pad 2: GND -> /MCU plokste/COM
- C15 pad 2: GND -> /MCU plokste/COM
- C16 pad 2: GND -> /MCU plokste/COM
- C17 pad 2: GND -> /MCU plokste/COM
- C18 pad 2: GND -> /MCU plokste/COM
- C19 pad 2: GND -> /MCU plokste/COM
- C2 pad 2: GND -> /MCP23017 modulis/COM1
- C20 pad 2: GND -> /MCU plokste/COM
- C21 pad 2: GND -> /MCU plokste/COM
- C22 pad 2: GND -> /MCP23017 modulis/COM1
- C3 pad 2: GND -> /MCU plokste/COM
- C4 pad 2: GND -> /MCU plokste/COM
- C5 pad 2: GND -> /MCU plokste/COM
- C6 pad 1: GND -> /MCU plokste/COM
- D4 pad 1: /MCU plokste/VB -> /MCU plokste/12VDC
- D5 pad 1: /MCU plokste/VB -> /MCU plokste/12VDC
- F1 pad 1: Net-(F1-Pad1) -> /Reliu modulis/VACL
- F2 pad 1: Net-(F1-Pad1) -> /Reliu modulis/VACL
- J10 pad 10: GND -> /MCP23017 modulis/COM1
- J10 pad 9: GND -> /MCP23017 modulis/COM1
- J14 pad 3: GND -> /MCU plokste/COM1
- J15 pad 3: GND -> /MCU plokste/COM1
- J16 pad 3: GND -> /MCU plokste/COM1
- J17 pad 3: GND -> /MCU plokste/COM1
- J18 pad 3: GND -> /MCU plokste/COM1
- J2 pad 10: /Reliu modulis/K14N -> /Reliu modulis/VACL
- J2 pad 4: Net-(J2-Pad4) -> /Reliu modulis/K14N
- J2 pad 5: /Reliu modulis/K14L -> /230N
- J2 pad 9: Net-(J2-Pad9) -> /Reliu modulis/K14L
- J3 pad 1: Net-(F1-Pad1) -> /MCU plokste/3VDC
- J4 pad 1: /230N -> /MCU plokste/VBAT
- J7 pad 10: GND -> /MCU plokste/COM1
- J7 pad 4: /MCU plokste/5VDC -> +5V
- J7 pad 9: GND -> /MCU plokste/COM1
- J9 pad 3: GND -> /MCP23017 modulis/COM1
- J9 pad 4: GND -> /MCP23017 modulis/COM1
- M1 pad 1: Net-(BT1-Pad1) -> /MCU plokste/VBAT
- M1 pad 10: Net-(M1-Pad10) -> /MCU plokste/A5
- M1 pad 11: Net-(M1-Pad11) -> /MCU plokste/A6
- M1 pad 12: Net-(M1-Pad12) -> /MCU plokste/A7
- M1 pad 13: Net-(M1-Pad13) -> /MCU plokste/B0
- M1 pad 14: Net-(M1-Pad14) -> /MCU plokste/B1
- M1 pad 15: Net-(M1-Pad15) -> /MCU plokste/B10
- M1 pad 16: Net-(M1-Pad16) -> /MCU plokste/B11
- M1 pad 17: Net-(M1-Pad17) -> /MCU plokste/~RST
- M1 pad 18: Net-(M1-Pad18) -> /MCU plokste/3VDC
- M1 pad 19: GND -> /MCU plokste/COM
- M1 pad 2: Net-(M1-Pad2) -> /MCU plokste/C13
- M1 pad 20: GND -> /MCU plokste/COM
- M1 pad 22: GND -> /MCU plokste/COM
- M1 pad 24: Net-(M1-Pad24) -> /MCU plokste/B9
- M1 pad 25: Net-(M1-Pad25) -> /MCU plokste/B8
- M1 pad 28: Net-(M1-Pad28) -> /MCU plokste/B5
- M1 pad 29: Net-(M1-Pad29) -> /MCU plokste/B4
- M1 pad 3: Net-(M1-Pad3) -> /MCU plokste/C14
- M1 pad 30: Net-(M1-Pad30) -> /MCU plokste/B3
- M1 pad 31: Net-(M1-Pad31) -> /MCU plokste/A15
- M1 pad 32: Net-(M1-Pad32) -> /MCU plokste/A12
- M1 pad 33: Net-(M1-Pad33) -> /MCU plokste/A11
- M1 pad 34: /MCU plokste/D1RX -> /MCU plokste/A10
- M1 pad 35: /MCU plokste/D1TX -> /MCU plokste/A9
- M1 pad 36: Net-(M1-Pad36) -> /MCU plokste/A8
- M1 pad 37: Net-(M1-Pad37) -> /MCU plokste/B15
- M1 pad 38: Net-(M1-Pad38) -> /MCU plokste/B14
- M1 pad 39: Net-(M1-Pad39) -> /MCU plokste/B13
- M1 pad 4: Net-(M1-Pad4) -> /MCU plokste/C15
- M1 pad 40: Net-(M1-Pad40) -> /MCU plokste/B12
- M1 pad 5: Net-(M1-Pad5) -> /MCU plokste/A0
- M1 pad 6: Net-(M1-Pad6) -> /MCU plokste/A1
- M1 pad 7: /MCU plokste/D2TX -> /MCU plokste/TBTX
- M1 pad 8: /MCU plokste/D2RX -> /MCU plokste/TBRX
- M1 pad 9: Net-(M1-Pad9) -> /MCU plokste/A4
- M2 pad 1: +5V -> /MCP23017 modulis/COM
- M2 pad 2: GND -> /MCP23017 modulis/5VDC1
- M2 pad 3: /MCU plokste/D2TX -> /MCP23017 modulis/TBTX
- M2 pad 4: /MCU plokste/D2RX -> /MCP23017 modulis/TBRX
- M2 pad 5: /MCU plokste/TDCMD -> /MCP23017 modulis/TBCMD
- R12 pad 2: GND -> /MCU plokste/COM
- R2 pad 2: /MCU plokste/5VDC -> +5V
- R27 pad 2: GND -> /MCU plokste/COM
- R28 pad 2: GND -> /MCU plokste/COM
- R29 pad 2: GND -> /MCU plokste/COM
- R3 pad 2: /MCU plokste/5VDC -> +5V
- R30 pad 2: GND -> /MCU plokste/COM
- R33 pad 2: GND -> /MCU plokste/COM
- R4 pad 2: /MCU plokste/5VDC -> +5V
- TH2 pad 1: GND -> /MCU plokste/COM1
- U10 pad 11: /MCU plokste/D1TX -> /MCU plokste/A9
- U10 pad 12: /MCU plokste/D1RX -> /MCU plokste/A10
- U10 pad 15: GND -> /MCU plokste/COM
- U4 pad 10: GND -> /MCP23017 modulis/COM1
- U4 pad 15: GND -> /MCP23017 modulis/COM1
- U4 pad 16: GND -> /MCP23017 modulis/COM1
- U4 pad 17: GND -> /MCP23017 modulis/COM1
- U5 pad 2: GND -> /MCP23017 modulis/COM1
- U6 pad 3: GND -> /MCU plokste/COM
- U7 pad 3: GND -> /MCU plokste/COM
- U8 pad 3: GND -> /MCU plokste/COM
- U9 pad 1: GND -> /MCU plokste/COM
- U9 pad 2: GND -> /MCU plokste/COM
- U9 pad 3: GND -> /MCU plokste/COM
- U9 pad 4: GND -> /MCU plokste/COM
- U9 pad 7: GND -> /MCU plokste/COM
Routing:
- net /MCP23017 modulis/TBCMD: track 0.00 -> 65.3 mm, vias 0 -> 1
- net /MCP23017 modulis/TBRX: track 0.00 -> 58.9 mm, vias 0 -> 1
- net /MCP23017 modulis/TBTX: track 0.00 -> 56.6 mm, vias 0 -> 1
- net /Reliu modulis/VACL: track 0.00 -> 51.4 mm
- net Net-(F1-Pad1): track 50.6 -> 0.00 mm
- net /MCU plokste/VB: track 50.2 -> 0.00 mm
- net /MCU plokste/12VDC: track 0.00 -> 50.2 mm
- net +5V: track 2.18 -> 37.5 mm
- net /MCU plokste/5VDC: track 26.4 -> 0.00 mm
- net /MCP23017 modulis/5VDC1: track 60.4 -> 78.2 mm, vias 0 -> 1
- net /MCU plokste/3VDC: track 0.00 -> 16.0 mm
- net /Reliu modulis/M2B: track 19.9 -> 32.3 mm, vias 0 -> 2
- net /MCU plokste/B8: track 0.00 -> 8.23 mm
- net /Reliu modulis/K14N: track 15.9 -> 7.75 mm
- net /MCU plokste/SDA: track 0.00 -> 8.00 mm
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- added copper zone on B.Cu, net /MCP23017 modulis/COM1
- added copper zone on F.Cu, net /MCP23017 modulis/COM1
- added copper zone on B.Cu, net /MCU plokste/COM
- added copper zone on F.Cu, net /MCU plokste/COM
- removed copper zone on F.Cu, net GND
Other:
- outline, holes or cut-outs redrawn
- board text removed: "L"
- board text removed: "N"

Commit message: schemos ir pcb ruosimas
Parts:
- removed J19, J20: Conn_01x20, Connector_PinHeader_2.54mm:PinHeader_1x20_P2.54mm_Vertical
- removed TR2: Transformer_TEZ_22x24_6V, Transformer_THT:Transformer_Breve_TEZ-22x24
- added 1: SolderWirePad_1x01_Drill0.8mm, Connector_Wire:SolderWirePad_1x01_Drill0.8mm, F.Cu at (242.2, 27.2)
- added 2: SolderWirePad_1x01_Drill0.8mm, Connector_Wire:SolderWirePad_1x01_Drill0.8mm, F.Cu at (242.2, 30.7)
- added 3: SolderWirePad_1x01_Drill0.8mm, Connector_Wire:SolderWirePad_1x01_Drill0.8mm, F.Cu at (242.1, 34.1)
- added 4: SolderWirePad_1x01_Drill0.8mm, Connector_Wire:SolderWirePad_1x01_Drill0.8mm, F.Cu at (243.6, 38.0)
- added 5: SolderWirePad_1x01_Drill0.8mm, Connector_Wire:SolderWirePad_1x01_Drill0.8mm, F.Cu at (243.0, 92.4)
- added 6: SolderWirePad_1x01_Drill0.8mm, Connector_Wire:SolderWirePad_1x01_Drill0.8mm, F.Cu at (244.2, 106.0)
- added D10: D, Diode_SMD:D_MiniMELF, F.Cu at (140.7, 5.16)
- added D9: FR2J, Diode_SMD:D_SMB, F.Cu at (141.7, 0.76)
- added REF**: SolderWirePad_1x01_Drill0.8mm, Connector_Wire:SolderWirePad_1x01_Drill0.8mm, F.Cu at (97.9, 126.7)
- added REF**: MountingHole_3.2mm_M3, MountingHole:MountingHole_3.2mm_M3, F.Cu at (194.0, 126.0)
- added REF**: MountingHole_3.2mm_M3, MountingHole:MountingHole_3.2mm_M3, F.Cu at (254.0, 126.0)
- added REF**: MountingHole_3.2mm_M3, MountingHole:MountingHole_3.2mm_M3, F.Cu at (254.0, 26.0)
- added REF**: MountingHole_3.2mm_M3, MountingHole:MountingHole_3.2mm_M3, F.Cu at (194.0, 26.0)
- added REF**: SolderWirePad_1x01_Drill0.8mm, Connector_Wire:SolderWirePad_1x01_Drill0.8mm, F.Cu at (148.5, 122.4)
- added REF**: SolderWirePad_1x01_Drill0.8mm, Connector_Wire:SolderWirePad_1x01_Drill0.8mm, F.Cu at (135.9, 122.3)
- added REF**: SolderWirePad_1x01_Drill0.8mm, Connector_Wire:SolderWirePad_1x01_Drill0.8mm, F.Cu at (123.0, 119.7)
- added REF**: SolderWirePad_1x01_Drill0.8mm, Connector_Wire:SolderWirePad_1x01_Drill0.8mm, F.Cu at (133.2, 97.2)
- added REF**: MountingHole_3.2mm_M3, MountingHole:MountingHole_3.2mm_M3, F.Cu at (169.0, 26.0)
- added REF**: MountingHole_3.2mm_M3, MountingHole:MountingHole_3.2mm_M3, F.Cu at (89.0, 26.0)
- added REF**: MountingHole_3.2mm_M3, MountingHole:MountingHole_3.2mm_M3, F.Cu at (89.0, 126.0)
- added REF**: MountingHole_3.2mm_M3, MountingHole:MountingHole_3.2mm_M3, F.Cu at (169.0, 126.0)
- C10: footprint Capacitor_THT:CP_Radial_D5.0mm_P2.50mm -> Capacitor_THT:CP_Radial_D5.0mm_P2.00mm
- C6, C7, C8, C9, R8, R9, U10, U9: moved to B.Cu
- R10: value 1k -> R
- R11: value 120 -> R
- R12, R13: value R -> 100; moved to B.Cu
- moved U9 65.1 mm to (123.0, 100.5)
- moved C10 60.8 mm to (148.3, 1.26)
- moved R10 55.4 mm to (146.3, 6.01), turned to 0 degrees
- moved R11 55.1 mm to (151.0, 6.01), turned to 0 degrees
- moved R8 55.0 mm to (118.2, 97.8), turned to 270 degrees
- moved R9 50.3 mm to (116.1, 97.8), turned to 270 degrees
- moved R12 49.1 mm to (129.9, 100.0), turned to 180 degrees
- moved R13 48.5 mm to (129.9, 102.0), turned to 180 degrees
- moved C6 48.4 mm to (99.2, 93.2), turned to 180 degrees
- moved U10 42.4 mm to (97.6, 101.3), turned to 0 degrees
- moved C7 40.9 mm to (90.7, 99.1), turned to 0 degrees
- moved C9 40.4 mm to (90.7, 103.2), turned to 0 degrees
- moved C8 40.3 mm to (98.8, 109.2), turned to 0 degrees
- moved R31 37.9 mm to (97.2, 122.9)
- moved C13 37.7 mm to (99.7, 122.9)
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Connections:
- net /MCP23017 modulis/~RST renamed /MCP23017 modulis/~MCPRST
- BT1 pad 2: /MCU plokste/COM -> /MCU plokste/COM1
- C10 pad 2: /MCU plokste/COM -> /MCU plokste/COM1
- C12 pad 2: /MCU plokste/COM -> /MCU plokste/COM1
- C13 pad 2: /MCU plokste/COM -> /MCU plokste/COM1
- C14 pad 1: /MCU plokste/OPTIC -> /MCU plokste/A0
- C14 pad 2: /MCU plokste/COM -> /MCU plokste/COM1
- C15 pad 1: /MCU plokste/HUM1 -> /MCU plokste/A1
- C15 pad 2: /MCU plokste/COM -> /MCU plokste/COM1
- C16 pad 1: /MCU plokste/HUM2 -> /MCU plokste/A4
- C16 pad 2: /MCU plokste/COM -> /MCU plokste/COM1
- C17 pad 1: /MCU plokste/HUM3 -> /MCU plokste/A5
- C17 pad 2: /MCU plokste/COM -> /MCU plokste/COM1
- C18 pad 2: /MCU plokste/COM -> /MCU plokste/COM1
- C19 pad 2: /MCU plokste/COM -> /MCU plokste/COM1
- C20 pad 2: /MCU plokste/COM -> /MCU plokste/COM1
- C21 pad 1: /MCU plokste/TEMP -> /MCU plokste/A6
- C21 pad 2: /MCU plokste/COM -> /MCU plokste/COM1
- C3 pad 2: /MCU plokste/COM -> /MCU plokste/COM1
- C4 pad 2: /MCU plokste/COM -> /MCU plokste/COM1
- C5 pad 2: /MCU plokste/COM -> /MCU plokste/COM1
- C6 pad 1: /MCU plokste/COM -> /MCU plokste/COM1
- J3 pad 2: /MCU plokste/COM -> /MCU plokste/COM1
- J4 pad 19: /MCU plokste/COM -> /MCU plokste/COM1
- J4 pad 20: /MCU plokste/COM -> /MCU plokste/COM1
- J7 pad 7: /MCU plokste/~RST -> /MCU plokste/~MCPRST
- M1 pad 19: /MCU plokste/COM -> /MCU plokste/COM1
- M1 pad 20: /MCU plokste/COM -> /MCU plokste/COM1
- M1 pad 22: /MCU plokste/COM -> /MCU plokste/COM1
- R10 pad 1: Net-(R10-Pad1) -> Net-(C10-Pad1)
- R11 pad 2: Net-(C10-Pad1) -> /MCU plokste/COM1
- R12 pad 1: Net-(C10-Pad1) -> /MCU plokste/A9
- R12 pad 2: /MCU plokste/COM -> Net-(R12-Pad2)
- R13 pad 1: /MCU plokste/3VDC -> /MCU plokste/A10
- R13 pad 2: Net-(C10-Pad1) -> Net-(R13-Pad2)
- R23 pad 1: /MCU plokste/OPTIC -> /MCU plokste/A0
- R24 pad 1: /MCU plokste/HUM1 -> /MCU plokste/A1
- R25 pad 1: /MCU plokste/HUM2 -> /MCU plokste/A4
- R26 pad 1: /MCU plokste/HUM3 -> /MCU plokste/A5
- R27 pad 1: /MCU plokste/OPTIC -> /MCU plokste/A0
- R27 pad 2: /MCU plokste/COM -> /MCU plokste/COM1
- R28 pad 1: /MCU plokste/HUM1 -> /MCU plokste/A1
- R28 pad 2: /MCU plokste/COM -> /MCU plokste/COM1
- R29 pad 1: /MCU plokste/HUM2 -> /MCU plokste/A4
- R29 pad 2: /MCU plokste/COM -> /MCU plokste/COM1
- R30 pad 1: /MCU plokste/HUM3 -> /MCU plokste/A5
- R30 pad 2: /MCU plokste/COM -> /MCU plokste/COM1
- R32 pad 1: /MCU plokste/TEMP -> /MCU plokste/A6
- R33 pad 1: /MCU plokste/TEMP -> /MCU plokste/A6
- R33 pad 2: /MCU plokste/COM -> /MCU plokste/COM1
- R8 pad 1: +5V -> /MCU plokste/3VDC
- R9 pad 1: +5V -> /MCU plokste/3VDC
- U10 pad 11: /MCU plokste/A9 -> Net-(R12-Pad2)
- U10 pad 12: /MCU plokste/A10 -> Net-(R13-Pad2)
- U10 pad 15: /MCU plokste/COM -> /MCU plokste/COM1
- U6 pad 3: /MCU plokste/COM -> /MCU plokste/COM1
- U7 pad 3: /MCU plokste/COM -> /MCU plokste/COM1
- U8 pad 3: /MCU plokste/COM -> /MCU plokste/COM1
- U9 pad 1: /MCU plokste/COM -> /MCU plokste/COM1
- U9 pad 2: /MCU plokste/COM -> /MCU plokste/COM1
- U9 pad 3: /MCU plokste/COM -> /MCU plokste/COM1
- U9 pad 4: /MCU plokste/COM -> /MCU plokste/COM1
- U9 pad 7: /MCU plokste/COM -> /MCU plokste/COM1
Routing:
- net +5V: track 37.5 -> 102.8 mm
- net /MCU plokste/TBTX: track 7.99 -> 65.3 mm
- net /MCU plokste/SDA: track 8.00 -> 63.6 mm
- net /MCU plokste/SCK: track 8.00 -> 62.6 mm
- net /MCU plokste/TBRX: track 7.99 -> 60.0 mm
- net /MCU plokste/230N: track 92.9 -> 47.4 mm, vias 4 -> 2
- net Net-(R12-Pad2): track 0.00 -> 29.8 mm
- net Net-(R13-Pad2): track 0.00 -> 29.1 mm
- net /MCU plokste/A6: track 7.99 -> 35.6 mm
- net Net-(C10-Pad1): track 24.2 -> 0.00 mm, vias 1 -> 0
- net /MCU plokste/230L: track 54.4 -> 33.0 mm
- net /MCU plokste/A0: track 7.99 -> 27.5 mm
- net /MCU plokste/A5: track 7.99 -> 26.0 mm
- net /MCU plokste/VBAT: track 7.99 -> 25.9 mm, vias 0 -> 1
- net /MCU plokste/3VDC: track 16.0 -> 28.7 mm
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- added copper zone on B.Cu, net /MCU plokste/COM1
- added copper zone on F.Cu, net /MCU plokste/COM1
- removed copper zone on B.Cu, net /MCU plokste/COM
- removed copper zone on F.Cu, net /MCU plokste/COM

Commit message: schemos paruosimas
Parts:
- added C23: C, Capacitor_SMD:C_0805_2012Metric_Pad1.15x1.40mm_HandSolder, B.Cu at (149.7, 65.8)
- added C24: C, Capacitor_SMD:C_0805_2012Metric_Pad1.15x1.40mm_HandSolder, B.Cu at (151.5, 10.4)
- added C25: C, Capacitor_SMD:C_0805_2012Metric_Pad1.15x1.40mm_HandSolder, B.Cu at (138.7, 74.9)
- added C26: CP, Capacitor_THT:CP_Radial_D6.3mm_P2.50mm, F.Cu at (149.0, 73.3)
- added C27: C, Capacitor_SMD:C_0805_2012Metric_Pad1.15x1.40mm_HandSolder, B.Cu at (143.9, 101.2)
- added U11: L7805, Package_TO_SOT_SMD:SOT-223-3_TabPin2, B.Cu at (141.0, 68.2)
- D10, D9, R10, R11: moved to B.Cu
- moved D9 61.4 mm to (161.0, 59.1), turned to 180 degrees
- moved C10 60.8 mm to (166.9, 59.1)
- moved R10 59.8 mm to (163.2, 63.4), turned to 270 degrees
- moved R11 59.2 mm to (165.4, 63.4), turned to 90 degrees
Connections:
- D10 pad 2: /MCU plokste/VLINE -> /MCU plokste/A7
- R10 pad 2: /MCU plokste/VLINE -> /MCU plokste/A7
- R11 pad 1: /MCU plokste/VLINE -> /MCU plokste/A7

Commit message: schemos ir pcb ruosimas
Parts:
- added C28: CP, Capacitor_THT:CP_Radial_D4.0mm_P2.00mm, F.Cu at (345.8, 111.9)
- added C29: C, Capacitor_SMD:C_0805_2012Metric_Pad1.15x1.40mm_HandSolder, B.Cu at (341.1, 86.0)
- added J13: RC, rj45_vertical_shelded:RJ45_Vertical, F.Cu at (66.5, 93.6)
- added J19: I2C, Connector_JST:JST_XH_B04B-XH-A_1x04_P2.50mm_Vertical, F.Cu at (120.8, 72.3)
- added J20: Conn_02x05_Odd_Even, Connector_IDC:IDC-Header_2x05_P2.54mm_Vertical, F.Cu at (306.9, 87.9)
- added JP: 0R, Resistor_SMD:R_0805_2012Metric_Pad1.15x1.40mm_HandSolder, B.Cu at (91.0, 101.3)
- added JP: 0R, Resistor_SMD:R_0805_2012Metric_Pad1.15x1.40mm_HandSolder, B.Cu at (75.9, 96.8)
- added REF**: SolderWirePad_1x01_Drill0.8mm, Connector_Wire:SolderWirePad_1x01_Drill0.8mm, F.Cu at (125.3, 67.5)
- added REF**: SolderWirePad_1x01_Drill0.8mm, Connector_Wire:SolderWirePad_1x01_Drill0.8mm, F.Cu at (130.6, 110.0)
- added REF**: R_0805_2012Metric_Pad1.15x1.40mm_HandSolder, Resistor_SMD:R_0805_2012Metric_Pad1.15x1.40mm_HandSolder, B.Cu at (125.2, 81.8)
- added REF**: SolderWirePad_1x01_Drill0.8mm, Connector_Wire:SolderWirePad_1x01_Drill0.8mm, F.Cu at (177.8, 33.0)
- added REF**: SolderWirePad_1x01_Drill0.8mm, Connector_Wire:SolderWirePad_1x01_Drill0.8mm, F.Cu at (108.9, 75.7)
- added REF**: SolderWirePad_1x01_Drill0.8mm, Connector_Wire:SolderWirePad_1x01_Drill0.8mm, F.Cu at (65.2, 118.5)
- added REF**: SolderWirePad_1x01_Drill0.8mm, Connector_Wire:SolderWirePad_1x01_Drill0.8mm, F.Cu at (57.5, 124.0)
- added REF**: SolderWirePad_1x01_Drill0.8mm, Connector_Wire:SolderWirePad_1x01_Drill0.8mm, F.Cu at (66.7, 107.8)
- added REF**: R_0805_2012Metric_Pad1.15x1.40mm_HandSolder, Resistor_SMD:R_0805_2012Metric_Pad1.15x1.40mm_HandSolder, B.Cu at (68.6, 105.5)
- added REF**: R_0805_2012Metric_Pad1.15x1.40mm_HandSolder, Resistor_SMD:R_0805_2012Metric_Pad1.15x1.40mm_HandSolder, B.Cu at (68.6, 103.4)
- added REF**: R_1206_3216Metric_Pad1.42x1.75mm_HandSolder, Resistor_SMD:R_1206_3216Metric_Pad1.42x1.75mm_HandSolder, B.Cu at (170.8, 33.0)
- added REF**: SolderWirePad_1x01_Drill0.8mm, Connector_Wire:SolderWirePad_1x01_Drill0.8mm, F.Cu at (74.0, 121.6)
- added SW1: SW_SPST, Button_Switch_THT:SW_PUSH_6mm, F.Cu at (131.7, 100.0)
- added TH3: Thermistor_PTC, Resistor_THT:R_Axial_DIN0204_L3.6mm_D1.6mm_P5.08mm_Horizontal, F.Cu at (319.5, 82.7)
- added U12: MCP23017_SO, Package_SO:SOIC-28W_7.5x17.9mm_P1.27mm, B.Cu at (334.8, 115.6)
- added U13: L293D, Package_DIP:DIP-16_W7.62mm_LongPads, F.Cu at (329.9, 82.0)
- D9: value FR2J -> BAS85; footprint Diode_SMD:D_SMB -> Diode_SMD:D_MiniMELF
- J14, J15, J16, J17, J18: footprint Connector_JST:JST_EH_B03B-EH-A_1x03_P2.50mm_Vertical -> Connector_JST:JST_XH_B03B-XH-A_1x03_P2.50mm_Vertical
- R12, R13: value 100 -> 4.7k
- R34: value R -> 4.7k; footprint Resistor_SMD:R_1206_3216Metric_Pad1.42x1.75mm_HandSolder -> Resistor_SMD:R_0805_2012Metric_Pad1.15x1.40mm_HandSolder
- moved R12 212.0 mm to (341.1, 81.9), turned to 0 degrees
- moved R13 193.2 mm to (322.8, 113.4), turned to 0 degrees
- moved R34 133.5 mm to (322.8, 117.5), turned to 0 degrees
- moved C24 132.2 mm to (65.8, 111.1), turned to 90 degrees
- moved D10 114.4 mm to (122.6, 118.2), turned to 270 degrees
- moved M2 107.6 mm to (174.6, 37.0), turned to 270 degrees
- moved U4 105.8 mm to (172.0, 43.8), turned to 0 degrees
- moved C22 104.4 mm to (167.2, 58.0), turned to 0 degrees
- moved D2 102.3 mm to (166.0, 71.8), turned to 270 degrees
- moved J8 100.9 mm to (182.0, 34.8), turned to 0 degrees
- moved C2 100.9 mm to (168.6, 62.5), turned to 0 degrees
- moved J10 96.3 mm to (170.0, 76.7), turned to 270 degrees
- moved U5 94.8 mm to (171.5, 70.4), turned to 90 degrees
- moved D3 86.6 mm to (176.8, 79.3), turned to 180 degrees
- moved J9 79.2 mm to (182.0, 77.9), turned to 0 degrees
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Connections:
- net +5V renamed /MCU plokste/5VDC
- net /MCP23017 modulis/GPA7 renamed /MCP23017 modulis/M1ENA
- net /MCP23017 modulis/GPB7 renamed /MCP23017 modulis/M2ENA
- net /MCP23017 modulis/M1EN renamed /MCP23017 modulis/MA1
- net /MCP23017 modulis/M2EN renamed /MCP23017 modulis/MB1
- net /MCU plokste/B0 renamed /MCU plokste/PWM3
- net /MCU plokste/B1 renamed /MCU plokste/PWM4
- net /MCU plokste/B4 renamed /MCU plokste/PWM1
- net /MCU plokste/B5 renamed /MCU plokste/PWM2
- net GND renamed /Reliu modulis/COM1
- net Net-(U10-Pad9) renamed /MCU plokste/RCEN
- 1 pad 1: (no net) -> /K1.14
- 2 pad 1: (no net) -> /K1.11
- 3 pad 1: (no net) -> /K2.14
- 4 pad 1: (no net) -> /K2.11
- 5 pad 1: (no net) -> /230N
- 6 pad 1: (no net) -> Net-(F2-Pad2)
- J10 pad 11: /MCP23017 modulis/TBTX -> /MCP23017 modulis/TBCMD
- J10 pad 14: /MCP23017 modulis/TBCMD -> /MCP23017 modulis/TBTX
- J3 pad 17: /MCU plokste/B15 -> /MCU plokste/TBCMD
- J3 pad 18: /MCU plokste/B14 -> /MCU plokste/MB
- J3 pad 19: /MCU plokste/B13 -> /MCU plokste/MA
- J3 pad 20: /MCU plokste/B12 -> /MCU plokste/~MCPRST
- J5 pad 8: /Reliu modulis/MA -> /Reliu modulis/M1ENA
- J5 pad 9: /Reliu modulis/MB -> /Reliu modulis/M2ENA
- J6 pad 5: /Reliu modulis/M1ENA -> /Reliu modulis/MA
- J6 pad 6: /Reliu modulis/M2ENA -> /Reliu modulis/MB
- J7 pad 11: /MCU plokste/TBTX -> /MCU plokste/TBCMD
- J7 pad 14: /MCU plokste/TBCMD -> /MCU plokste/TBTX
- J7 pad 6: /MCU plokste/M1EN -> /MCU plokste/MA
- J7 pad 8: /MCU plokste/M2EN -> /MCU plokste/MB
- M1 pad 37: /MCU plokste/B15 -> /MCU plokste/TBCMD
- M1 pad 38: /MCU plokste/B14 -> /MCU plokste/MB
- M1 pad 39: /MCU plokste/B13 -> /MCU plokste/MA
- M1 pad 40: /MCU plokste/B12 -> /MCU plokste/~MCPRST
- M2 pad 1: /MCP23017 modulis/COM -> /MCP23017 modulis/COM1
- R12 pad 1: /MCU plokste/A9 -> /Papildomu IO modulis/5VDC
- R13 pad 1: /MCU plokste/A10 -> /Papildomu IO modulis/5VDC
- R13 pad 2: Net-(R13-Pad2) -> /Papildomu IO modulis/INTA
- R34 pad 1: Net-(R34-Pad1) -> /Papildomu IO modulis/5VDC
- R34 pad 2: /MCP23017 modulis/~MCPRST -> /Papildomu IO modulis/INTB
- U10 pad 11: Net-(R12-Pad2) -> /MCU plokste/A9
- U10 pad 12: Net-(R13-Pad2) -> /MCU plokste/A10
- U4 pad 18: Net-(R34-Pad1) -> /MCP23017 modulis/~MCPRST
Routing:
- net /MCU plokste/5VDC: track 102.8 -> 228.7 mm, vias 0 -> 4
- net /MCU plokste/12VDC: track 50.2 -> 161.3 mm
- net /MCU plokste/MB: track 0.00 -> 55.7 mm, vias 0 -> 2
- net /Reliu modulis/MB: track 84.9 -> 36.6 mm, vias 2 -> 0
- net /MCU plokste/MA: track 0.00 -> 48.2 mm, vias 0 -> 2
- net /Reliu modulis/M1ENA: track 17.8 -> 64.2 mm, vias 0 -> 2
- net /Reliu modulis/MA: track 69.6 -> 31.2 mm, vias 2 -> 0
- net /MCU plokste/A9: track 17.8 -> 56.1 mm
- net /MCU plokste/A10: track 15.1 -> 53.1 mm
- net /Reliu modulis/M2ENA: track 39.1 -> 76.8 mm, vias 0 -> 4
- net /MCU plokste/A7: track 7.99 -> 40.4 mm
- net Net-(R12-Pad2): track 29.8 -> 0.00 mm
- net Net-(R13-Pad2): track 29.1 -> 0.00 mm
- net /MCU plokste/TBCMD: track 0.00 -> 28.8 mm
- net /MCU plokste/~RST: track 7.99 -> 32.1 mm, vias 0 -> 2
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Other:
- board size 175 x 135 mm -> 212 x 110 mm

Commit message: schemos ir pcb paruosymas
Parts:
- added J21: Conn_02x02_Top_Bottom, Connector_Molex:Molex_Mini-Fit_Jr_5566-04A_2x02_P4.20mm_Vertical, F.Cu at (329.4, 116.5)
- added TH4: Thermistor_PTC, Resistor_SMD:R_1206_3216Metric_Pad1.42x1.75mm_HandSolder, B.Cu at (62.9, 116.7)
- TH2: footprint Resistor_SMD:R_1210_3225Metric -> Resistor_SMD:R_2816_7142Metric
- TH3: footprint Resistor_THT:R_Axial_DIN0204_L3.6mm_D1.6mm_P5.08mm_Horizontal -> Resistor_SMD:R_2816_7142Metric; moved to B.Cu
- moved C28 35.5 mm to (326.5, 82.1), turned to 180 degrees
- moved U12 32.9 mm to (317.0, 87.9)
- moved R34 31.3 mm to (325.5, 86.3), turned to 180 degrees
- moved R13 29.3 mm to (325.5, 84.3), turned to 180 degrees
- moved J20 22.3 mm to (314.5, 108.9)
- moved TH3 21.2 mm to (317.0, 103.8)
- moved R12 15.8 mm to (325.5, 79.5), turned to 180 degrees
- moved U13 9.36 mm to (327.8, 91.1)
- moved C29 5.88 mm to (335.4, 87.5), turned to 90 degrees
- moved TH2 3.93 mm to (78.5, 72.5), turned to 90 degrees
- moved REF** 2.82 mm to (67.6, 117.1)
Connections:
- C13 pad 1: /MCU plokste/5VDC -> Net-(C13-Pad1)
- R31 pad 1: /MCU plokste/5VDC -> Net-(C13-Pad1)
- U13 pad 11: /Papildomu IO modulis/M3B -> /Papildomu IO modulis/M4B
- U13 pad 14: /Papildomu IO modulis/M3A -> /Papildomu IO modulis/M4A
- U13 pad 3: /Papildomu IO modulis/M4A -> /Papildomu IO modulis/M3A
- U13 pad 6: /Papildomu IO modulis/M4B -> /Papildomu IO modulis/M3B
Routing:
- net Net-(C13-Pad1): track 0.00 -> 6.27 mm
- net /MCU plokste/VBAT: track 25.9 -> 27.9 mm
- net /MCU plokste/5VDC: track 228.7 -> 227.4 mm
- added copper zone on B.Cu, net /Papildomu IO modulis/COM
Other:
- board size 212 x 110 mm -> 293 x 110 mm
