File: Kicad/ihouse_power/ihouse_power/ihouse_power.kicad_pcb (KiCad board)
At the start: 2 copper layers, 293 x 110 mm, 164 parts, among them J1 Conn_02x12_Top_Bottom, J10 Conn_02x07_Odd_Even, J11 Conn_01x06, J13 RC, J14 Optic, J15 Hum1, J16 Hum2, J17 Hum3, J18 Temp, J19 I2C, J2 Conn_02x05_Top_Bottom, J20 Conn_02x05_Odd_Even, J21 Conn_02x02_Top_Bottom, J3 Conn_01x20, J4 Conn_01x20, J5 Conn_01x16, J6 Conn_01x06, J7 Conn_02x07_Odd_Even, J8 Conn_01x16, J9 Conn_01x06, K1 FINDER-34.51, K10 FINDER-34.51, K11 FINDER-41.52, K12 FINDER-34.51, K13 FINDER-34.51, K14 FINDER-34.51, K2 FINDER-34.51, K3 FINDER-34.51, K4 FINDER-34.51, K5 FINDER-34.51, K6 FINDER-34.51, K7 FINDER-34.51, K8 FINDER-34.51, K9 FINDER-34.51, M1 stm32f1_module, M2 tb387_uart_expander, SW1 SW_SPST, U1 ULN2004, U10 MAX232, U11 L7805, U12 MCP23017_SO, U13 L293D, U2 ULN2004, U3 L293D, U4 MCP23017_SO, U5 L7805, U6 EL814, U7 EL814, U8 EL814, U9 24LC32

Commit message: schemos ir pcb ruosimas
Parts:
- removed the REF** at (68.6, 105.5)
- removed the REF** at (68.6, 103.4)
- moved J13 1.50 mm to (65.0, 93.5)
Connections:
- net /MCP23017 modulis/M1ENA renamed /MCP23017 modulis/MA
- net /MCP23017 modulis/M2ENA renamed /MCP23017 modulis/MB
- net /MCP23017 modulis/MA1 renamed /MCP23017 modulis/M1EN
- net /MCP23017 modulis/MB1 renamed /MCP23017 modulis/M2EN
- net /MCU plokste/MA renamed /MCU plokste/M1ENA
- net /MCU plokste/MB renamed /MCU plokste/M2ENA
- J5 pad 8: /Reliu modulis/M1ENA -> /Reliu modulis/MA
- J5 pad 9: /Reliu modulis/M2ENA -> /Reliu modulis/MB
- J6 pad 5: /Reliu modulis/MA -> /Reliu modulis/M1ENA
- J6 pad 6: /Reliu modulis/MB -> /Reliu modulis/M2ENA
Routing:
- net /Reliu modulis/MB: track 36.6 -> 85.2 mm, vias 0 -> 2
- net /Reliu modulis/M1ENA: track 64.2 -> 16.9 mm, vias 2 -> 0
- net /Reliu modulis/MA: track 31.2 -> 71.1 mm, vias 0 -> 2
- net /Reliu modulis/M2ENA: track 76.8 -> 39.7 mm, vias 4 -> 0
- net /MCU plokste/5VDC: track 227.4 -> 229.6 mm, vias 4 -> 6
- net /MCU plokste/A10: track 53.1 -> 55.2 mm
- net /MCU plokste/A9: track 56.1 -> 58.1 mm
- net /MCU plokste/RSTX: track 20.3 -> 19.8 mm
- net /MCU plokste/RSRX: track 23.0 -> 22.5 mm
- net Net-(J13-Pad4): track 16.9 -> 16.4 mm

Commit message: plokstes pataisymai
Parts:
- moved REF** 0.54 mm to (125.1, 67.0)
Routing:
- net /MCU plokste/5VDC: track 229.6 -> 237.3 mm
- net /MCU plokste/M2ENA: track 55.7 -> 59.1 mm
- net /MCU plokste/M1ENA: track 48.2 -> 51.4 mm
