File: Kicad/ihouse_power/ihouse_power/ihouse_power.sch (KiCad schematic (older format))
At the start: 13 parts, among them J10 Conn_02x05_Odd_Even, J11 Conn_01x06, J12 Conn_01x06, J14 Optic, J15 Hum1, J16 Hum2, J17 Hum3, J18 Temp, J5 Conn_01x16, J6 Conn_01x06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

Commit message: principines schemos, pcb ruosimas
Connections:
- wire segments 139 -> 145
Changed lines of the file:
@@
 EESchema Schematic File Version 4
 LIBS:ihouse_power-cache
-EELAYER 26 0
+EELAYER 29 0
 EELAYER END
 $Descr A4 11693 8268
@@
 F24 "M2EN" I L 6900 4200 50
 F25 "COM1" U R 7800 4100 50
-F26 "12VDC" I L 6900 3900 50
+F26 "12VDC" I L 6900 3700 50
 F27 "12VDC1" O R 7800 3800 50
 F28 "5VDC1" O R 7800 3900 50
@@
 Wire Wire Line
 	6750 3900 6650 3900
-Connection ~ 6750 3900
 Wire Wire Line
 	6900 3600 5950 3600
@@
 Wire Wire Line
 	6750 4300 6900 4300
-Wire Wire Line
-	6750 3900 6900 3900
 Wire Wire Line
 	6650 4100 6900 4100
@@
 F3 "SDA" B R 3900 4100 50
 F4 "SCK" O R 3900 4000 50
-F5 "12VDC" O R 3900 3900 50
+F5 "12VDC" O R 3900 3700 50
 F6 "5VDC" O R 3900 3600 50
 F7 "COM" U R 3900 4300 50
@@
 F18 "VDDA" O L 3000 2300 50
 F19 "Temp" I L 3000 4200 50
+F20 "M1EN" O R 3900 3500 50
+F21 "M2EN" O R 3900 3400 50
 $EndSheet
 $Comp
@@
 Wire Wire Line
 	4200 3900 4300 3900
-Wire Wire Line
-	3900 3900 4200 3900
-Connection ~ 4200 3900
 Wire Wire Line
 	3900 3600 5000 3600
@@
 Wire Wire Line
 	2650 4100 2650 3650
+Connection ~ 2650 3650
+Wire Wire Line
+	3900 3700 4200 3700
+Connection ~ 4200 3700
+Wire Wire Line
+	3900 3500 5100 3500
+Wire Wire Line
+	5100 3500 5100 4100
+Wire Wire Line
+	5100 4100 4800 4100
+Wire Wire Line
+	3900 3400 5200 3400
+Wire Wire Line
+	5200 3400 5200 4200
+Wire Wire Line
+	5200 4200 4800 4200
+Wire Wire Line
+	6750 3700 6900 3700
 Wire Bus Line
 	5400 1400 5400 2450
 Wire Bus Line
 	10100 1400 10100 4150
-Connection ~ 2650 3650
+Connection ~ 6750 3700
 $EndSCHEMATC

Commit message: schemos ir pcb paruosimas
Parts:
- removed J10, J7: Conn_02x05_Odd_Even, Connector_IDC:IDC-Header_2x05_P2.54mm_Vertical, symbol Connector_Generic:Conn_02x05_Odd_Even
- added J10, J7: Conn_02x07_Odd_Even, Connector_Multicomp:Multicomp_MC9A12-1434_2x07_P2.54mm_Vertical, symbol Connector_Generic:Conn_02x07_Odd_Even
Connections:
- net labels removed: GND
- wire segments 145 -> 151
Other:
- moved on the sheet: J11, J12, J14, J15, J16, J17, J18

Commit message: schemos ir pcb ruosimas
Connections:
- net MCP23017 modulis/~RST renamed MCP23017 modulis/~MCPRST
- net MCU plokste/~RST renamed MCU plokste/~MCPRST
Changed lines of the file:
@@
 EESchema Schematic File Version 4
 LIBS:ihouse_power-cache
-EELAYER 26 0
+EELAYER 29 0
 EELAYER END
 $Descr A4 11693 8268
@@
 F16 "GPB7" O R 7800 2500 50
 F17 "GPA7" O R 7800 2400 50
-F18 "~RST" I L 6900 2800 50
-F19 "SCK" I L 6900 3000 50
-F20 "SDA" B L 6900 2900 50
-F21 "M1EN" I L 6900 3500 50
-F22 "M1ENA" O R 7800 4200 50
-F23 "M2ENA" O R 7800 4300 50
-F24 "M2EN" I L 6900 3600 50
-F25 "COM1" U L 6900 3700 50
-F26 "12VDC" I L 6900 3100 50
-F27 "12VDC1" O R 7800 3800 50
-F28 "5VDC1" O R 7800 3900 50
-F29 "5VDC" B L 6900 3400 50
-F30 "TBTX" O L 6900 4100 50
-F31 "TBRX" I L 6900 4000 50
-F32 "TBCMD" I L 6900 3900 50
-F33 "COM2" U R 7800 4100 50
+F18 "SCK" I L 6900 3000 50
+F19 "SDA" B L 6900 2900 50
+F20 "M1EN" I L 6900 3500 50
+F21 "M1ENA" O R 7800 4200 50
+F22 "M2ENA" O R 7800 4300 50
+F23 "M2EN" I L 6900 3600 50
+F24 "COM1" U L 6900 3700 50
+F25 "12VDC" I L 6900 3100 50
+F26 "12VDC1" O R 7800 3800 50
+F27 "5VDC1" O R 7800 3900 50
+F28 "5VDC" B L 6900 3400 50
+F29 "TBTX" O L 6900 4100 50
+F30 "TBRX" I L 6900 4000 50
+F31 "TBCMD" I L 6900 3900 50
+F32 "COM2" U R 7800 4100 50
+F33 "~MCPRST" I L 6900 2800 50
 $EndSheet
 $Comp
@@
 F0 "MCU plokste" 50
 F1 "mcu.sch" 50
-F2 "~RST" O R 3900 3650 50
-F3 "SDA" B R 3900 3550 50
-F4 "SCK" O R 3900 3450 50
-F5 "12VDC" O R 3900 3150 50
-F6 "5VDC" O R 3900 3050 50
-F7 "230L" I R 3900 1800 50
-F8 "230N" I R 3900 1900 50
-F9 "K1.14" I R 3900 2100 50
-F10 "K1.11" I R 3900 2000 50
-F11 "K2.14" I R 3900 2300 50
-F12 "K2.11" I R 3900 2200 50
-F13 "Optic" I L 3000 2450 50
-F14 "Hum1" I L 3000 2900 50
-F15 "Hum2" I L 3000 3350 50
-F16 "Hum3" I L 3000 3800 50
-F17 "VDDA" O L 3000 2350 50
-F18 "Temp" I L 3000 4250 50
-F19 "M1EN" O R 3900 2950 50
-F20 "M2EN" O R 3900 2850 50
-F21 "TBTX" O R 3900 3850 50
-F22 "TBRX" I R 3900 3950 50
-F23 "TBCMD" O R 3900 4050 50
-F24 "COM1" U L 3000 4350 50
-F25 "COM2" U R 3900 3750 50
+F2 "SDA" B R 3900 3550 50
+F3 "SCK" O R 3900 3450 50
+F4 "12VDC" O R 3900 3150 50
+F5 "5VDC" O R 3900 3050 50
+F6 "230L" I R 3900 1800 50
+F7 "230N" I R 3900 1900 50
+F8 "K1.14" I R 3900 2100 50
+F9 "K1.11" I R 3900 2000 50
+F10 "K2.14" I R 3900 2300 50
+F11 "K2.11" I R 3900 2200 50
+F12 "Optic" I L 3000 2450 50
+F13 "Hum1" I L 3000 2900 50
+F14 "Hum2" I L 3000 3350 50
+F15 "Hum3" I L 3000 3800 50
+F16 "VDDA" O L 3000 2350 50
+F17 "Temp" I L 3000 4250 50
+F18 "M1EN" O R 3900 2950 50
+F19 "M2EN" O R 3900 2850 50
+F20 "TBTX" O R 3900 3850 50
+F21 "TBRX" I R 3900 3950 50
+F22 "TBCMD" O R 3900 4050 50
+F23 "COM1" U L 3000 4350 50
+F24 "COM2" U R 3900 3750 50
+F25 "~MCPRST" O R 3900 3650 50
 $EndSheet
 Wire Wire Line
@@
 Wire Wire Line
 	5850 4200 6750 4200
+Wire Wire Line
+	5000 3750 5000 4150
+Wire Wire Line
+	6750 3700 6750 4200
 Wire Bus Line
 	5400 1400 5400 2450
 Wire Bus Line
 	10100 1400 10100 4150
-Wire Wire Line
-	5000 3750 5000 4150
-Wire Wire Line
-	6750 3700 6750 4200
 $EndSCHEMATC

Commit message: schemos ir pcb ruosimas
Parts:
- added J19: I2C, Connector_JST:JST_PH_B4B-PH-K_1x04_P2.00mm_Vertical, symbol Connector_Generic:Conn_01x04
- added J20: Conn_02x05_Odd_Even, Connector_IDC:IDC-Header_2x05_P2.54mm_Vertical, symbol Connector_Generic:Conn_02x05_Odd_Even
- J14, J15, J16, J17, J18: footprint Connector_JST:JST_EH_B03B-EH-A_1x03_P2.50mm_Vertical -> Connector_JST:JST_PH_B3B-PH-K_1x03_P2.00mm_Vertical
Connections:
- net MCP23017 modulis/GPA7 is gone; now on net MCP23017 modulis/M1ENA: J8.8 (Pin_8)
- net MCP23017 modulis/GPB7 is gone; now on net MCP23017 modulis/M2ENA: J8.9 (Pin_9)
- net MCP23017 modulis/M1ENA: no longer J9.5 (Pin_5)
- net MCP23017 modulis/M2ENA: no longer J9.6 (Pin_6)
- net MCP23017 modulis/TBCMD: now also J10.11 (Pin_11); no longer J10.14 (Pin_14)
- net MCP23017 modulis/TBTX: now also J10.14 (Pin_14); no longer J10.11 (Pin_11)
- net MCU plokste/5VDC: now also J19.1 (Pin_1)
- net MCU plokste/COM2: now also J19.4 (Pin_4)
- net MCU plokste/SCK: now also J19.2 (Pin_2)
- net MCU plokste/SDA: now also J19.3 (Pin_3)
- net MCU plokste/TBCMD: now also J7.11 (Pin_11); no longer J7.14 (Pin_14)
- net MCU plokste/TBTX: now also J7.14 (Pin_14); no longer J7.11 (Pin_11)
- net Reliu modulis/M1ENA: now also J5.8 (Pin_8); no longer J6.5 (Pin_5)
- net Reliu modulis/M2ENA: now also J5.9 (Pin_9); no longer J6.6 (Pin_6)
- net Reliu modulis/MA: now also J6.5 (Pin_5); no longer J5.8 (Pin_8)
- net Reliu modulis/MB: now also J6.6 (Pin_6); no longer J5.9 (Pin_9)
- net MCP23017 modulis/M1EN renamed MCP23017 modulis/MA1
- net MCP23017 modulis/M2EN renamed MCP23017 modulis/MB1
- net MCU plokste/M1EN renamed MCU plokste/MA
- net MCU plokste/M2EN renamed MCU plokste/MB
- net Reliu modulis/COM renamed Reliu modulis/COM2
- new net MCP23017 modulis/MA2: J9.5 (Pin_5)
- new net MCP23017 modulis/MB2: J9.6 (Pin_6)
- new net Papildomu IO modulis/12VDC: J20.1 (Pin_1), J20.2 (Pin_2)
- new net Papildomu IO modulis/5VDC: J20.4 (Pin_4)
- new net Papildomu IO modulis/COM: J20.10 (Pin_10), J20.9 (Pin_9)
- new net Papildomu IO modulis/MA: J20.6 (Pin_6)
- new net Papildomu IO modulis/MB: J20.8 (Pin_8)
- new net Papildomu IO modulis/SCK: J20.3 (Pin_3)
- new net Papildomu IO modulis/SDA: J20.5 (Pin_5)
- new net Papildomu IO modulis/~MCPRST: J20.7 (Pin_7)
Other:
- moved on the sheet: J10, J11, J12, J14, J15, J16, J17, J18, J5, J6, J7, J8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

Commit message: schemos ir pcb paruosymas
Changed lines of the file:
@@
 EESchema Schematic File Version 4
 LIBS:ihouse_power-cache
-EELAYER 29 0
+EELAYER 26 0
 EELAYER END
 $Descr A4 11693 8268
@@
 F22 "GPA5" O R 9600 5450 50
 F23 "GPA6" O R 9600 5550 50
-F24 "M3A" O R 9600 5750 50
-F25 "M3B" O R 9600 5850 50
-F26 "M4A" O R 9600 6000 50
-F27 "M4B" O R 9600 6100 50
-F28 "INTA" O L 8800 5600 50
-F29 "INTB" O L 8800 5700 50
+F24 "INTA" O L 8800 5600 50
+F25 "INTB" O L 8800 5700 50
 $EndSheet
 Wire Wire Line

Commit message: schemos ir pcb ruosimas
Connections:
- net MCP23017 modulis/MA1 is gone; now on net MCP23017 modulis/M1ENA: J10.6 (Pin_6)
- net MCP23017 modulis/MB1 is gone; now on net MCP23017 modulis/M2ENA: J10.8 (Pin_8)
- net MCP23017 modulis/M1ENA: no longer J8.8 (Pin_8)
- net MCP23017 modulis/M2ENA: no longer J8.9 (Pin_9)
- net Reliu modulis/M1ENA: now also J6.5 (Pin_5); no longer J5.8 (Pin_8)
- net Reliu modulis/M2ENA: now also J6.6 (Pin_6); no longer J5.9 (Pin_9)
- net Reliu modulis/MA: now also J5.8 (Pin_8); no longer J6.5 (Pin_5)
- net Reliu modulis/MB: now also J5.9 (Pin_9); no longer J6.6 (Pin_6)
- net MCP23017 modulis/MA2 renamed MCP23017 modulis/M1EN
- net MCP23017 modulis/MB2 renamed MCP23017 modulis/M2EN
- net MCU plokste/MA renamed MCU plokste/M1ENA
- net MCU plokste/MB renamed MCU plokste/M2ENA
- new net MCP23017 modulis/MA: J8.8 (Pin_8)
- new net MCP23017 modulis/MB: J8.9 (Pin_9)
Changed lines of the file:
@@
 EESchema Schematic File Version 4
 LIBS:ihouse_power-cache
-EELAYER 26 0
+EELAYER 29 0
 EELAYER END
 $Descr A4 11693 8268
@@
 F26 "COM2" U R 7800 3400 50
 F27 "~MCPRST" I L 6900 2100 50
-F28 "MA1" I L 6900 2800 50
-F29 "MA2" O R 7800 3500 50
-F30 "MB2" O R 7800 3600 50
-F31 "MB1" I L 6900 2900 50
-F32 "M2ENA" O R 7800 1800 50
-F33 "M1ENA" O R 7800 1700 50
+F28 "MB" O R 7800 1800 50
+F29 "MA" O R 7800 1700 50
+F30 "M1ENA" I L 6900 2800 50
+F31 "M1EN" O R 7800 3500 50
+F32 "M2EN" O R 7800 3600 50
+F33 "M2ENA" I L 6900 2900 50
 $EndSheet
 $Comp
@@
 F2 "12VDC" I L 8800 3100 50
 F3 "5VDC" I L 8800 3200 50
-F4 "M1ENA" I L 8800 1700 50
-F5 "M2ENA" I L 8800 1800 50
-F6 "MA" I L 8800 3500 50
-F7 "MB" I L 8800 3600 50
+F4 "M1ENA" I L 8800 3500 50
+F5 "M2ENA" I L 8800 3600 50
+F6 "MA" I L 8800 1700 50
+F7 "MB" I L 8800 1800 50
 F8 "REL1" I L 8800 1000 50
 F9 "REL2" I L 8800 1100 50
@@
 F22 "~MCPRST" O R 3500 2950 50
 F23 "COM1" U L 2600 3650 50
-F24 "MA" O R 3500 2250 50
-F25 "MB" O R 3500 2150 50
+F24 "M1ENA" O R 3500 2250 50
+F25 "M2ENA" O R 3500 2150 50
 $EndSheet
 Wire Wire Line

Commit message: programos rasymas, schemos ir pcb koregavimai. veikia stm bootloaderis per Demonstrator
Parts:
- removed J20: Conn_02x05_Odd_Even, Connector_IDC:IDC-Header_2x05_P2.54mm_Vertical, symbol Connector_Generic:Conn_02x05_Odd_Even
Connections:
- net MCP23017 modulis/M2EN renamed MCP23017 modulis/M23EN
- net MCP23017 modulis/M2ENA renamed MCP23017 modulis/M23ENA
- net MCP23017 modulis/TBCMD renamed MCP23017 modulis/~TBCMD
- net MCU plokste/M2ENA renamed MCU plokste/M23ENA
- net MCU plokste/TBCMD renamed MCU plokste/~TBCMD
- net Reliu modulis/M2ENA renamed Reliu modulis/M23ENA
Other:
- moved on the sheet: J19, J7
