File: Kicad/ihouse_power/ihouse_power/mcp_module.sch (KiCad schematic (older format))
At the start: 5 parts, among them U4 MCP23017_SO, U5 L7805

Commit message: principines schemos, pcb ruosimas
Parts:
- added C22: C, Capacitor_SMD:C_0805_2012Metric_Pad1.15x1.40mm_HandSolder, symbol Device:C
- added R34: R, Resistor_SMD:R_1206_3216Metric_Pad1.42x1.75mm_HandSolder, symbol Device:R
Connections:
- net 5VDC1: now also C22.1
- net COM: now also C22.2
- net ~RST: now also R34.2; no longer U4.18 (~RESET~)
- new net: R34.1, U4.18 (~RESET~)
Other:
- moved on the sheet: D3
Changed lines of the file:
@@
 EESchema Schematic File Version 4
 LIBS:ihouse_power-cache
-EELAYER 26 0
+EELAYER 29 0
 EELAYER END
 $Descr A4 11693 8268
@@
 	4800 2850 5050 2850
 Wire Wire Line
-	4800 3650 5050 3650
+	4650 3650 4700 3650
 Wire Wire Line
 	6450 3650 6650 3650
@@
 Text HLabel 6650 4650 2    50   UnSpc ~ 0
 COM1
-Text HLabel 4800 3650 0    50   Input ~ 0
+Text HLabel 4650 3650 0    50   Input ~ 0
 ~RST
 Text HLabel 4800 2850 0    50   Input ~ 0
@@
 Connection ~ 3500 3350
 Wire Wire Line
-	3500 3350 4350 3350
+	3500 3350 4050 3350
 $Comp
 L Device:CP C2
@@
 Connection ~ 4350 3350
 Wire Wire Line
-	4350 2800 4200 2800
+	4350 2800 4050 2800
 Connection ~ 4350 2800
 Wire Wire Line
@@
 L Device:D D3
 U 1 1 5C997522
-P 4050 2800
-F 0 "D3" H 4050 2676 50  0000 C CNN
-F 1 "BAS32" H 4050 2675 50  0001 C CNN
-F 2 "Diode_SMD:D_MiniMELF" H 4050 2800 50  0001 C CNN
-F 3 "~" H 4050 2800 50  0001 C CNN
-	1    4050 2800
+P 3800 2800
+F 0 "D3" H 3800 2676 50  0000 C CNN
+F 1 "BAS32" H 3800 2675 50  0001 C CNN
+F 2 "Diode_SMD:D_MiniMELF" H 3800 2800 50  0001 C CNN
+F 3 "~" H 3800 2800 50  0001 C CNN
+	1    3800 2800
 	-1   0    0    1
 $EndComp
 Wire Wire Line
-	3900 2800 2950 2800
+	3650 2800 2950 2800
+$Comp
+L Device:R R34
+U 1 1 5CA60758
+P 4850 3650
+F 0 "R34" V 4850 3650 50  0000 C CNN
+F 1 "R" V 4734 3650 50  0001 C CNN
+F 2 "Resistor_SMD:R_1206_3216Metric_Pad1.42x1.75mm_HandSolder" V 4780 3650 50  0001 C CNN
+F 3 "~" H 4850 3650 50  0001 C CNN
+	1    4850 3650
+	0    1    1    0
+$EndComp
+Wire Wire Line
+	5000 3650 5050 3650
+$Comp
+L Device:C C22
+U 1 1 5CAE4084
+P 4050 3100
+F 0 "C22" H 3800 3150 50  0000 L CNN
+F 1 "C" H 3800 3050 50  0000 L CNN
+F 2 "Capacitor_SMD:C_0805_2012Metric_Pad1.15x1.40mm_HandSolder" H 4088 2950 50  0001 C CNN
+F 3 "~" H 4050 3100 50  0001 C CNN
+	1    4050 3100
+	1    0    0    -1
+$EndComp
+Wire Wire Line
+	4050 2950 4050 2800
+Connection ~ 4050 2800
+Wire Wire Line
+	4050 2800 3950 2800
+Wire Wire Line
+	4050 3250 4050 3350
+Connection ~ 4050 3350
+Wire Wire Line
+	4050 3350 4350 3350
 $EndSCHEMATC

Commit message: schemos ir pcb paruosimas
Parts:
- added M2: tb387_uart_expander, uart_expander:TB387_UART_expander, symbol tb387:tb387_uart_expander
Connections:
- net labels added: COM2, TBCMD, TBRX, TBTX
- wire segments 52 -> 57
Changed lines of the file:
@@
 EESchema Schematic File Version 4
 LIBS:ihouse_power-cache
-EELAYER 29 0
+EELAYER 26 0
 EELAYER END
 $Descr A4 11693 8268
@@
 Text HLabel 6650 4350 2    50   Output ~ 0
 GPA7
-Text HLabel 6650 4650 2    50   UnSpc ~ 0
+Text HLabel 2950 3350 0    50   UnSpc ~ 0
 COM1
 Text HLabel 4650 3650 0    50   Input ~ 0
@@
 Text HLabel 6650 2450 2    50   Output ~ 0
 5VDC1
-Text HLabel 2950 3350 0    50   UnSpc ~ 0
-COM
 Text HLabel 4850 4900 0    50   Input ~ 0
 M1EN
@@
 Wire Wire Line
 	4050 3350 4350 3350
+$Comp
+L tb387:tb387_uart_expander M2
+U 1 1 5CB77400
+P 5350 5550
+F 0 "M2" H 5300 5850 60  0000 C CNN
+F 1 "tb387_uart_expander" H 6100 5400 60  0001 C CNN
+F 2 "uart_expander:TB387_UART_expander" H 5900 5100 60  0001 C CNN
+F 3 "" H 5400 5100 60  0001 C CNN
+	1    5350 5550
+	-1   0    0    -1
+$EndComp
+Wire Wire Line
+	5700 5750 6650 5750
+Wire Wire Line
+	5700 5650 6650 5650
+Wire Wire Line
+	5700 5550 6650 5550
+Wire Wire Line
+	5700 5450 6000 5450
+Wire Wire Line
+	5700 5350 6000 5350
+Text Label 6000 5450 2    50   ~ 0
+5VDC1
+Text Label 6000 5350 2    50   ~ 0
+COM
+Text HLabel 6650 5550 2    50   Output ~ 0
+TBTX
+Text HLabel 6650 5650 2    50   Input ~ 0
+TBRX
+Text HLabel 6650 5750 2    50   Input ~ 0
+TBCMD
+Text HLabel 6650 4650 2    50   UnSpc ~ 0
+COM2
 $EndSCHEMATC

Commit message: schemos ir pcb ruosimas
Connections:
- net labels added: ~MCPRST
- net labels removed: ~RST
Changed lines of the file:
@@
 EESchema Schematic File Version 4
 LIBS:ihouse_power-cache
-EELAYER 26 0
+EELAYER 29 0
 EELAYER END
 $Descr A4 11693 8268
@@
 	4800 2850 5050 2850
 Wire Wire Line
-	4650 3650 4700 3650
+	4100 3650 4700 3650
 Wire Wire Line
 	6450 3650 6650 3650
@@
 Text HLabel 2950 3350 0    50   UnSpc ~ 0
 COM1
-Text HLabel 4650 3650 0    50   Input ~ 0
-~RST
+Text HLabel 4100 3650 0    50   Input ~ 0
+~MCPRST
 Text HLabel 4800 2850 0    50   Input ~ 0
 SCK

Commit message: schemos paruosimas
Parts:
- M2: symbol tb387:tb387_uart_expander -> ihouse_power-rescue:tb387_uart_expander-tb387
Changed lines of the file:
@@
 EESchema Schematic File Version 4
 LIBS:ihouse_power-cache
-EELAYER 29 0
+EELAYER 26 0
 EELAYER END
 $Descr A4 11693 8268
@@
 	4050 3350 4350 3350
 $Comp
-L tb387:tb387_uart_expander M2
+L ihouse_power-rescue:tb387_uart_expander-tb387 M2
 U 1 1 5CB77400
 P 5350 5550

Commit message: schemos ir pcb ruosimas
Parts:
- removed R34: R, Resistor_SMD:R_1206_3216Metric_Pad1.42x1.75mm_HandSolder, symbol Device:R
Connections:
- net COM is gone; now on net COM1: M2.1 (VCC)
- net ~MCPRST: now also U4.18 (~RESET~)
- net GPA7 renamed M1ENA
- net GPB7 renamed M2ENA
Changed lines of the file:
@@
 EESchema Schematic File Version 4
 LIBS:ihouse_power-cache
-EELAYER 26 0
+EELAYER 29 0
 EELAYER END
 $Descr A4 11693 8268
 encoding utf-8
-Sheet 2 4
+Sheet 2 5
 Title ""
 Date ""
@@
 Wire Wire Line
 	4800 2850 5050 2850
-Wire Wire Line
-	4100 3650 4700 3650
 Wire Wire Line
 	6450 3650 6650 3650
@@
 Text Label 6650 2750 2    50   ~ 0
 GPB0
-Text Label 6650 4350 2    50   ~ 0
-MA
-Text Label 6650 3450 2    50   ~ 0
-MB
 Text HLabel 6650 2750 2    50   Output ~ 0
 GPB0
@@
 GPA6
 Text HLabel 6650 3450 2    50   Output ~ 0
-GPB7
+M2ENA
 Text HLabel 6650 4350 2    50   Output ~ 0
-GPA7
+M1ENA
 Text HLabel 2950 3350 0    50   UnSpc ~ 0
 COM1
-Text HLabel 4100 3650 0    50   Input ~ 0
+Text HLabel 4800 3650 0    50   Input ~ 0
 ~MCPRST
 Text HLabel 4800 2850 0    50   Input ~ 0
@@
 5VDC1
 Text HLabel 4850 4900 0    50   Input ~ 0
-M1EN
+MA1
 Text HLabel 6650 4900 2    50   Output ~ 0
-M1ENA
+MA2
 Text HLabel 6650 5000 2    50   Output ~ 0
-M2ENA
+MB2
 Text HLabel 4850 5000 0    50   Input ~ 0
-M2EN
+MB1
 Wire Wire Line
 	4850 4900 6650 4900
@@
 Wire Wire Line
 	3650 2800 2950 2800
-$Comp
-L Device:R R34
-U 1 1 5CA60758
-P 4850 3650
-F 0 "R34" V 4850 3650 50  0000 C CNN
-F 1 "R" V 4734 3650 50  0001 C CNN
-F 2 "Resistor_SMD:R_1206_3216Metric_Pad1.42x1.75mm_HandSolder" V 4780 3650 50  0001 C CNN
-F 3 "~" H 4850 3650 50  0001 C CNN
-	1    4850 3650
-	0    1    1    0
-$EndComp
-Wire Wire Line
-	5000 3650 5050 3650
 $Comp
 L Device:C C22
@@
 Text HLabel 6650 4650 2    50   UnSpc ~ 0
 COM2
+Text Label 5400 4650 2    50   ~ 0
+COM
+Wire Wire Line
+	4800 3650 5050 3650
 $EndSCHEMATC

Commit message: schemos ir pcb ruosimas
Connections:
- net M1ENA renamed MA
- net M2ENA renamed MB
Changed lines of the file:
@@
 EESchema Schematic File Version 4
 LIBS:ihouse_power-cache
-EELAYER 26 0
+EELAYER 29 0
 EELAYER END
 $Descr A4 11693 8268
@@
 GPA6
 Text HLabel 6650 3450 2    50   Output ~ 0
-M2ENA
+MB
 Text HLabel 6650 4350 2    50   Output ~ 0
-M1ENA
+MA
 Text HLabel 2950 3350 0    50   UnSpc ~ 0
 COM1
@@
 5VDC1
 Text HLabel 4850 4900 0    50   Input ~ 0
-MA1
+M1ENA
 Text HLabel 6650 4900 2    50   Output ~ 0
-MA2
+M1EN
 Text HLabel 6650 5000 2    50   Output ~ 0
-MB2
+M2EN
 Text HLabel 4850 5000 0    50   Input ~ 0
-MB1
+M2ENA
 Wire Wire Line
 	4850 4900 6650 4900

Commit message: programos rasymas, schemos ir pcb koregavimai. veikia stm bootloaderis per Demonstrator
Connections:
- net TBCMD renamed ~TBCMD
Changed lines of the file:
@@
 $Descr A4 11693 8268
 encoding utf-8
-Sheet 2 5
+Sheet 2 4
 Title ""
 Date ""
@@
 M1EN
 Text HLabel 6650 5000 2    50   Output ~ 0
-M2EN
+M23EN
 Text HLabel 4850 5000 0    50   Input ~ 0
-M2ENA
+M23ENA
 Wire Wire Line
 	4850 4900 6650 4900
@@
 P 5350 5550
 F 0 "M2" H 5300 5850 60  0000 C CNN
-F 1 "tb387_uart_expander" H 6100 5400 60  0001 C CNN
+F 1 "tb387_uart_expander" H 5300 5200 60  0000 C CNN
 F 2 "uart_expander:TB387_UART_expander" H 5900 5100 60  0001 C CNN
 F 3 "" H 5400 5100 60  0001 C CNN
@@
 TBRX
 Text HLabel 6650 5750 2    50   Input ~ 0
-TBCMD
+~TBCMD
 Text HLabel 6650 4650 2    50   UnSpc ~ 0
 COM2
