File: Kicad/ihouse_power/ihouse_power/mcp_module.sch (KiCad schematic (older format))
At the start: 7 parts, among them M2 tb387_uart_expander, U4 MCP23017_SO, U5 L7805

Commit message: schemos korekcijos ir ploksciu paruosimas
Connections:
- net SCK renamed SCL
Changed lines of the file:
@@
 ~MCPRST
 Text HLabel 4800 2850 0    50   Input ~ 0
-SCK
+SCL
 Text HLabel 4800 2750 0    50   BiDi ~ 0
 SDA
