File: Kicad/ihouse_power/ihouse_power/mcu.sch (KiCad schematic (older format))
At the start: 68 parts, among them J13 RC, M1 stm32f1_module, M2 TB387, U10 MAX232, U6 EL814, U7 EL814, U8 EL814, U9 24LC32

Commit message: principines schemos, pcb ruosimas
Connections:
- net labels added: M1EN, M2EN
- wire segments 262 -> 264
Changed lines of the file:
@@
 EESchema Schematic File Version 4
 LIBS:ihouse_power-cache
-EELAYER 26 0
+EELAYER 29 0
 EELAYER END
 $Descr A3 16535 11693
@@
 Text Label 2700 10350 2    50   ~ 0
 TEMP
+Text HLabel 14700 2450 2    50   Output ~ 0
+M1EN
+Text HLabel 14700 2550 2    50   Output ~ 0
+M2EN
+Wire Wire Line
+	14700 2450 14400 2450
+Wire Wire Line
+	14700 2550 14400 2550
 $EndSCHEMATC

Commit message: schemos ir pcb paruosimas
Parts:
- removed M2: TB387, uart_expander:TB387_UART_expander, symbol tb387:tb387_uart_expander
- added C?: CP, Capacitor_THT:CP_Radial_D5.0mm_P2.00mm, symbol Device:CP
- added D?: FR2J, Diode_SMD:D_SMB, symbol Diode:1N4003
- added J19, J20, J3, J4: Conn_01x20, Connector_PinHeader_2.54mm:PinHeader_1x20_P2.54mm_Vertical, symbol Connector_Generic:Conn_01x20
- added R? (x2): R, Resistor_SMD:R_0805_2012Metric_Pad1.15x1.40mm_HandSolder, symbol ihouse_power-rescue:Device_R-ihouse-rescue-ihouse-rescue
- M1: symbol stm32f1_module:stm32f1_module -> ihouse_power-rescue:stm32f1_module-stm32f1_module
- TR1: symbol disc:TEZ8.0 -> ihouse_power-rescue:TEZ8.0-disc
- U10: symbol ics:MAX232 -> ihouse_power-rescue:MAX232-ics
Connections:
- net labels added: A0, A1, A10, A11, A12, A15, A2, A3, A4, A5, A6, A7, A8, A9, B0, B1, B10, B11, B12, B13, B14, B15, B3, B4, B5, B6, B7, B8, B9, C13, C14, C15, COM1, COM2, COM3, TBCMD, TBRX, TBTX, VBAT
- net labels removed: D2RX, D2TX, TDCMD, VB
- wire segments 264 -> 380
Other:
- moved on the sheet: C11, R8, R9

Commit message: schemos ir pcb ruosimas
Parts:
- removed C10: CP, Capacitor_THT:CP_Radial_D5.0mm_P2.50mm, symbol Device:CP
- removed J19, J20: Conn_01x20, Connector_PinHeader_2.54mm:PinHeader_1x20_P2.54mm_Vertical, symbol Connector_Generic:Conn_01x20
- removed R10: 1k, Resistor_SMD:R_0805_2012Metric_Pad1.15x1.40mm_HandSolder, symbol ihouse_power-rescue:Device_R-ihouse-rescue-ihouse-rescue
- removed R11: 120, Resistor_SMD:R_0805_2012Metric_Pad1.15x1.40mm_HandSolder, symbol ihouse_power-rescue:Device_R-ihouse-rescue-ihouse-rescue
- removed R12, R13: R, Resistor_SMD:R_0805_2012Metric_Pad1.15x1.40mm_HandSolder, symbol ihouse_power-rescue:Device_R-ihouse-rescue-ihouse-rescue
- removed TR2: Transformer_TEZ_22x24_6V, Transformer_THT:Transformer_Breve_TEZ-22x24, symbol ihouse_power-rescue:disc_Transformer_TEZ_22x24_6V-ihouse-rescue-ihouse-rescue
- added D10: D, Diode_SMD:D_MiniMELF, symbol Device:D
- added R12, R13: 100, Resistor_SMD:R_0805_2012Metric_Pad1.15x1.40mm_HandSolder, symbol Device:R
- gave numbers to parts that had none: 4
Connections:
- net labels added: ~MCPRST
- wire segments 380 -> 321
Other:
- moved on the sheet: C10, C11, D4, D5, D9, R10, R11, TH2, TR1

Commit message: schemos paruosimas
Parts:
- added C23, C24, C25, C27: C, Capacitor_SMD:C_0805_2012Metric_Pad1.15x1.40mm_HandSolder, symbol Device:C
- added C26: CP, Capacitor_THT:CP_Radial_D6.3mm_P2.50mm, symbol Device:CP
- added U11: L7805, Package_TO_SOT_SMD:SOT-223-3_TabPin2, symbol Regulator_Linear:L7805
Connections:
- net labels removed: HUM1, HUM2, HUM3, OPTIC, TEMP
- wire segments 321 -> 346
Changed lines of the file:
@@
 EESchema Schematic File Version 4
 LIBS:ihouse_power-cache
-EELAYER 29 0
+EELAYER 26 0
 EELAYER END
 $Descr A3 16535 11693
@@
 Wire Wire Line
 	3800 4700 3900 4700
-Text Label 4500 4400 2    50   ~ 0
-D1TX
-Text Label 4500 4700 2    50   ~ 0
-D1RX
 Text Label 2300 4400 0    50   ~ 0
 RSTX
@@
 Wire Wire Line
 	2300 10200 2700 10200
-Text Label 2700 8150 2    50   ~ 0
-OPTIC
-Text Label 2700 8700 2    50   ~ 0
-HUM1
-Text Label 2700 9250 2    50   ~ 0
-HUM2
-Text Label 2700 9800 2    50   ~ 0
-HUM3
 Text HLabel 1350 7450 0    50   Output ~ 0
 VDDA
@@
 Wire Wire Line
 	2300 10750 2700 10750
-Text Label 2700 10350 2    50   ~ 0
-TEMP
 Text HLabel 14700 2450 2    50   Output ~ 0
 M1EN
@@
 Connection ~ 4500 1950
 Wire Wire Line
-	5150 1450 5450 1450
+	5150 1450 5400 1450
 Connection ~ 5150 1450
-Text Label 5450 1450 2    50   ~ 0
-VLINE
 Wire Wire Line
 	950  1750 1600 1750
@@
 Text Label 7300 5050 0    50   ~ 0
 ~RST
-Text Label 7150 5200 0    50   ~ 0
-OPTIC
-Text Label 7150 5300 0    50   ~ 0
-HUM1
-Text Label 7150 5600 0    50   ~ 0
-HUM2
-Text Label 7150 5700 0    50   ~ 0
-HUM3
-Text Label 7150 5800 0    50   ~ 0
-TEMP
 Text Label 12350 5000 0    50   ~ 0
 A0
-Text Label 7500 5200 0    50   ~ 0
+Text Label 7150 5200 0    50   ~ 0
 A0
-Text Label 7500 5300 0    50   ~ 0
+Text Label 7150 5300 0    50   ~ 0
 A1
-Text Label 7500 5600 0    50   ~ 0
+Text Label 7150 5600 0    50   ~ 0
 A4
-Text Label 7500 5700 0    50   ~ 0
+Text Label 7150 5700 0    50   ~ 0
 A5
-Text Label 7500 5800 0    50   ~ 0
+Text Label 7150 5800 0    50   ~ 0
 A6
+$Comp
+L Regulator_Linear:L7805 U11
+U 1 1 5CA0D926
+P 2600 2350
+F 0 "U11" H 2600 2592 50  0000 C CNN
+F 1 "L7805" H 2600 2501 50  0000 C CNN
+F 2 "Package_TO_SOT_SMD:SOT-223-3_TabPin2" H 2625 2200 50  0001 L CIN
+F 3 "http://www.st.com/content/ccc/resource/technical/document/datasheet/41/4f/b3/b0/12/d4/47/88/CD00000444.pdf/files/CD00000444.pdf/jcr:content/translations/en.CD00000444.pdf" H 2600 2300 50  0001 C CNN
+	1    2600 2350
+	1    0    0    -1
+$EndComp
+Wire Wire Line
+	2300 2350 2100 2350
+Text Label 1700 2350 0    50   ~ 0
+12VDC
+Wire Wire Line
+	1700 2750 2100 2750
+Wire Wire Line
+	2600 2750 2600 2650
+Wire Wire Line
+	2900 2350 3050 2350
+Wire Wire Line
+	2600 2750 3050 2750
+Connection ~ 2600 2750
+Text Label 1700 2750 0    50   ~ 0
+COM
+Text Label 4150 2750 2    50   ~ 0
+COM
+Text Label 4150 2350 2    50   ~ 0
+5VDC
+$Comp
+L Device:CP C26
+U 1 1 5CAA6900
+P 3850 2550
+F 0 "C26" H 4050 2600 50  0000 L CNN
+F 1 "CP" H 4050 2500 50  0000 L CNN
+F 2 "Capacitor_THT:CP_Radial_D6.3mm_P2.50mm" H 3888 2400 50  0001 C CNN
+F 3 "~" H 3850 2550 50  0001 C CNN
+	1    3850 2550
+	1    0    0    -1
+$EndComp
+Wire Wire Line
+	3850 2400 3850 2350
+Connection ~ 3850 2350
+Wire Wire Line
+	3850 2350 4150 2350
+Wire Wire Line
+	3850 2700 3850 2750
+Connection ~ 3850 2750
+Wire Wire Line
+	3850 2750 4150 2750
+$Comp
+L Device:C C24
+U 1 1 5CB232AD
+P 3050 2550
+F 0 "C24" H 3165 2596 50  0000 L CNN
+F 1 "C" H 3165 2505 50  0000 L CNN
+F 2 "Capacitor_SMD:C_0805_2012Metric_Pad1.15x1.40mm_HandSolder" H 3088 2400 50  0001 C CNN
+F 3 "~" H 3050 2550 50  0001 C CNN
+	1    3050 2550
+	1    0    0    -1
+$EndComp
+$Comp
+L Device:C C25
+U 1 1 5CB233A4
+P 3450 2550
+F 0 "C25" H 3565 2596 50  0000 L CNN
+F 1 "C" H 3565 2505 50  0000 L CNN
+F 2 "Capacitor_SMD:C_0805_2012Metric_Pad1.15x1.40mm_HandSolder" H 3488 2400 50  0001 C CNN
+F 3 "~" H 3450 2550 50  0001 C CNN
+	1    3450 2550
+	1    0    0    -1
+$EndComp
+Wire Wire Line
+	3050 2400 3050 2350
+Connection ~ 3050 2350
+Wire Wire Line
+	3050 2350 3450 2350
+Wire Wire Line
+	3050 2700 3050 2750
+Connection ~ 3050 2750
+Wire Wire Line
+	3050 2750 3450 2750
+Wire Wire Line
+	3450 2400 3450 2350
+Connection ~ 3450 2350
+Wire Wire Line
+	3450 2350 3850 2350
+Wire Wire Line
+	3450 2700 3450 2750
+Connection ~ 3450 2750
+Wire Wire Line
+	3450 2750 3850 2750
+$Comp
+L Device:C C23
+U 1 1 5CC22128
+P 2100 2550
+F 0 "C23" H 2215 2596 50  0000 L CNN
+F 1 "C" H 2215 2505 50  0000 L CNN
+F 2 "Capacitor_SMD:C_0805_2012Metric_Pad1.15x1.40mm_HandSolder" H 2138 2400 50  0001 C CNN
+F 3 "~" H 2100 2550 50  0001 C CNN
+	1    2100 2550
+	1    0    0    -1
+$EndComp
+Wire Wire Line
+	2100 2400 2100 2350
+Connection ~ 2100 2350
+Wire Wire Line
+	2100 2350 1700 2350
+Wire Wire Line
+	2100 2700 2100 2750
+Connection ~ 2100 2750
+Wire Wire Line
+	2100 2750 2600 2750
+$Comp
+L Device:C C27
+U 1 1 5CC65F8C
+P 5400 1700
+F 0 "C27" H 5515 1746 50  0000 L CNN
+F 1 "C" H 5515 1655 50  0000 L CNN
+F 2 "Capacitor_SMD:C_0805_2012Metric_Pad1.15x1.40mm_HandSolder" H 5438 1550 50  0001 C CNN
+F 3 "~" H 5400 1700 50  0001 C CNN
+	1    5400 1700
+	1    0    0    -1
+$EndComp
+Wire Wire Line
+	5150 1950 5400 1950
+Wire Wire Line
+	5400 1950 5400 1850
+Connection ~ 5150 1950
+Wire Wire Line
+	5400 1550 5400 1450
+Connection ~ 5400 1450
+Wire Wire Line
+	5400 1450 6000 1450
+Text Label 4500 4400 2    50   ~ 0
+A9
+Text Label 4500 4700 2    50   ~ 0
+A10
+Text Label 2700 8150 2    50   ~ 0
+A0
+Text Label 2700 8700 2    50   ~ 0
+A1
+Text Label 2700 9250 2    50   ~ 0
+A4
+Text Label 2700 9800 2    50   ~ 0
+A5
+Text Label 2700 10350 2    50   ~ 0
+A6
+Text Label 6000 1450 2    50   ~ 0
+A7
+Text Label 5550 1450 0    50   ~ 0
+VLINE
 $EndSCHEMATC

Commit message: schemos ir pcb ruosimas
Parts:
- removed R12, R13: 100, Resistor_SMD:R_0805_2012Metric_Pad1.15x1.40mm_HandSolder, symbol Device:R
- added SW1: SW_SPST, Button_Switch_THT:SW_PUSH_6mm, symbol Switch:SW_SPST
- D9: value FR2J -> BAS85; footprint Diode_SMD:D_SMB -> Diode_SMD:D_MiniMELF
- J13: footprint (none) -> rj45_vertical_shelded:RJ45_Vertical
Connections:
- net labels added: MA, MB, PWM1, PWM2, PWM3, PWM4
- net labels removed: +5V, D1RX, D1TX, M1EN, M2EN
- wire segments 346 -> 352
Other:
- moved on the sheet: BT1, C12, C13, C14, C15, C16, C17, C18, C19, C20, C21, R23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

Commit message: schemos ir pcb paruosymas
Parts:
- added TH4: Thermistor_PTC, Resistor_SMD:R_1206_3216Metric_Pad1.42x1.75mm_HandSolder, symbol Device:Thermistor_PTC
- TH2: footprint Resistor_SMD:R_1210_3225Metric -> Resistor_SMD:R_2816_7142Metric
Connections:
- net 5VDC: now also TH4.2; no longer C13.1, R31.1
- new net: C13.1, R31.1, TH4.1
Other:
- moved on the sheet: C12, C13, C19, C20, R31
Changed lines of the file:
@@
 EESchema Schematic File Version 4
 LIBS:ihouse_power-cache
-EELAYER 29 0
+EELAYER 26 0
 EELAYER END
 $Descr A3 16535 11693
@@
 F 0 "TH2" V 2200 1650 50  0000 C CNN
 F 1 "Thermistor_PTC" V 2151 1650 50  0001 C CNN
-F 2 "Resistor_SMD:R_1210_3225Metric" H 2400 1450 50  0001 L CNN
+F 2 "Resistor_SMD:R_2816_7142Metric" H 2400 1450 50  0001 L CNN
 F 3 "~" H 2350 1650 50  0001 C CNN
 	1    2350 1650
@@
 L Device:C C12
 U 1 1 5CBB980C
-P 2000 7250
-F 0 "C12" H 2115 7296 50  0000 L CNN
-F 1 "C" H 2115 7205 50  0000 L CNN
-F 2 "Capacitor_SMD:C_0805_2012Metric_Pad1.15x1.40mm_HandSolder" H 2038 7100 50  0001 C CNN
-F 3 "~" H 2000 7250 50  0001 C CNN
-	1    2000 7250
+P 1950 7250
+F 0 "C12" H 2065 7296 50  0000 L CNN
+F 1 "C" H 2065 7205 50  0000 L CNN
+F 2 "Capacitor_SMD:C_0805_2012Metric_Pad1.15x1.40mm_HandSolder" H 1988 7100 50  0001 C CNN
+F 3 "~" H 1950 7250 50  0001 C CNN
+	1    1950 7250
 	1    0    0    -1
 $EndComp
@@
 L Device:R R31
 U 1 1 5CBB9976
-P 3450 7000
-F 0 "R31" V 3450 6950 50  0000 L CNN
-F 1 "100" V 3550 6950 50  0001 L CNN
-F 2 "Resistor_SMD:R_0805_2012Metric_Pad1.15x1.40mm_HandSolder" V 3380 7000 50  0001 C CNN
-F 3 "~" H 3450 7000 50  0001 C CNN
-	1    3450 7000
-	0    1    1    0
-$EndComp
-Wire Wire Line
-	1750 7000 2000 7000
-Wire Wire Line
-	2000 7100 2000 7000
-Connection ~ 2000 7000
-Wire Wire Line
-	2000 7000 2400 7000
-Wire Wire Line
-	2000 7400 2000 7500
-Wire Wire Line
-	2000 7500 2400 7500
-Wire Wire Line
-	3600 7000 3750 7000
-Wire Wire Line
-	4150 7000 3750 7000
+P 3550 7000
+F 0 "R31" V 3550 6950 50  0000 L CNN
+F 1 "100" V 3650 6950 50  0001 L CNN
+F 2 "Resistor_SMD:R_0805_2012Metric_Pad1.15x1.40mm_HandSolder" V 3480 7000 50  0001 C CNN
+F 3 "~" H 3550 7000 50  0001 C CNN
+	1    3550 7000
+	0    1    1    0
+$EndComp
+Wire Wire Line
+	1950 7100 1950 7000
+Connection ~ 1950 7000
+Wire Wire Line
+	1950 7000 2400 7000
+Wire Wire Line
+	1950 7400 1950 7500
+Wire Wire Line
+	1950 7500 2400 7500
+Wire Wire Line
+	3700 7000 3800 7000
+Wire Wire Line
+	4600 7000 4300 7000
 $Comp
 L Device:C C13
 U 1 1 5CC3D68C
-P 3750 7250
-F 0 "C13" H 3865 7296 50  0000 L CNN
-F 1 "C" H 3865 7205 50  0000 L CNN
-F 2 "Capacitor_SMD:C_0805_2012Metric_Pad1.15x1.40mm_HandSolder" H 3788 7100 50  0001 C CNN
-F 3 "~" H 3750 7250 50  0001 C CNN
-	1    3750 7250
-	1    0    0    -1
-$EndComp
-Wire Wire Line
-	3750 7100 3750 7000
-Connection ~ 3750 7000
-Wire Wire Line
-	3750 7400 3750 7500
-Connection ~ 3750 7500
-Wire Wire Line
-	3750 7500 4150 7500
-Text Label 4150 7500 2    50   ~ 0
+P 3800 7250
+F 0 "C13" H 3915 7296 50  0000 L CNN
+F 1 "C" H 3915 7205 50  0000 L CNN
+F 2 "Capacitor_SMD:C_0805_2012Metric_Pad1.15x1.40mm_HandSolder" H 3838 7100 50  0001 C CNN
+F 3 "~" H 3800 7250 50  0001 C CNN
+	1    3800 7250
+	1    0    0    -1
+$EndComp
+Wire Wire Line
+	3800 7100 3800 7000
+Connection ~ 3800 7000
+Wire Wire Line
+	3800 7400 3800 7500
+Connection ~ 3800 7500
+Wire Wire Line
+	3800 7500 4600 7500
+Text Label 4600 7500 2    50   ~ 0
 COM
 $Comp
@@
 L Device:C C19
 U 1 1 5CCAD297
-P 2800 7250
-F 0 "C19" H 2915 7296 50  0000 L CNN
-F 1 "C" H 2915 7205 50  0000 L CNN
-F 2 "Capacitor_SMD:C_0805_2012Metric_Pad1.15x1.40mm_HandSolder" H 2838 7100 50  0001 C CNN
-F 3 "~" H 2800 7250 50  0001 C CNN
-	1    2800 7250
+P 2850 7250
+F 0 "C19" H 2965 7296 50  0000 L CNN
+F 1 "C" H 2965 7205 50  0000 L CNN
+F 2 "Capacitor_SMD:C_0805_2012Metric_Pad1.15x1.40mm_HandSolder" H 2888 7100 50  0001 C CNN
+F 3 "~" H 2850 7250 50  0001 C CNN
+	1    2850 7250
 	1    0    0    -1
 $EndComp
@@
 L Device:C C20
 U 1 1 5CCAD333
-P 3200 7250
-F 0 "C20" H 3315 7296 50  0000 L CNN
-F 1 "C" H 3315 7205 50  0000 L CNN
-F 2 "Capacitor_SMD:C_0805_2012Metric_Pad1.15x1.40mm_HandSolder" H 3238 7100 50  0001 C CNN
-F 3 "~" H 3200 7250 50  0001 C CNN
-	1    3200 7250
+P 3300 7250
+F 0 "C20" H 3415 7296 50  0000 L CNN
+F 1 "C" H 3415 7205 50  0000 L CNN
+F 2 "Capacitor_SMD:C_0805_2012Metric_Pad1.15x1.40mm_HandSolder" H 3338 7100 50  0001 C CNN
+F 3 "~" H 3300 7250 50  0001 C CNN
+	1    3300 7250
 	1    0    0    -1
 $EndComp
@@
 Connection ~ 2400 7000
 Wire Wire Line
-	2400 7000 2800 7000
-Wire Wire Line
-	2800 7100 2800 7000
-Connection ~ 2800 7000
-Wire Wire Line
-	2800 7000 3200 7000
-Wire Wire Line
-	3200 7100 3200 7000
-Connection ~ 3200 7000
-Wire Wire Line
-	3200 7000 3300 7000
+	2400 7000 2850 7000
+Wire Wire Line
+	2850 7100 2850 7000
+Connection ~ 2850 7000
+Wire Wire Line
+	2850 7000 3300 7000
+Wire Wire Line
+	3300 7100 3300 7000
+Connection ~ 3300 7000
+Wire Wire Line
+	3300 7000 3400 7000
 Wire Wire Line
 	2400 7400 2400 7500
 Connection ~ 2400 7500
 Wire Wire Line
-	2400 7500 2800 7500
-Wire Wire Line
-	2800 7400 2800 7500
-Connection ~ 2800 7500
-Wire Wire Line
-	2800 7500 3200 7500
-Wire Wire Line
-	3200 7400 3200 7500
-Connection ~ 3200 7500
-Wire Wire Line
-	3200 7500 3750 7500
+	2400 7500 2850 7500
+Wire Wire Line
+	2850 7400 2850 7500
+Connection ~ 2850 7500
+Wire Wire Line
+	2850 7500 3300 7500
+Wire Wire Line
+	3300 7400 3300 7500
+Connection ~ 3300 7500
+Wire Wire Line
+	3300 7500 3800 7500
 Text HLabel 1750 9900 0    50   Input ~ 0
 Temp
@@
 Text Label 3000 5850 2    50   ~ 0
 5VDC
-Text Label 4150 7000 2    50   ~ 0
+Text Label 4600 7000 2    50   ~ 0
 5VDC
 Wire Wire Line
@@
 Text HLabel 9000 4700 2    50   Output ~ 0
 PWM4
+$Comp
+L Device:Thermistor_PTC TH4
+U 1 1 5CAF42DC
+P 4150 7000
+F 0 "TH4" V 4294 7000 50  0000 C CNN
+F 1 "Thermistor_PTC" V 4294 7000 50  0001 C CNN
+F 2 "Resistor_SMD:R_1206_3216Metric_Pad1.42x1.75mm_HandSolder" H 4200 6800 50  0001 L CNN
+F 3 "~" H 4150 7000 50  0001 C CNN
+	1    4150 7000
+	0    -1   -1   0
+$EndComp
+Wire Wire Line
+	1750 7000 1950 7000
+Wire Wire Line
+	4000 7000 3800 7000
 $EndSCHEMATC

Commit message: schemos ir pcb ruosimas
Connections:
- net MA renamed M1ENA
- net MB renamed M2ENA
Changed lines of the file:
@@
 EESchema Schematic File Version 4
 LIBS:ihouse_power-cache
-EELAYER 26 0
+EELAYER 29 0
 EELAYER END
 $Descr A3 16535 11693
@@
 	2700 10300 3100 10300
 Text HLabel 9000 5800 2    50   Output ~ 0
-MA
+M1ENA
 Text HLabel 9000 5900 2    50   Output ~ 0
-MB
+M2ENA
 Wire Wire Line
 	7150 5500 7600 5500

Commit message: programos rasymas, schemos ir pcb koregavimai. veikia stm bootloaderis per Demonstrator
Parts:
- removed SW1: SW_SPST, Button_Switch_THT:SW_PUSH_6mm, symbol Switch:SW_SPST
Connections:
- net PWM1: now also J4.13 (Pin_13), M1.13 (B0); no longer J3.9 (Pin_9), M1.29 (B4)
- net PWM2: now also J4.14 (Pin_14), M1.14 (B1); no longer J3.8 (Pin_8), M1.28 (B5)
- net PWM3: now also J3.9 (Pin_9), M1.29 (B4); no longer J4.13 (Pin_13), M1.13 (B0)
- net PWM4: now also J3.8 (Pin_8), M1.28 (B5); no longer J4.14 (Pin_14), M1.14 (B1)
- net TBRX: now also J3.14 (Pin_14), M1.34 (A10); no longer J4.8 (Pin_8), M1.8 (A3)
- net TBTX: now also J3.15 (Pin_15), M1.35 (A9); no longer J4.7 (Pin_7), M1.7 (A2)
- removed net A10: J3.14 (Pin_14), M1.34 (A10), U10.12 (R1OUT)
- net A11 renamed QCH_D3
- net A12 renamed QCH_D2
- removed net A9: J3.15 (Pin_15), M1.35 (A9), U10.11 (T1IN)
- net B8 renamed QCH_D0
- net B9 renamed QCH_D1
- net M2ENA renamed M23ENA
- net TBCMD renamed ~TBCMD
- new net A2: J4.7 (Pin_7), M1.7 (A2), U10.11 (T1IN)
- new net A3: J4.8 (Pin_8), M1.8 (A3), U10.12 (R1OUT)
Changed lines of the file:
@@
 $Descr A3 16535 11693
 encoding utf-8
-Sheet 4 5
+Sheet 4 4
 Title ""
 Date ""
@@
 Wire Wire Line
 	3200 1950 3850 1950
-Wire Wire Line
-	6550 4950 6450 4950
 Text HLabel 10300 2700 2    50   Input ~ 0
 230L
@@
 M1ENA
 Text HLabel 9000 5900 2    50   Output ~ 0
-M2ENA
+M23ENA
 Wire Wire Line
 	7150 5500 7600 5500
 Wire Wire Line
 	7150 5400 7600 5400
-Text HLabel 7150 5400 0    50   Output ~ 0
+Text HLabel 7150 6100 0    50   Input ~ 0
 TBTX
-Text HLabel 7150 5500 0    50   Input ~ 0
+Text HLabel 7150 6200 0    50   Output ~ 0
 TBRX
 Text HLabel 9000 6000 2    50   Output ~ 0
-TBCMD
+~TBCMD
 Wire Wire Line
 	7600 4800 7150 4800
@@
 Text Label 7150 6000 0    50   ~ 0
 A8
-Text Label 7150 6300 0    50   ~ 0
+Text Label 7400 6300 0    50   ~ 0
 A11
-Text Label 7150 6100 0    50   ~ 0
+Text Label 7400 6100 0    50   ~ 0
 A9
-Text Label 7150 6200 0    50   ~ 0
+Text Label 7400 6200 0    50   ~ 0
 A10
-Text Label 7150 6400 0    50   ~ 0
+Text Label 7400 6400 0    50   ~ 0
 A12
 Text Label 7150 6500 0    50   ~ 0
@@
 Text Label 9000 5200 2    50   ~ 0
 B7
-Text Label 9000 5300 2    50   ~ 0
+Text Label 8850 5300 2    50   ~ 0
 B8
-Text Label 9000 5400 2    50   ~ 0
+Text Label 8850 5400 2    50   ~ 0
 B9
 Text Label 3500 3350 2    50   ~ 0
@@
 Text Label 9000 6500 2    50   ~ 0
 C15
-Text Label 7400 5400 0    50   ~ 0
+Text Label 7150 5400 0    50   ~ 0
 A2
-Text Label 7400 5500 0    50   ~ 0
+Text Label 7150 5500 0    50   ~ 0
 A3
 Text Label 7150 5900 0    50   ~ 0
@@
 Text Label 9950 4600 0    50   ~ 0
 3VDC
-Text Label 7300 5050 0    50   ~ 0
+Text Label 7150 5050 0    50   ~ 0
 ~RST
 Text Label 12350 5000 0    50   ~ 0
@@
 	5400 1450 6000 1450
 Text Label 4100 4400 2    50   ~ 0
-A9
+A2
 Text Label 4100 4700 2    50   ~ 0
-A10
+A3
 Text Label 3100 7700 2    50   ~ 0
 A0
@@
 	3800 4700 4100 4700
 Wire Wire Line
-	7100 5150 7100 5050
-Wire Wire Line
-	7100 5050 7600 5050
-Wire Wire Line
-	6450 5150 6450 4950
-Connection ~ 6450 4950
-Wire Wire Line
-	6450 4950 6150 4950
+	7150 5050 7600 5050
 Text Label 8850 4700 2    50   ~ 0
 B1
@@
 Text Label 8850 5000 2    50   ~ 0
 B5
-Wire Wire Line
-	6600 5150 6450 5150
-Wire Wire Line
-	7000 5150 7100 5150
-$Comp
-L Switch:SW_SPST SW1
-U 1 1 5CA31C9D
-P 6800 5150
-F 0 "SW1" H 6800 5050 50  0000 C CNN
-F 1 "SW_SPST" H 6800 5294 50  0001 C CNN
-F 2 "Button_Switch_THT:SW_PUSH_6mm" H 6800 5150 50  0001 C CNN
-F 3 "" H 6800 5150 50  0001 C CNN
-	1    6800 5150
-	1    0    0    -1
-$EndComp
 Text Label 8850 4900 2    50   ~ 0
 B4
@@
 	3800 4800 4100 4800
 Text HLabel 9000 4900 2    50   Output ~ 0
+PWM3
+Text HLabel 9000 5000 2    50   Output ~ 0
+PWM4
+Text HLabel 9000 4600 2    50   Output ~ 0
 PWM1
-Text HLabel 9000 5000 2    50   Output ~ 0
+Text HLabel 9000 4700 2    50   Output ~ 0
 PWM2
-Text HLabel 9000 4600 2    50   Output ~ 0
-PWM3
-Text HLabel 9000 4700 2    50   Output ~ 0
-PWM4
 $Comp
 L Device:Thermistor_PTC TH4
@@
 Wire Wire Line
 	4000 7000 3800 7000
+Text HLabel 9000 5300 2    50   Output ~ 0
+QCH_D0
+Text HLabel 9000 5400 2    50   Output ~ 0
+QCH_D1
+Text HLabel 7150 6400 0    50   Output ~ 0
+QCH_D2
+Text HLabel 7150 6300 0    50   Output ~ 0
+QCH_D3
+Wire Wire Line
+	6150 4950 6550 4950
 $EndSCHEMATC
