File: Kicad/ihouse_power/ihouse_power/relays.sch (KiCad schematic (older format))
At the start: 27 parts, among them J1 Conn_02x12_Top_Bottom, J2 Conn_02x05_Top_Bottom, J3 230L, J4 230N, K1 FINDER-34.51, K10 FINDER-34.51, K11 FINDER-41.52, K12 FINDER-34.51, K13 FINDER-34.51, K14 FINDER-34.51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

Commit message: schemos ir pcb paruosimas
Parts:
- removed J3: 230L, mech:Faston_6.3x0.8x14, symbol Connector_Generic:Conn_01x01
- removed J4: 230N, mech:Faston_6.3x0.8x14, symbol Connector_Generic:Conn_01x01
Connections:
- net labels added: VACL, VACN
- wire segments 177 -> 179
- no-connect marks 0 -> 17
Changed lines of the file:
@@
 EESchema Schematic File Version 4
 LIBS:ihouse_power-cache
-EELAYER 29 0
+EELAYER 26 0
 EELAYER END
 $Descr A4 11693 8268
@@
 	8750 5150 8750 5250
 Connection ~ 8750 5250
-$Comp
-L Connector_Generic:Conn_01x01 J?
-U 1 1 5D604662
-P 9200 2500
-AR Path="/5D604662" Ref="J?"  Part="1"
-AR Path="/5D5ECDB6/5D604662" Ref="J3"  Part="1"
-F 0 "J3" V 9200 2300 50  0001 L CNN
-F 1 "230L" V 9300 2400 50  0000 L CNN
-F 2 "mech:Faston_6.3x0.8x14" H 9200 2500 50  0001 C CNN
-F 3 "~" H 9200 2500 50  0001 C CNN
-	1    9200 2500
-	0    -1   -1   0
-$EndComp
-$Comp
-L Connector_Generic:Conn_01x01 J?
-U 1 1 5D604668
-P 9600 2500
-AR Path="/5D604668" Ref="J?"  Part="1"
-AR Path="/5D5ECDB6/5D604668" Ref="J4"  Part="1"
-F 0 "J4" V 9600 2300 50  0001 L CNN
-F 1 "230N" V 9700 2400 50  0000 L CNN
-F 2 "mech:Faston_6.3x0.8x14" H 9600 2500 50  0001 C CNN
-F 3 "~" H 9600 2500 50  0001 C CNN
-	1    9600 2500
-	0    -1   -1   0
-$EndComp
 Text Label 9000 5850 2    50   ~ 0
 230N
@@
 K12L
 Wire Wire Line
-	9200 2700 9200 2950
+	9900 2950 9200 2950
 Wire Wire Line
 	9100 4050 9100 4400
@@
 	9200 3350 9200 3450
 Wire Wire Line
-	9600 2700 9600 2800
+	9900 2800 9600 2800
 Wire Wire Line
 	1150 7150 2000 7150
@@
 Wire Wire Line
 	2850 5500 2600 5500
-Wire Wire Line
-	10350 6000 10550 6000
-Wire Wire Line
-	9850 6000 9650 6000
-Text Label 10550 6000 2    50   ~ 0
+Text Label 9650 5900 0    50   ~ 0
 K14N
-Text Label 9650 6000 0    50   ~ 0
+Text Label 10550 5900 2    50   ~ 0
 K14L
 Text Label 9500 4400 1    50   ~ 0
@@
 Connection ~ 6400 4150
 Connection ~ 7900 4150
+Wire Wire Line
+	9850 5900 9650 5900
+Wire Wire Line
+	10350 5900 10550 5900
+Wire Wire Line
+	9650 6000 9850 6000
+Wire Wire Line
+	10550 6000 10350 6000
+Text Label 9650 6000 0    50   ~ 0
+VACN
+Text Label 10550 6000 2    50   ~ 0
+VACL
+Text Label 9900 2950 2    50   ~ 0
+VACL
+Text Label 9900 2800 2    50   ~ 0
+VACN
+NoConn ~ 9850 5800
+NoConn ~ 10350 5800
+NoConn ~ 9400 3450
+NoConn ~ 9000 3450
+NoConn ~ 8000 3450
+NoConn ~ 6300 3450
+NoConn ~ 5300 3450
+NoConn ~ 9300 1100
+NoConn ~ 10300 1100
+NoConn ~ 8300 1100
+NoConn ~ 7300 1100
+NoConn ~ 6300 1100
+NoConn ~ 5300 1100
+NoConn ~ 4300 1100
+NoConn ~ 3300 1100
+NoConn ~ 2300 1100
+NoConn ~ 1300 1100
 Wire Bus Line
 	750  2100 10200 2100

Commit message: schemos ir pcb ruosimas
Connections:
- net labels added: COM1, COM2
- net labels removed: GND
- wire segments 179 -> 195
Changed lines of the file:
@@
 EESchema Schematic File Version 4
 LIBS:ihouse_power-cache
-EELAYER 26 0
+EELAYER 29 0
 EELAYER END
 $Descr A4 11693 8268
 encoding utf-8
-Sheet 3 4
+Sheet 3 5
 Title ""
 Date ""
@@
 	8700 3400 8700 3450
 $Comp
-L power:GND #PWR?
-U 1 1 5D6045DC
-P 2400 3750
-AR Path="/5D6045DC" Ref="#PWR?"  Part="1"
-AR Path="/5D5ECDB6/5D6045DC" Ref="#PWR0112"  Part="1"
-F 0 "#PWR0112" H 2400 3500 50  0001 C CNN
-F 1 "GND" H 2405 3577 50  0000 C CNN
-F 2 "" H 2400 3750 50  0001 C CNN
-F 3 "" H 2400 3750 50  0001 C CNN
-	1    2400 3750
-	1    0    0    -1
-$EndComp
-$Comp
-L power:GND #PWR?
-U 1 1 5D6045E2
-P 2400 5150
-AR Path="/5D6045E2" Ref="#PWR?"  Part="1"
-AR Path="/5D5ECDB6/5D6045E2" Ref="#PWR0113"  Part="1"
-F 0 "#PWR0113" H 2400 4900 50  0001 C CNN
-F 1 "GND" H 2405 4977 50  0000 C CNN
-F 2 "" H 2400 5150 50  0001 C CNN
-F 3 "" H 2400 5150 50  0001 C CNN
-	1    2400 5150
-	1    0    0    -1
-$EndComp
-$Comp
 L Device:Fuse F?
 U 1 1 5D6045E8
@@
 	1900 6950 1900 6150
 Connection ~ 1900 6150
-$Comp
-L power:GND #PWR?
-U 1 1 5D6045FC
-P 2300 7550
-AR Path="/5D6045FC" Ref="#PWR?"  Part="1"
-AR Path="/5D5ECDB6/5D6045FC" Ref="#PWR0114"  Part="1"
-F 0 "#PWR0114" H 2300 7300 50  0001 C CNN
-F 1 "GND" H 2305 7377 50  0000 C CNN
-F 2 "" H 2300 7550 50  0001 C CNN
-F 3 "" H 2300 7550 50  0001 C CNN
-	1    2300 7550
-	1    0    0    -1
-$EndComp
-$Comp
-L power:GND #PWR?
-U 1 1 5D604602
-P 2400 7550
-AR Path="/5D604602" Ref="#PWR?"  Part="1"
-AR Path="/5D5ECDB6/5D604602" Ref="#PWR0115"  Part="1"
-F 0 "#PWR0115" H 2400 7300 50  0001 C CNN
-F 1 "GND" H 2405 7377 50  0000 C CNN
-F 2 "" H 2400 7550 50  0001 C CNN
-F 3 "" H 2400 7550 50  0001 C CNN
-	1    2400 7550
-	1    0    0    -1
-$EndComp
-$Comp
-L power:GND #PWR?
-U 1 1 5D604608
-P 2600 7550
-AR Path="/5D604608" Ref="#PWR?"  Part="1"
-AR Path="/5D5ECDB6/5D604608" Ref="#PWR0116"  Part="1"
-F 0 "#PWR0116" H 2600 7300 50  0001 C CNN
-F 1 "GND" H 2605 7377 50  0000 C CNN
-F 2 "" H 2600 7550 50  0001 C CNN
-F 3 "" H 2600 7550 50  0001 C CNN
-	1    2600 7550
-	1    0    0    -1
-$EndComp
-$Comp
-L power:GND #PWR?
-U 1 1 5D60460E
-P 2700 7550
-AR Path="/5D60460E" Ref="#PWR?"  Part="1"
-AR Path="/5D5ECDB6/5D60460E" Ref="#PWR0117"  Part="1"
-F 0 "#PWR0117" H 2700 7300 50  0001 C CNN
-F 1 "GND" H 2705 7377 50  0000 C CNN
-F 2 "" H 2700 7550 50  0001 C CNN
-F 3 "" H 2700 7550 50  0001 C CNN
-	1    2700 7550
-	1    0    0    -1
-$EndComp
 Wire Wire Line
 	2800 4150 2900 4150
@@
 	-1   0    0    1
 $EndComp
-$Comp
-L power:GND #PWR?
-U 1 1 5D6046FD
-P 3450 5500
-AR Path="/5D6046FD" Ref="#PWR?"  Part="1"
-AR Path="/5D5ECDB6/5D6046FD" Ref="#PWR0124"  Part="1"
-F 0 "#PWR0124" H 3450 5250 50  0001 C CNN
-F 1 "GND" V 3455 5372 50  0000 R CNN
-F 2 "" H 3450 5500 50  0001 C CNN
-F 3 "" H 3450 5500 50  0001 C CNN
-	1    3450 5500
-	0    -1   -1   0
-$EndComp
 Wire Wire Line
 	2850 5500 2600 5500
@@
 	1    0    0    -1
 $EndComp
-$Comp
-L power:GND #PWR?
-U 1 1 5D604713
-P 1400 6900
-AR Path="/5D604713" Ref="#PWR?"  Part="1"
-AR Path="/5D5ECDB6/5D604713" Ref="#PWR0125"  Part="1"
-F 0 "#PWR0125" H 1400 6650 50  0001 C CNN
-F 1 "GND" H 1405 6727 50  0000 C CNN
-F 2 "" H 1400 6900 50  0001 C CNN
-F 3 "" H 1400 6900 50  0001 C CNN
-	1    1400 6900
-	1    0    0    -1
-$EndComp
 Wire Wire Line
 	1750 6350 1750 6750
@@
 Wire Wire Line
 	950  6150 1900 6150
-$Comp
-L power:GND #PWR?
-U 1 1 5D60472D
-P 1050 5800
-AR Path="/5D60472D" Ref="#PWR?"  Part="1"
-AR Path="/5D5ECDB6/5D60472D" Ref="#PWR0126"  Part="1"
-F 0 "#PWR0126" H 1050 5550 50  0001 C CNN
-F 1 "GND" V 1055 5672 50  0000 R CNN
-F 2 "" H 1050 5800 50  0001 C CNN
-F 3 "" H 1050 5800 50  0001 C CNN
-	1    1050 5800
-	0    -1   -1   0
-$EndComp
-$Comp
-L power:GND #PWR?
-U 1 1 5D604733
-P 1050 5600
-AR Path="/5D604733" Ref="#PWR?"  Part="1"
-AR Path="/5D5ECDB6/5D604733" Ref="#PWR0127"  Part="1"
-F 0 "#PWR0127" H 1050 5350 50  0001 C CNN
-F 1 "GND" V 1055 5472 50  0000 R CNN
-F 2 "" H 1050 5600 50  0001 C CNN
-F 3 "" H 1050 5600 50  0001 C CNN
-	1    1050 5600
-	0    -1   -1   0
-$EndComp
 Wire Wire Line
 	950  5700 1400 5700
@@
 Text HLabel 1050 4850 0    50   Input ~ 0
 REL13
-Wire Wire Line
-	1050 5600 950  5600
-Wire Wire Line
-	1050 5800 950  5800
 Text HLabel 950  5500 0    50   Input ~ 0
 12VDC
 Text HLabel 950  5600 0    50   UnSpc ~ 0
-COM
+COM1
 Text HLabel 950  5700 0    50   Input ~ 0
 5VDC
 Text HLabel 950  5800 0    50   UnSpc ~ 0
-COM
+COM2
 Text HLabel 950  5900 0    50   Input ~ 0
 M1ENA
@@
 NoConn ~ 2300 1100
 NoConn ~ 1300 1100
+Wire Wire Line
+	1400 6900 1400 7650
+Wire Wire Line
+	1400 7650 2300 7650
+Wire Wire Line
+	2700 7650 2700 7550
+Wire Wire Line
+	2600 7550 2600 7650
+Connection ~ 2600 7650
+Wire Wire Line
+	2600 7650 2700 7650
+Wire Wire Line
+	2400 7550 2400 7650
+Connection ~ 2400 7650
+Wire Wire Line
+	2400 7650 2600 7650
+Wire Wire Line
+	2300 7550 2300 7650
+Connection ~ 2300 7650
+Wire Wire Line
+	2300 7650 2400 7650
+Wire Wire Line
+	1150 5800 1150 5600
+Wire Wire Line
+	950  5600 1150 5600
+Wire Wire Line
+	950  5800 1150 5800
+Wire Wire Line
+	1150 5600 1450 5600
+Connection ~ 1150 5600
+Text Label 1600 7650 0    50   ~ 0
+COM
+Text Label 1450 5600 2    50   ~ 0
+COM
+Wire Wire Line
+	3450 5500 3700 5500
+Text Label 3700 5500 2    50   ~ 0
+COM
+Wire Wire Line
+	2400 5150 2400 5200
+Wire Wire Line
+	2400 5200 2100 5200
+Wire Wire Line
+	2400 3750 2400 3800
+Wire Wire Line
+	2400 3800 2100 3800
+Text Label 2100 5200 0    50   ~ 0
+COM
+Text Label 2100 3800 0    50   ~ 0
+COM
 Wire Bus Line
 	750  2100 10200 2100

Commit message: schemos ir pcb ruosimas
Parts:
- added K? (x2): FINDER-41.52, symbol Relay:FINDER-41.52
- added K?: FINDER-34.51, symbol Relay:FINDER-34.51
- added R?: 4R7, symbol Device:R
Connections:
- net +12V: now also K?.11, K?.A2
- net COM1: now also R?.2
- net K3: now also K?.A1
- net K4: now also K?.A2
- net K5: now also K?.A1
- net M2A: now also K?.12; no longer J2.2 (Pin_2), U3.14 (4Y)
- net M2B: now also K?.22; no longer J2.7 (Pin_7), U3.11 (3Y)
- new net: K?.14, K?.14, K?.22, K?.A1, K?.A2
- new net M23A: J2.2 (Pin_2), K?.21, K?.21, U3.14 (4Y)
- new net M23B: J2.7 (Pin_7), K?.11, K?.11, U3.11 (3Y)
- new net M3A: K?.14
- new net M3B: K?.24
- new net OUT: K?.12, K?.24, R?.1
Other:
- note added: "K1 - vonios jungiklis\nK2 - WC jungiklis\nK3 - karsto/salto vandens sklende\n\n\n \nK7 - ventiliatorius vonios\nK8 - virtuves darb. zonos mazas apsvietimas\nK9 - virtuves darb. zonos pilnas apsvietimas\nK10 - koridorius\nK11 - koridorius naktinis apsvietimas\nK12 - garnikas\nK13 - bendras rele (NC)\nK14 - virtuves rozete"
Changed lines of the file:
@@
 EESchema Schematic File Version 4
 LIBS:ihouse_power-cache
-EELAYER 26 0
+EELAYER 29 0
 EELAYER END
 $Descr A4 11693 8268
@@
 $EndComp
 Wire Wire Line
-	2000 6150 1900 6150
-Wire Wire Line
-	2000 6350 1750 6350
-Wire Wire Line
-	1900 6950 1900 6150
-Connection ~ 1900 6150
+	2000 6150 1750 6150
+Wire Wire Line
+	2000 6350 1900 6350
+Wire Wire Line
+	1750 6950 1750 6150
+Connection ~ 1750 6150
 Wire Wire Line
 	2800 4150 2900 4150
@@
 M1A
 Text Label 9650 5700 0    50   ~ 0
-M2A
+M23A
 Text Label 10550 5600 2    50   ~ 0
 M1B
 Text Label 10550 5700 2    50   ~ 0
-M2B
+M23B
 Text Label 3450 6150 2    50   ~ 0
 M1A
@@
 M1B
 Text Label 3450 6950 2    50   ~ 0
-M2A
+M23A
 Text Label 3450 6750 2    50   ~ 0
-M2B
-Wire Wire Line
-	2000 6750 1750 6750
-Wire Wire Line
-	1900 6950 2000 6950
+M23B
+Wire Wire Line
+	2000 6750 1900 6750
+Wire Wire Line
+	1750 6950 2000 6950
 $Comp
 L Device:R R?
@@
 $EndComp
 Wire Wire Line
-	1750 6350 1750 6750
-Connection ~ 1750 6350
+	1900 6350 1900 6750
+Connection ~ 1900 6350
 Wire Wire Line
 	1400 6600 1400 5700
@@
 	1400 5700 2400 5700
 Wire Wire Line
-	950  6350 1750 6350
-Wire Wire Line
-	950  6150 1900 6150
+	950  6350 1900 6350
+Wire Wire Line
+	950  6150 1750 6150
 Wire Wire Line
 	950  5700 1400 5700
@@
 Text Label 2100 3800 0    50   ~ 0
 COM
+Text Notes 5000 7550 0    50   ~ 0
+K1 - vonios jungiklis\nK2 - WC jungiklis\nK3 - karsto/salto vandens sklende\n\n\n \nK7 - ventiliatorius vonios\nK8 - virtuves darb. zonos mazas apsvietimas\nK9 - virtuves darb. zonos pilnas apsvietimas\nK10 - koridorius\nK11 - koridorius naktinis apsvietimas\nK12 - garnikas\nK13 - bendras rele (NC)\nK14 - virtuves rozete
+$Comp
+L Relay:FINDER-41.52 K?
+U 1 1 5CB5537E
+P 16250 5250
+AR Path="/5CB5537E" Ref="K?"  Part="1"
+AR Path="/5D5ECDB6/5CB5537E" Ref="K?"  Part="1"
+F 0 "K?" V 15600 5150 50  0000 L CNN
+F 1 "FINDER-41.52" H 16880 5205 50  0001 L CNN
+F 2 "" H 17600 5220 50  0001 C CNN
+F 3 "http://gfinder.findernet.com/assets/Series/357/S41EN.pdf" H 16050 5250 50  0001 C CNN
+	1    16250 5250
+	0    1    1    0
+$EndComp
+Text Label 15500 5250 0    50   ~ 0
+M23B
+Text Label 15500 5650 0    50   ~ 0
+M23A
+Wire Wire Line
+	16550 4850 16950 4850
+Text Label 16950 4850 2    50   ~ 0
+K3
+Wire Wire Line
+	16550 5150 16950 5150
+Wire Wire Line
+	16550 5550 16750 5550
+Wire Wire Line
+	16750 5550 16750 5250
+Wire Wire Line
+	16750 5250 16950 5250
+Wire Wire Line
+	16550 5750 16950 5750
+Wire Wire Line
+	16550 5350 16650 5350
+Wire Wire Line
+	16650 5350 16650 5650
+Wire Wire Line
+	16650 5650 16950 5650
+Text Label 16950 5150 2    50   ~ 0
+M2A
+Text Label 16950 5250 2    50   ~ 0
+M2B
+Text Label 16950 5650 2    50   ~ 0
+M3A
+Text Label 16950 5750 2    50   ~ 0
+M3B
+$Comp
+L Relay:FINDER-41.52 K?
+U 1 1 5CBEF7DF
+P 14950 5250
+AR Path="/5CBEF7DF" Ref="K?"  Part="1"
+AR Path="/5D5ECDB6/5CBEF7DF" Ref="K?"  Part="1"
+F 0 "K?" V 14300 5150 50  0000 L CNN
+F 1 "FINDER-41.52" H 15580 5205 50  0001 L CNN
+F 2 "" H 16300 5220 50  0001 C CNN
+F 3 "http://gfinder.findernet.com/assets/Series/357/S41EN.pdf" H 14750 5250 50  0001 C CNN
+	1    14950 5250
+	0    -1   1    0
+$EndComp
+Wire Wire Line
+	15250 5250 15950 5250
+Wire Wire Line
+	15250 5650 15950 5650
+Wire Wire Line
+	14650 5150 14450 5150
+Text Label 13800 5750 0    50   ~ 0
+COM
+$Comp
+L power:+12V #PWR?
+U 1 1 5CC5031D
+P 14550 3700
+AR Path="/5CC5031D" Ref="#PWR?"  Part="1"
+AR Path="/5D5ECDB6/5CC5031D" Ref="#PWR?"  Part="1"
+F 0 "#PWR?" H 14550 3550 50  0001 C CNN
+F 1 "+12V" H 14565 3873 50  0000 C CNN
+F 2 "" H 14550 3700 50  0001 C CNN
+F 3 "" H 14550 3700 50  0001 C CNN
+	1    14550 3700
+	1    0    0    -1
+$EndComp
+Wire Wire Line
+	14650 4850 14550 4850
+Wire Wire Line
+	15250 4850 15600 4850
+Text Label 15600 4850 2    50   ~ 0
+K4
+Wire Wire Line
+	14650 5550 14550 5550
+Wire Wire Line
+	14650 5750 14450 5750
+Wire Wire Line
+	14450 5750 14450 5550
+Wire Wire Line
+	14650 5350 14550 5350
+Wire Wire Line
+	14550 5350 14550 5550
+$Comp
+L Relay:FINDER-34.51 K?
+U 1 1 5CCD8501
+P 14950 4000
+AR Path="/5CCD8501" Ref="K?"  Part="1"
+AR Path="/5D5ECDB6/5CCD8501" Ref="K?"  Part="1"
+F 0 "K?" V 14500 3950 50  0000 L CNN
+F 1 "FINDER-34.51" H 15380 3955 50  0001 L CNN
+F 2 "" H 16090 3960 50  0001 C CNN
+F 3 "https://gfinder.findernet.com/public/attachments/34/EN/S34USAEN.pdf" H 14950 4000 50  0001 C CNN
+	1    14950 4000
+	0    1    1    0
+$EndComp
+Wire Wire Line
+	14650 4200 14550 4200
+Wire Wire Line
+	14550 4200 14550 3800
+Wire Wire Line
+	14650 3800 14550 3800
+Connection ~ 14550 3800
+Wire Wire Line
+	14550 3800 14550 3700
+Wire Wire Line
+	15250 4300 15350 4300
+Wire Wire Line
+	15350 4300 15350 4500
+Wire Wire Line
+	15350 4500 14550 4500
+Wire Wire Line
+	14550 4500 14550 4850
+Wire Wire Line
+	15250 3800 15600 3800
+Text Label 15600 3800 2    50   ~ 0
+K5
+Wire Wire Line
+	15950 4850 15850 4850
+Wire Wire Line
+	15850 4850 15850 4500
+Wire Wire Line
+	15850 4500 15350 4500
+Connection ~ 15350 4500
+Wire Wire Line
+	14450 5750 14350 5750
+Connection ~ 14450 5750
+Wire Wire Line
+	14550 4850 14550 5350
+Connection ~ 14550 4850
+Connection ~ 14550 5350
+$Comp
+L Device:R R?
+U 1 1 5CFEF408
+P 14200 5750
+F 0 "R?" V 14200 5750 50  0000 C CNN
+F 1 "4R7" V 14300 5750 50  0000 C CNN
+F 2 "" V 14130 5750 50  0001 C CNN
+F 3 "~" H 14200 5750 50  0001 C CNN
+	1    14200 5750
+	0    1    1    0
+$EndComp
+Wire Wire Line
+	14050 5750 13800 5750
+Wire Wire Line
+	14450 5550 13800 5550
+Connection ~ 14450 5550
+Wire Wire Line
+	14450 5550 14450 5150
+Text Label 13800 5550 0    50   ~ 0
+OUT
 Wire Bus Line
 	750  2100 10200 2100

Commit message: programos rasymas, schemos ir pcb koregavimai. veikia stm bootloaderis per Demonstrator
Parts:
- removed K14: FINDER-34.51, Relay_THT:Relay_SPDT_Finder_34.51_Vertical, symbol Relay:FINDER-34.51
- removed K? (x2): FINDER-41.52, symbol Relay:FINDER-41.52
- removed K?: FINDER-34.51, symbol Relay:FINDER-34.51
- removed R?: 4R7, symbol Device:R
- added K13: FINDER-34.51, Relay_THT:Relay_SPDT_Finder_34.51_Vertical, symbol Relay:FINDER-34.51
- renumbered K12 to K11, K13 to K12, K11 to K14
Connections:
- net M23B is gone; now on net M2B: J2.7 (Pin_7), U3.11 (3Y)
- net +12V: now also K13.A1
- net 230L: now also K10.11, K11.11, K12.11, K3.11, K4.11, K5.11, K6.11, K7.11, K8.11, K9.11
- net K13: now also K13.A2
- net M2A: now also J2.2 (Pin_2), K13.12
- net M2B: now also J2.8 (Pin_8)
- net M3A: now also J2.3 (Pin_3), K13.14
- net M23A: no longer names the net of U3.14 (4Y)
- net M23A: now also K13.11; no longer J2.2 (Pin_2)
- net M2ENA renamed M23ENA
- no-connect marks 17 -> 14
Other:
- note added: "K1 - vonios jungiklis\nK2 - WC jungiklis\n\n\n\n \nK7 - ventiliatorius vonios\nK8 - virtuves darb. zonos mazas apsvietimas\nK9 - virtuves darb. zonos pilnas apsvietimas\nK10 - koridorius\nK11 - koridorius naktinis apsvietimas\nK12 - garnikas\nK13 - karsto/salto vandens sklende\nK14 - virtuves rozete"
- note removed: "K1 - vonios jungiklis\nK2 - WC jungiklis\nK3 - karsto/salto vandens sklende\n\n\n \nK7 - ventiliatorius vonios\nK8 - virtuves darb. zonos mazas apsvietimas\nK9 - virtuves darb. zonos pilnas apsvietimas\nK10 - koridorius\nK11 - koridorius naktinis apsvietimas\nK12 - garnikas\nK13 - bendras rele (NC)\nK14 - virtuves rozete"
- moved on the sheet: J1, J2
