File: Kicad/ihouse_power/ihouse_power/gamyba.kicad_pcb (KiCad board)
At the start: 2 copper layers, 80 x 120 mm, 85 parts, among them J12 OPTIC, J14 OPT1, J15 LEAK1, J16 LEAK2, J17 LEAK3, J18 DHT22, J21 RS232, J22 Nextion, J23 Valve1, J24 Valve2, J25 Conn_01x14, J26 Valve1, J27 Valve2, J28 OPT2, J29 OPT3, U12 MAX232, U6 LM393, U7 LM393

Commit message: schemos ir pcb ruosimas
Parts:
- removed the C31 at (106.4, 85.9)
- removed the C31 at (106.4, 153.9)
- removed the C31 at (79.4, 153.9)
- removed the C31 at (52.4, 153.9)
- removed the C31 at (106.4, 119.9)
- removed the C31 at (79.4, 119.9)
- removed the C32 at (111.3, 85.9)
- removed the C32 at (111.3, 153.9)
- removed the C32 at (84.3, 153.9)
- removed the C32 at (57.3, 153.9)
- removed the C32 at (111.3, 119.9)
- removed the C32 at (84.3, 119.9)
- removed the C33 at (119.7, 76.6)
- removed the C33 at (119.7, 144.6)
- removed the C33 at (92.7, 144.6)
- removed the C33 at (65.7, 144.6)
- removed the C33 at (119.7, 110.6)
- removed the C33 at (92.7, 110.6)
- removed the C34 at (115.3, 85.9)
- removed the C34 at (115.3, 153.9)
- removed the C34 at (88.3, 153.9)
- removed the C34 at (61.3, 153.9)
- removed the C34 at (115.3, 119.9)
- removed the C34 at (88.3, 119.9)
- removed the J21 at (104.3, 91.7)
- removed the J21 at (104.3, 159.7)
- removed the J21 at (77.3, 159.7)
- removed the J21 at (50.3, 159.7)
- removed the J21 at (104.3, 125.7)
- removed the J21 at (77.3, 125.7)
- removed the J22 at (116.4, 70.9)
- removed the J22 at (116.4, 138.9)
- removed the J22 at (89.4, 138.9)
- removed the J22 at (62.4, 138.9)
- removed the J22 at (116.4, 104.9)
- removed the J22 at (89.4, 104.9)
- removed the REF** at (66.6, 58.6)
- removed the U12 at (112.2, 77.7)
- removed the U12 at (112.2, 145.7)
- removed the U12 at (85.2, 145.7)
- removed the U12 at (58.2, 145.7)
- removed the U12 at (112.2, 111.7)
- removed the U12 at (85.2, 111.7)
- added ?: BU+, Connector_Wire:SolderWirePad_1x01_Drill0.8mm, B.Cu at (135.0, 60.6)
- added ?: BU-, Connector_Wire:SolderWirePad_1x01_Drill0.8mm, B.Cu at (131.5, 60.6)
- added C31: 10,0, Capacitor_SMD:CP_Elec_3x5.4, B.Cu at (81.0, 133.6)
- added C32: 10,0, Capacitor_SMD:CP_Elec_3x5.4, B.Cu at (81.0, 138.5)
- added C33: 10,0, Capacitor_SMD:CP_Elec_3x5.4, B.Cu at (90.3, 146.9)
- added C34: 10,0, Capacitor_SMD:CP_Elec_3x5.4, B.Cu at (81.0, 142.5)
- added C39: C, Capacitor_SMD:C_0805_2012Metric_Pad1.15x1.40mm_HandSolder, B.Cu at (139.4, 89.0)
- added C41: 0.1, Capacitor_SMD:C_0805_2012Metric, B.Cu at (137.2, 154.4)
- added C42: 0.1, Capacitor_SMD:C_0805_2012Metric, B.Cu at (131.8, 147.1)
- added CN6: Conn_01x06, Connector_PinHeader_2.54mm:PinHeader_1x06_P2.54mm_Vertical, B.Cu at (134.4, 94.7)
- added D12: BAS32, Diode_SMD:D_MiniMELF, B.Cu at (133.2, 63.3)
- added D8: POWER, LED_THT:LED_D3.0mm, F.Cu at (73.2, 64.7)
- added J21: RS232, Connector_PinHeader_2.54mm:PinHeader_1x08_P2.54mm_Horizontal, B.Cu at (75.2, 131.5)
- added J22: Nextion, Connector_PinHeader_2.54mm:PinHeader_1x04_P2.54mm_Vertical, B.Cu at (96.0, 143.6)
- added J32: Conn_01x06, Connector_PinHeader_2.54mm:PinHeader_1x06_P2.54mm_Vertical, B.Cu at (134.4, 78.0)
- added JP5: 0R, Resistor_SMD:R_0805_2012Metric_Pad1.15x1.40mm_HandSolder, B.Cu at (72.7, 77.9)
- added JP5: 0R, Resistor_SMD:R_0805_2012Metric_Pad1.15x1.40mm_HandSolder, B.Cu at (62.1, 74.8)
- added JP5: 0R, Resistor_SMD:R_0805_2012Metric_Pad1.15x1.40mm_HandSolder, B.Cu at (62.1, 83.8)
- added JP5: 0R, Resistor_SMD:R_0805_2012Metric_Pad1.15x1.40mm_HandSolder, B.Cu at (91.6, 78.1)
- added Q5: BC847, Package_TO_SOT_SMD:SOT-23, B.Cu at (133.1, 57.3)
- added R28: 4.7k, Resistor_SMD:R_0805_2012Metric, B.Cu at (139.4, 50.6)
- added R30: 4.7k, Resistor_SMD:R_0805_2012Metric, B.Cu at (138.4, 97.2)
- added R32: R_PHOTO, Resistor_THT:R_Axial_DIN0204_L3.6mm_D1.6mm_P5.08mm_Horizontal, B.Cu at (131.2, 116.7)
- added R33: R, Resistor_SMD:R_0805_2012Metric_Pad1.15x1.40mm_HandSolder, B.Cu at (136.2, 147.8)
- added R34: 100, Resistor_SMD:R_0805_2012Metric_Pad1.15x1.40mm_HandSolder, B.Cu at (136.9, 142.3)
- added R35: 10k, Resistor_SMD:R_0805_2012Metric_Pad1.15x1.40mm_HandSolder, B.Cu at (133.9, 140.6)
- added R46: 10k, Resistor_SMD:R_0805_2012Metric_Pad1.15x1.40mm_HandSolder, B.Cu at (133.2, 51.6)
- added R47: 10k, Resistor_SMD:R_0805_2012Metric_Pad1.15x1.40mm_HandSolder, B.Cu at (133.2, 53.8)
- added R48: 47, Resistor_SMD:R_1206_3216Metric, B.Cu at (133.2, 65.9)
- added R49: 10k, Resistor_SMD:R_0805_2012Metric_Pad1.15x1.40mm_HandSolder, B.Cu at (72.2, 139.1)
- added R49: 10k, Resistor_SMD:R_0805_2012Metric_Pad1.15x1.40mm_HandSolder, B.Cu at (72.2, 110.6)
- added R7: 4.7k, Resistor_SMD:R_1206_3216Metric, B.Cu at (74.2, 72.0)
- added REF**: MountingHole_3.2mm_M3, MountingHole:MountingHole_3.2mm_M3, F.Cu at (134.4, 127.7)
- added REF**: MountingHole_3.2mm_M3, MountingHole:MountingHole_3.2mm_M3, F.Cu at (134.4, 71.7)
- added RV4: 5k, Potentiometer_THT:Potentiometer_Piher_PT-6-V_Vertical, F.Cu at (131.2, 138.8)
- added SW1: BLDR, Resistor_THT:R_Axial_DIN0411_L9.9mm_D3.6mm_P15.24mm_Horizontal, B.Cu at (139.4, 62.7)
- added SW2: USER, Resistor_THT:R_Axial_DIN0411_L9.9mm_D3.6mm_P15.24mm_Horizontal, B.Cu at (139.4, 107.7)
- added SW3: RESET, Resistor_THT:R_Axial_DIN0411_L9.9mm_D3.6mm_P15.24mm_Horizontal, B.Cu at (139.4, 152.9)
- added U12: MAX232, Package_SO:SOIC-16_3.9x9.9mm_P1.27mm, B.Cu at (89.2, 139.5)
- added U13: LM393, Package_SO:SOIC-8_3.9x4.9mm_P1.27mm, B.Cu at (133.0, 152.7)
- moved J22 35.1 mm to (96.0, 115.1), turned to 0 degrees
- moved J21 33.7 mm to (75.2, 103.0), turned to 180 degrees
- moved C31 32.2 mm to (81.0, 105.1), turned to 0 degrees
- moved U12 31.0 mm to (89.2, 110.9), turned to 0 degrees
- moved C33 25.8 mm to (90.3, 118.4), turned to 0 degrees
- moved C32 25.7 mm to (81.0, 110.0), turned to 0 degrees
- moved C34 20.6 mm to (81.0, 114.0), turned to 0 degrees
- moved R19 14.5 mm to (91.4, 88.0)
- moved R14 14.5 mm to (85.9, 55.5)
- moved R20 14.5 mm to (85.9, 58.4)
- moved C35 14.5 mm to (73.2, 83.0)
- moved J15 14.5 mm to (62.1, 64.1)
- moved J16 14.5 mm to (62.1, 71.1)
- moved J17 14.5 mm to (62.1, 78.1)
- moved RV1 14.5 mm to (69.2, 88.0)
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Connections:
- net /COM renamed Net-(C31-Pad1)
- net /Paskirstymo dezute/DATA renamed /Paskirstymo dezute/DHTIO
- net /RS1 renamed /RSRX
- net /RS2 renamed /RSTX
- J21 pad 4: /RCEN -> Net-(J21-Pad4)
- U12 pad 7: /RCEN -> Net-(U12-Pad7)
Routing:
- net /RSTX: track 257.0 -> 73.4 mm, vias 14 -> 4
- net /5VDC: track 240.7 -> 68.8 mm
- net /RSRX: track 236.6 -> 67.6 mm
- net /MCU plokste/5V@1: track 0.00 -> 105.9 mm
- net /RCEN: track 87.2 -> 0.00 mm
- net Net-(J32-Pad4): track 0.00 -> 69.8 mm, vias 0 -> 2
- net Net-(J32-Pad2): track 0.00 -> 65.7 mm
- net Net-(CN6-Pad3): track 0.00 -> 61.4 mm
- net Net-(C31-Pad2): track 69.5 -> 19.9 mm
- net /MCU plokste/3V@1: track 0.00 -> 40.8 mm
- net Net-(C32-Pad1): track 56.2 -> 16.1 mm
- net Net-(C34-Pad1): track 55.7 -> 15.9 mm
- net Net-(R32-Pad2): track 0.00 -> 37.2 mm
- net Net-(J32-Pad1): track 0.00 -> 30.5 mm
- net Net-(C33-Pad1): track 42.7 -> 12.2 mm
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- added copper zone on B.Cu, net /MCU plokste/COM@1
Other:
- board size 80 x 120 mm -> 84.2 x 120 mm
